File: Eagle files/FLYTE-v1.brd (EAGLE design)
At the start: 116 x 55 mm, 49 parts, among them J2 CONSMA002, Q1 IRF540NPBF, Q2 IRF540NPBF, SW1 1825159-1, U3 CORE1262-868M, U6 W25Q32JVSSIQ

Commit message: Finish ground station
Other:
- board text added: "AADS"
- board text added: "AK47"
- board text added: "AR69"
- board text added: "AXAY"
- board text added: "KayK"
- board text added: "MC04"
- board text added: "NM"
- board text added: "RAGO"
- board text added: "SM01"
Changed lines of the file:
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@@
 <drawing>
 <settings>
-<setting alwaysvectorfont="no"/>
+<setting alwaysvectorfont="yes"/>
 <setting verticaltext="up"/>
 </settings>
-<grid distance="1" unitdist="mm" unit="mm" style="lines" multiple="1" display="no" altdistance="1" altunitdist="mm" altunit="mm"/>
+<grid distance="0.5" unitdist="mm" unit="mm" style="lines" multiple="1" display="no" altdistance="1" altunitdist="mm" altunit="mm"/>
 <layers>
-<layer number="1" name="Top" color="4" fill="1" visible="no" active="yes"/>
+<layer number="1" name="Top" color="4" fill="1" visible="yes" active="yes"/>
 <layer number="2" name="Route2" color="16" fill="1" visible="no" active="no"/>
 <layer number="3" name="Route3" color="17" fill="1" visible="no" active="no"/>
@@
 <layer number="14" name="Route14" color="22" fill="1" visible="no" active="no"/>
 <layer number="15" name="Route15" color="23" fill="1" visible="no" active="no"/>
-<layer number="16" name="Bottom" color="1" fill="1" visible="yes" active="yes"/>
+<layer number="16" name="Bottom" color="1" fill="1" visible="no" active="yes"/>
 <layer number="17" name="Pads" color="2" fill="1" visible="yes" active="yes"/>
 <layer number="18" name="Vias" color="2" fill="1" visible="yes" active="yes"/>
 <layer number="19" name="Unrouted" color="6" fill="1" visible="yes" active="yes"/>
 <layer number="20" name="Dimension" color="24" fill="1" visible="yes" active="yes"/>
-<layer number="21" name="tPlace" color="7" fill="1" visible="no" active="yes"/>
-<layer number="22" name="bPlace" color="7" fill="1" visible="yes" active="yes"/>
-<layer number="23" name="tOrigins" color="15" fill="1" visible="no" active="yes"/>
-<layer number="24" name="bOrigins" color="15" fill="1" visible="yes" active="yes"/>
-<layer number="25" name="tNames" color="7" fill="1" visible="no" active="yes"/>
-<layer number="26" name="bNames" color="7" fill="1" visible="yes" active="yes"/>
+<layer number="21" name="tPlace" color="7" fill="1" visible="yes" active="yes"/>
+<layer number="22" name="bPlace" color="7" fill="1" visible="no" active="yes"/>
+<layer number="23" name="tOrigins" color="15" fill="1" visible="yes" active="yes"/>
+<layer number="24" name="bOrigins" color="15" fill="1" visible="no" active="yes"/>
+<layer number="25" name="tNames" color="7" fill="1" visible="yes" active="yes"/>
+<layer number="26" name="bNames" color="7" fill="1" visible="no" active="yes"/>
 <layer number="27" name="tValues" color="7" fill="1" visible="no" active="yes"/>
 <layer number="28" name="bValues" color="7" fill="1" visible="no" active="yes"/>
@@
 <layer number="37" name="tTest" color="7" fill="1" visible="no" active="yes"/>
 <layer number="38" name="bTest" color="7" fill="1" visible="no" active="yes"/>
-<layer number="39" name="tKeepout" color="4" fill="11" visible="no" active="yes"/>
-<layer number="40" name="bKeepout" color="1" fill="11" visible="yes" active="yes"/>
-<layer number="41" name="tRestrict" color="4" fill="10" visible="no" active="yes"/>
-<layer number="42" name="bRestrict" color="1" fill="10" visible="yes" active="yes"/>
+<layer number="39" name="tKeepout" color="4" fill="11" visible="yes" active="yes"/>
+<layer number="40" name="bKeepout" color="1" fill="11" visible="no" active="yes"/>
+<layer number="41" name="tRestrict" color="4" fill="10" visible="yes" active="yes"/>
+<layer number="42" name="bRestrict" color="1" fill="10" visible="no" active="yes"/>
 <layer number="43" name="vRestrict" color="2" fill="10" visible="no" active="yes"/>
 <layer number="44" name="Drills" color="7" fill="1" visible="no" active="yes"/>
@@
 <layer number="49" name="Reference" color="7" fill="1" visible="no" active="yes"/>
 <layer number="50" name="dxf" color="7" fill="1" visible="no" active="no"/>
-<layer number="51" name="tDocu" color="7" fill="1" visible="no" active="yes"/>
-<layer number="52" name="bDocu" color="7" fill="1" visible="yes" active="yes"/>
+<layer number="51" name="tDocu" color="7" fill="1" visible="yes" active="yes"/>
+<layer number="52" name="bDocu" color="7" fill="1" visible="no" active="yes"/>
 <layer number="53" name="tGND_GNDA" color="7" fill="9" visible="no" active="no"/>
 <layer number="54" name="bGND_GNDA" color="1" fill="9" visible="no" active="no"/>
@@
 <dimension x1="64.4" y1="52.6" x2="0" y2="52.6" x3="32.2" y3="62.1" textsize="1.778" layer="21"/>
 <dimension x1="113.6" y1="37" x2="113.6" y2="55" x3="129.2" y3="46" textsize="1.778" layer="21"/>
+<text x="34.5" y="15" size="1.27" layer="21">RAGO</text>
+<text x="41.5" y="15" size="1.27" layer="21">SM01</text>
+<text x="42.5" y="18" size="1.27" layer="21">NM</text>
+<text x="59" y="19" size="1.27" layer="21">AR69</text>
+<text x="109" y="25" size="1.27" layer="21">MC04</text>
+<text x="109" y="14" size="1.27" layer="21">AK47</text>
+<text x="47.5" y="15" size="1.27" layer="21">KayK</text>
+<text x="28.5" y="15" size="1.27" layer="21">AXAY</text>
+<text x="52.5" y="15" size="1.27" layer="21">AADS</text>
 </plain>
 <attributes>
@@
 <via x="89" y="10" extent="1-16" drill="0.35"/>
 <via x="112" y="11" extent="1-16" drill="0.35"/>
-<via x="62" y="20" extent="1-16" drill="0.35"/>
+<via x="63" y="21" extent="1-16" drill="0.35"/>
 <via x="38" y="19" extent="1-16" drill="0.35"/>
 <via x="30" y="10" extent="1-16" drill="0.35"/>

Commit message: Minor changes
Parts:
- R3, R4: value 3.3K ohm -> 4.7K ohm
Changed lines of the file:
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@@
 <drawing>
 <settings>
-<setting alwaysvectorfont="yes"/>
+<setting alwaysvectorfont="no"/>
 <setting verticaltext="up"/>
 </settings>
@@
 <attribute name="VALUE" x="60.635" y="15.46" size="1.27" layer="28" rot="MR0"/>
 </element>
-<element name="R3" library="rcl" library_urn="urn:adsk.eagle:library:334" package="R0805" package3d_urn="urn:adsk.eagle:package:23553/2" value="3.3K ohm" x="61.8" y="41.2" smashed="yes" rot="MR0">
+<element name="R3" library="rcl" library_urn="urn:adsk.eagle:library:334" package="R0805" package3d_urn="urn:adsk.eagle:package:23553/2" value="4.7K ohm" x="61.8" y="41.2" smashed="yes" rot="MR0">
 <attribute name="NAME" x="65.53" y="42.335" size="1.27" layer="26" rot="MR270"/>
 <attribute name="POPULARITY" value="85" x="61.8" y="41.2" size="1.778" layer="28" rot="MR0" display="off"/>
@@
 <attribute name="VALUE" x="62.435" y="38.66" size="1.27" layer="28" rot="MR0"/>
 </element>
-<element name="R4" library="rcl" library_urn="urn:adsk.eagle:library:334" package="R0805" package3d_urn="urn:adsk.eagle:package:23553/2" value="3.3K ohm" x="61.8" y="38.4" smashed="yes" rot="MR0">
+<element name="R4" library="rcl" library_urn="urn:adsk.eagle:library:334" package="R0805" package3d_urn="urn:adsk.eagle:package:23553/2" value="4.7K ohm" x="61.8" y="38.4" smashed="yes" rot="MR0">
 <attribute name="NAME" x="65.53" y="39.635" size="1.27" layer="26" rot="MR270"/>
 <attribute name="POPULARITY" value="85" x="61.8" y="38.4" size="1.778" layer="28" rot="MR0" display="off"/>
