File: Eagle files/FLYTE-v1.sch (EAGLE design)
At the start: 45 parts, among them J2 CONSMA002, Q1 IRF540NPBF, Q2 IRF540NPBF, SW1 1825159-1, U2 AMS1117-3.3, U3 CORE1262-868M, U4 AMS1117-3.3, U6 W25Q32JVSSIQ

Commit message: Finish wiring and top layout
Parts:
- removed BATT_IN: XT60, XT60:XT60
- removed U2, U4: AMS1117-3.3, AMS1117-3.3:AMS1117-3.3
- added 3.3V_REGULATOR, 5V_REGULATOR: AMS1117-3.3, AMS1117-3.3:AMS1117-3.3
- added BATTERY: XT30UPB-M, XT30UPB-M:XT30UPB-M
Connections:
- net N$4 renamed ANT
- net 3V3: now also 3.3V_REGULATOR.VOUT, D1.A; no longer U2.VOUT
- net 5V: now also 5V_REGULATOR.VOUT; no longer U4.VOUT
- net BUZZER: now also U1.GP6; no longer U1.GP20
- net GND: now also 3.3V_REGULATOR.ADJ/GND, 5V_REGULATOR.ADJ/GND, BATTERY.-; no longer BATT_IN.GND, U2.ADJ/GND, U4.ADJ/GND
- net MAIN: now also U1.GP20; no longer U1.GP14
- net PROG: now also U1.GP14; no longer U1.GP6
- net SERVO1: now also U1.GP7; no longer U1.GP4
- net SERVO2: now also U1.GP8; no longer U1.GP5
- net SERVO3: now also U1.GP4; no longer U1.GP7
- net SERVO4: now also U1.GP5; no longer U1.GP8
- net VCC: now also 3.3V_REGULATOR.VIN, 5V_REGULATOR.VIN, BATTERY.+; no longer BATT_IN.VCC, D1.A, U2.VIN, U4.VIN
Other:
- note added: "MCU and PERIPHERALS"
- note added: "These headers are used to connect servo motors for actuation in future rockets"
- moved on the sheet: C1, C2, C3, C4, D1, DROGUE_IN, DR_ARM_IN, DR_ARM_OUT, JP1, JP2, JP3, JP4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

Commit message: Minor changes
Parts:
- R3, R4: value 3.3K ohm -> 4.7K ohm
Changed lines of the file:
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@@
 <part name="R14" library="rcl" library_urn="urn:adsk.eagle:library:334" deviceset="R-US_" device="R0805" package3d_urn="urn:adsk.eagle:package:23553/2" value="4.7K ohm"/>
 <part name="R15" library="rcl" library_urn="urn:adsk.eagle:library:334" deviceset="R-US_" device="R0805" package3d_urn="urn:adsk.eagle:package:23553/2" value="4.7K ohm"/>
-<part name="R3" library="rcl" library_urn="urn:adsk.eagle:library:334" deviceset="R-US_" device="R0805" package3d_urn="urn:adsk.eagle:package:23553/2" value="3.3K ohm"/>
-<part name="R4" library="rcl" library_urn="urn:adsk.eagle:library:334" deviceset="R-US_" device="R0805" package3d_urn="urn:adsk.eagle:package:23553/2" value="3.3K ohm"/>
+<part name="R3" library="rcl" library_urn="urn:adsk.eagle:library:334" deviceset="R-US_" device="R0805" package3d_urn="urn:adsk.eagle:package:23553/2" value="4.7K ohm"/>
+<part name="R4" library="rcl" library_urn="urn:adsk.eagle:library:334" deviceset="R-US_" device="R0805" package3d_urn="urn:adsk.eagle:package:23553/2" value="4.7K ohm"/>
 <part name="R16" library="rcl" library_urn="urn:adsk.eagle:library:334" deviceset="R-US_" device="R0805" package3d_urn="urn:adsk.eagle:package:23553/2" value="100K ohm"/>
 <part name="R17" library="rcl" library_urn="urn:adsk.eagle:library:334" deviceset="R-US_" device="R0805" package3d_urn="urn:adsk.eagle:package:23553/2" value="100K ohm"/>
