File: Eagle files/TERRA-v1.brd (EAGLE design)
At the start: 100 x 70 mm, 21 parts, among them J1 XT60-M, J2 NANO_FOOTPRINT, SW1 1825159-1, U1 RASPBERRY_PICOTH, U2 CORE1262-868M, U3 AMS1117-3.3, X1 BU-SMA-G

Commit message: Finish ground station
Parts:
- removed S2: (no value), switch:M9040P
- removed U$2: (no value), HX711:HX711
- added DROGUE: (no value), switch:M9040P
- added HX711: HX711, HX711:HX711
- added LS1: BUZZER-PTH, SparkFun-Electromechanical:BUZZER-12MM
- added PICO_PWR: 1825159-1, 1825159-1:SW_1825159-1
- added R3, R4: 4.7K, rcl:R0805
- moved J3 65.9 mm to (25.5, 3.90)
- moved U$1 15.5 mm to (25.8, 28.6), turned to 180 degrees
- moved U3 12.1 mm to (92.0, 53.6), flipped to the bottom
- moved R1 9.30 mm to (54.3, 62.0)
- moved SV1 5.10 mm to (89.0, 8.60)
- moved C2 2.64 mm to (85.8, 52.6), flipped to the bottom, turned to 90 degrees
- moved J1 1.89 mm to (81.0, 65.6), turned to 180 degrees
- moved C1 1.22 mm to (85.8, 56.8), flipped to the bottom, turned to 90 degrees
- moved J2 1.00 mm to (65.0, 24.0)
- turned U1 to 180 degrees
- renumbered S1 to MAIN, SW1 to NANO_PWR, U2 to SX1262, X1 to LORA_ANT
Connections:
- new net BUZZER: J2.7, LS1.-
- new net PICO_PWR: PICO_PWR.2, U1.39
- net 3V3: now also DROGUE.1, HX711.VCC, LS1.+, PICO_PWR.3; no longer S2.1, U$2.VCC, U1.39
- net CLK-ARD: now also HX711.SCK; no longer U$2.SCK
- net CS: now also R3.1
- net DATA: now also HX711.DT; no longer U$2.DT
- net DROG: now also DROGUE.2, U1.17; no longer S2.2, U1.29
- net GND: now also DROGUE.3, HX711.GND, PICO_PWR.1, R3.2, R4.2; no longer S2.3, U$2.GND
- net MAIN: now also U1.15; no longer U1.21
- net N$2: now also HX711.B+; no longer U$2.B+
- net N$3: now also HX711.B-; no longer U$2.B-
- net N$4: now also HX711.A+; no longer U$2.A+
- net N$5: now also HX711.A-; no longer U$2.A-
- net N$6: now also HX711.E-; no longer U$2.E-
- net N$7: now also HX711.E+; no longer U$2.E+
- net SD_CLK: now also J2.16
- net SD_CS: now also J2.13, R4.1
- net SD_MISO: now also J2.15
- net SD_MOSI: now also J2.14
Routing:
- net 3V3: track 0.00 -> 176.4 mm
- net SD_CS: track 0.00 -> 84.0 mm
- net SD_CLK: track 0.00 -> 83.6 mm
- net DIO1: track 0.00 -> 58.7 mm, vias 0 -> 1
- net DIO2: track 0.00 -> 56.6 mm
- net PICO_PWR: track 0.00 -> 54.2 mm
- net CS: track 0.00 -> 46.2 mm, vias 0 -> 1
- net SD_MISO: track 0.00 -> 45.1 mm, vias 0 -> 1
- net SD_MOSI: track 0.00 -> 37.9 mm
- net BUZZER: track 0.00 -> 36.9 mm
- net RESET: track 0.00 -> 36.8 mm, vias 0 -> 1
- net CLK-ARD: track 0.00 -> 36.5 mm
- net DATA: track 0.00 -> 33.8 mm
- net BUSY: track 0.00 -> 33.7 mm
- net MAIN: track 0.00 -> 31.0 mm
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Other:
- board text added: "DEPLOY"
- board text added: "HX breakout"
- board text added: "IITB ROCKET TEAM TERRA-V1"
- board text added: "NANO"
- board text added: "ON"
- board text added: "UART to USB"

Commit message: Minor changes
Parts:
- removed U$4: (no value), holes:3,0
- added U$2: (no value), holes:3,0
- moved U$6 90.0 mm to (5.00, 65.0)
- moved U$3 60.0 mm to (5.00, 5.00)
