File: Eagle files/TERRA-v1.sch (EAGLE design)
At the start: 17 parts, among them J1 XT60-M, J2 NANO_FOOTPRINT, SW1 1825159-1, U1 RASPBERRY_PICOTH, U2 CORE1262-868M, U3 AMS1117-3.3, X1 BU-SMA-G

Commit message: Finish ground station
Parts:
- added LS1: BUZZER-PTH, SparkFun-Electromechanical:BUZZER-PTH
- added PICO_PWR: 1825159-1, 1825159-1:1825159-1
- added R3, R4: 4.7K, rcl:R-US_R0805
- HX711: value (none) -> HX711
- renumbered S1 to MAIN, S2 to DROGUE, SW1 to NANO_PWR, U$2 to HX711, U2 to SX1262, X1 to LORA_ANT
Connections:
- new net BUZZER: J2.D4, LS1.2
- new net PICO_PWR: PICO_PWR.2, U1.VSYS
- net 3V3: now also LS1.1, PICO_PWR.3; no longer U1.VSYS
- net CS: now also R3.1
- net DROG: now also U1.GP13; no longer U1.GP22
- net GND: now also PICO_PWR.1, R3.2, R4.2
- net MAIN: now also U1.GP11; no longer U1.GP16
- net SD_CLK: now also J2.D13
- net SD_CS: now also J2.D10, R4.1
- net SD_MISO: now also J2.D12
- net SD_MOSI: now also J2.D11
