File: FLYTE 2.0/FLYTE-v1.brd (EAGLE design)
At the start: 160 x 100 mm, 45 parts, among them Q1 IRF540NPBF, Q2 IRF540NPBF, U2 XBP9B-XCST-021, U3 ADS1115IDGSR, U6 W25Q32JVSSIQ

Commit message: .
Parts:
- removed U$4: BNO055, BNO055:BNO055
Connections:
- net 3V3: no longer U$4.VIN
- net BNO_INT: no longer U$4.INT
- net GND: no longer U$4.ADR, U$4.GND, U$4.RST
- net SCL: no longer U$4.SCL
- net SDA: no longer U$4.SDA
Changed lines of the file:
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@@
 <element name="U$2" library="BMP280" package="BMP280" override_package3d_urn="urn:adsk.eagle:package:38477931/2" override_package_urn="urn:adsk.eagle:footprint:38477932/1" value="BMP280" x="-27.94" y="81.28" smashed="yes"/>
 <element name="U$3" library="SDREADER" package="SDREADER" override_package3d_urn="urn:adsk.eagle:package:40384096/2" override_package_urn="urn:adsk.eagle:footprint:40384097/1" value="SDREADER" x="-64.77" y="57.15" smashed="yes"/>
-<element name="U$4" library="BNO055" package="BNO055" value="BNO055" x="-39.37" y="59.69" smashed="yes"/>
 <element name="U1" library="RpiPico" package="PICO-PKG-NO_DEBUG" override_package3d_urn="urn:adsk.eagle:package:40381806/2" override_package_urn="urn:adsk.eagle:footprint:40381807/1" value="" x="-26.67" y="27.94" smashed="yes">
 <attribute name="NAME" x="-35.814" y="1.143" size="1.778" layer="25"/>
@@
 <contactref element="U$2" pad="GND"/>
 <contactref element="U$1" pad="SDO"/>
-<contactref element="U$4" pad="GND"/>
-<contactref element="U$4" pad="RST"/>
 <contactref element="U2" pad="10"/>
 <contactref element="R25" pad="2"/>
@@
 <contactref element="C3" pad="1"/>
 <contactref element="C4" pad="1"/>
-<contactref element="U$4" pad="ADR"/>
 <contactref element="U3" pad="3"/>
 <contactref element="C5" pad="2"/>
@@
 <wire x1="-29.21" y1="98.2495" x2="-16.51" y2="98.2495" width="0" layer="19" extent="1-1"/>
 <wire x1="-24.13" y1="82.28" x2="-29.21" y2="98.2495" width="0" layer="19" extent="1-1"/>
-<wire x1="-27.87" y1="77.19" x2="-24.13" y2="82.28" width="0" layer="19" extent="1-1"/>
-<wire x1="-27.87" y1="62.19" x2="-27.87" y2="77.19" width="0" layer="19" extent="1-1"/>
-<wire x1="-20.37" y1="62.19" x2="-27.87" y2="62.19" width="0" layer="19" extent="1-1"/>
-<wire x1="-15.4" y1="48.26" x2="-20.37" y2="62.19" width="0" layer="19" extent="1-1"/>
-<wire x1="-15.4" y1="35.56" x2="-15.4" y2="48.26" width="0" layer="19" extent="1-1"/>
-<wire x1="-15.4" y1="22.86" x2="-15.4" y2="35.56" width="0" layer="19" extent="1-1"/>
-<wire x1="-15.4" y1="10.16" x2="-15.4" y2="22.86" width="0" layer="19" extent="1-1"/>
-<wire x1="-35.4" y1="48.26" x2="-27.87" y2="62.19" width="0" layer="19" extent="1-1"/>
-<wire x1="-35.4" y1="35.56" x2="-35.4" y2="48.26" width="0" layer="19" extent="1-1"/>
-<wire x1="-35.4" y1="22.86" x2="-35.4" y2="35.56" width="0" layer="19" extent="1-1"/>
-<wire x1="-35.4" y1="10.16" x2="-35.4" y2="22.86" width="0" layer="19" extent="1-1"/>
-<wire x1="-45.47" y1="84.285" x2="-27.87" y2="77.19" width="0" layer="19" extent="1-1"/>
+<wire x1="-45.47" y1="84.285" x2="-29.21" y2="98.2495" width="0" layer="19" extent="1-1"/>
 <wire x1="-63.25" y1="84.285" x2="-45.47" y2="84.285" width="0" layer="19" extent="1-1"/>
 <wire x1="-63.77" y1="71.85" x2="-63.25" y2="84.285" width="0" layer="19" extent="1-1"/>
@@
 <wire x1="-94.3" y1="115.57" x2="-87.95" y2="115.57" width="0" layer="19" extent="1-1"/>
 <wire x1="-93.77" y1="83.185" x2="-87.24" y2="97.79" width="0" layer="19" extent="1-1"/>
+<wire x1="-35.4" y1="48.26" x2="-67.31" y2="58.15" width="0" layer="19" extent="1-1"/>
+<wire x1="-35.4" y1="35.56" x2="-35.4" y2="48.26" width="0" layer="19" extent="1-1"/>
+<wire x1="-35.4" y1="22.86" x2="-35.4" y2="35.56" width="0" layer="19" extent="1-1"/>
+<wire x1="-35.4" y1="10.16" x2="-35.4" y2="22.86" width="0" layer="19" extent="1-1"/>
+<wire x1="-15.4" y1="48.26" x2="-35.4" y2="48.26" width="0" layer="19" extent="1-1"/>
+<wire x1="-15.4" y1="35.56" x2="-15.4" y2="48.26" width="0" layer="19" extent="1-1"/>
+<wire x1="-15.4" y1="22.86" x2="-15.4" y2="35.56" width="0" layer="19" extent="1-1"/>
+<wire x1="-15.4" y1="10.16" x2="-15.4" y2="22.86" width="0" layer="19" extent="1-1"/>
 <wire x1="-65.61" y1="8.53" x2="-35.4" y2="10.16" width="0" layer="19" extent="1-1"/>
 </signal>
@@
 <contactref element="R4" pad="2"/>
 <contactref element="U$2" pad="SCL"/>
-<contactref element="U$4" pad="SCL"/>
 <contactref element="U3" pad="10"/>
 <wire x1="-21.59" y1="82.28" x2="-40.96" y2="115.57" width="0" layer="19" extent="1-1"/>
-<wire x1="-25.37" y1="62.19" x2="-21.59" y2="82.28" width="0" layer="19" extent="1-1"/>
-<wire x1="-35.4" y1="43.18" x2="-25.37" y2="62.19" width="0" layer="19" extent="1-1"/>
+<wire x1="-35.4" y1="43.18" x2="-21.59" y2="82.28" width="0" layer="19" extent="1-1"/>
 <wire x1="-74.93" y1="58.15" x2="-35.4" y2="43.18" width="0" layer="19" extent="1-1"/>
 <wire x1="-82.94" y1="98.79" x2="-74.93" y2="58.15" width="0" layer="19" extent="1-1"/>
@@
 <contactref element="R3" pad="2"/>
 <contactref element="U$2" pad="SDA"/>
-<contactref element="U$4" pad="SDA"/>
 <contactref element="U3" pad="9"/>
 <wire x1="-19.05" y1="82.28" x2="-30.8" y2="115.57" width="0" layer="19" extent="1-1"/>
-<wire x1="-22.87" y1="62.19" x2="-19.05" y2="82.28" width="0" layer="19" extent="1-1"/>
-<wire x1="-35.4" y1="45.72" x2="-22.87" y2="62.19" width="0" layer="19" extent="1-1"/>
+<wire x1="-35.4" y1="45.72" x2="-19.05" y2="82.28" width="0" layer="19" extent="1-1"/>
 <wire x1="-72.39" y1="58.15" x2="-35.4" y2="45.72" width="0" layer="19" extent="1-1"/>
 <wire x1="-82.94" y1="98.29" x2="-72.39" y2="58.15" width="0" layer="19" extent="1-1"/>
@@
 <contactref element="D1" pad="A"/>
 <contactref element="U$2" pad="VCC"/>
-<contactref element="U$4" pad="VIN"/>
 <contactref element="R22" pad="1"/>
 <contactref element="3.3V_REGULATOR1" pad="2"/>
@@
 <wire x1="-26.67" y1="82.28" x2="-43.18" y2="84.285" width="0" layer="19" extent="1-1"/>
 <wire x1="-13.97" y1="107.95" x2="-32.7" y2="115.57" width="0" layer="19" extent="1-1"/>
-<wire x1="-32.87" y1="62.19" x2="-26.67" y2="82.28" width="0" layer="19" extent="1-1"/>
 <wire x1="-63.77" y1="59.15" x2="-60.96" y2="84.285" width="0" layer="19" extent="1-1"/>
 <wire x1="-80.01" y1="58.15" x2="-63.77" y2="59.15" width="0" layer="19" extent="1-1"/>
@@
 </signal>
 <signal name="BNO_INT">
-<contactref element="U$4" pad="INT"/>
 <contactref element="U1" pad="P$19"/>
-<wire x1="-35.4" y1="7.62" x2="-30.37" y2="77.19" width="0" layer="19" extent="1-1"/>
 </signal>
 <signal name="ATTN">
