File: FLYTE 2.0/FLYTE-v1.sch (EAGLE design)
At the start: 48 parts, among them Q1 IRF540NPBF, Q2 IRF540NPBF, SW1 1825159-1, U2 XBP9B-XCST-021, U6 W25Q32JVSSIQ

Commit message: Cleanup resistors, add ADC
Parts:
- removed R18: 4.7K ohm, rcl:R-US_R0805
- removed R19, R20, R21, R7: 100K ohm, rcl:R-US_R0805
- removed SW1: 1825159-1, 1825159-1:1825159-1
- added C5: 0.1uF, SparkFun-Capacitors:22UF-0805-6.3V-20%
- added JP1: (no value), pinhead:PINHD-1X2
- added U3: ADS1115IDGSR, ADS1115IDGSR:ADS1115IDGSR
- R1, R8: value 470ohm -> 4.7K
Connections:
- removed net N$10: R7.2, U$2.SDO
- removed net N$11: R20.2, U$4.RST
- removed net N$15: R21.1, U$4.ADR
- removed net N$16: R21.2
- removed net N$9: R19.2, U$1.SDO
- removed net PROG: R18.2, SW1.2
- new net VBUS_REG: 3.3V_REGULATOR1.VIN, C4.2, JP1.2
- net 3.3V: now also U$2.SDO; no longer R7.1
- net 3V3: now also C5.1, U2.VCC, U3.AIN2, U3.VDD; no longer SW1.3
- net GND: now also C5.2, U$1.SDO, U$4.ADR, U$4.RST, U3.ADDR, U3.GND; no longer R18.1, R19.1, R20.1, SW1.1
- net SCL: now also U3.SCL
- net SDA: now also U3.SDA
- net SENSE_DROG: now also U3.AIN1
- net SENSE_MAIN: now also U3.AIN0
- net VBUS: now also JP1.1; no longer 3.3V_REGULATOR1.VIN, C4.2
- net VCC: now also U3.AIN3; no longer U2.VCC
Other:
- note added: "Push button to reset pico (Bad idea)"
- note removed: "GPS"
- note removed: "LoRa TELEMETRY"
- note removed: "MCU and PERIPHERALS"
- note removed: "POWER and PYRO"
- note removed: "Push button to reset pico"
- note removed: "SENSORS and LOGGING"
- note removed: "This is the program switch. When ON, data logging is enabled and liftoff detection is running When OFF, No sensors or logging is running Current drains when PROG is high"

Commit message: .
Parts:
- removed U$4: BNO055, BNO055:BNO055
Connections:
- net 3V3: no longer U$4.VIN
- net BNO_INT: no longer U$4.INT
- net GND: no longer U$4.ADR, U$4.GND, U$4.RST
- net SCL: no longer U$4.SCL
- net SDA: no longer U$4.SDA
Changed lines of the file:
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@@
 <part name="BATTERY" library="XT30UPB-M" deviceset="XT30UPB-M" device="" override_package3d_urn="urn:adsk.eagle:package:40384065/5" override_package_urn="urn:adsk.eagle:footprint:40384066/1" override_locally_modified="yes"/>
 <part name="U$2" library="BMP280" deviceset="BMP280" device="" override_package3d_urn="urn:adsk.eagle:package:38477931/2" override_package_urn="urn:adsk.eagle:footprint:38477932/1"/>
-<part name="U$4" library="BNO055" deviceset="BNO055" device=""/>
 <part name="U2" library="XBP9B-XCST-021" deviceset="XBP9B-XCST-021" device=""/>
 <part name="R22" library="rcl" library_urn="urn:adsk.eagle:library:334" deviceset="R-US_" device="R0805" package3d_urn="urn:adsk.eagle:package:23553/2" value="4.7K ohm"/>
@@
 </instance>
 <instance part="U$2" gate="G$1" x="358.14" y="88.9" smashed="yes" rot="R270"/>
-<instance part="U$4" gate="G$1" x="368.3" y="55.88" smashed="yes" rot="R90"/>
 <instance part="U2" gate="G$1" x="213.36" y="218.44" smashed="yes">
 <attribute name="NAME" x="190.4351" y="243.9121" size="1.2736" layer="95"/>
@@
 </segment>
 <segment>
-<pinref part="U$4" gate="G$1" pin="GND"/>
 <wire x1="345.44" y1="53.34" x2="337.82" y2="53.34" width="0.1524" layer="91"/>
 <label x="337.82" y="53.34" size="1.27" layer="95" rot="R180" xref="yes"/>
@@
 <segment>
 <label x="337.82" y="63.5" size="1.27" layer="95" rot="R180" xref="yes"/>
-<pinref part="U$4" gate="G$1" pin="RST"/>
 <wire x1="337.82" y1="63.5" x2="345.44" y2="63.5" width="0.1524" layer="91"/>
 </segment>
@@
 </segment>
 <segment>
-<pinref part="U$4" gate="G$1" pin="ADR"/>
 <wire x1="373.38" y1="53.34" x2="378.46" y2="53.34" width="0.1524" layer="91"/>
 <label x="378.46" y="53.34" size="1.27" layer="95" xref="yes"/>
@@
 </segment>
 <segment>
-<pinref part="U$4" gate="G$1" pin="SCL"/>
 <wire x1="345.44" y1="58.42" x2="337.82" y2="58.42" width="0.1524" layer="91"/>
 <label x="337.82" y="58.42" size="1.27" layer="95" rot="R180" xref="yes"/>
@@
 </segment>
 <segment>
-<pinref part="U$4" gate="G$1" pin="SDA"/>
 <wire x1="345.44" y1="60.96" x2="337.82" y2="60.96" width="0.1524" layer="91"/>
 <label x="337.82" y="60.96" size="1.27" layer="95" rot="R180" xref="yes"/>
@@
 </segment>
 <segment>
-<pinref part="U$4" gate="G$1" pin="VIN"/>
 <wire x1="345.44" y1="48.26" x2="337.82" y2="48.26" width="0.1524" layer="91"/>
 <label x="337.82" y="48.26" size="1.27" layer="95" rot="R180" xref="yes"/>
@@
 <net name="BNO_INT" class="0">
 <segment>
-<pinref part="U$4" gate="G$1" pin="INT"/>
 <wire x1="373.38" y1="48.26" x2="375.92" y2="48.26" width="0.1524" layer="91"/>
 <label x="375.92" y="48.26" size="1.27" layer="95" xref="yes"/>
