File: Eagle files/FLYTE 2.0/FLYTE-v1.sch (EAGLE design)
At the start: 43 parts, among them Q1 IRF540NPBF, Q2 IRF540NPBF, U2 XBP9B-XCST-021, U6 W25Q32JVSSIQ

Commit message: bno added
Parts:
- added C5: 0.1uF, SparkFun-Capacitors:22UF-0805-6.3V-20%
- added U3: ADS1115IDGSR, ADS1115IDGSR:ADS1115IDGSR
Connections:
- net 3V3: now also C5.1, U3.AIN2, U3.VDD
- net GND: now also C5.2, U3.ADDR, U3.GND
- net SCL: now also U3.SCL
- net SDA: now also U3.SDA
- net SENSE_DROG: now also U3.AIN1
- net SENSE_MAIN: now also U3.AIN0
- net VCC: now also U3.AIN3
Other:
- note removed: "GPS"
- note removed: "LoRa TELEMETRY"
- note removed: "MCU and PERIPHERALS"
- note removed: "POWER and PYRO"
- note removed: "SENSORS and LOGGING"
