File: Eagle files/FLYTE 2.0/FLYTE-v2.sch (EAGLE design)
At the start: 45 parts, among them Q1 IRF540NPBF, Q2 IRF540NPBF, U2 XBP9B-XCST-021, U3 ADS1115IDGSR, U6 W25Q32JVSSIQ

Commit message: Add JST, MOSFET, and high g accel
Parts:
- added C6: 10 uF, SparkFun-Capacitors:22UF-0805-6.3V-20%
- added C7: 100 nF, SparkFun-Capacitors:22UF-0805-6.3V-20%
- added GPS, MOTOR, SERIAL: 4392, 4392:4392
- added R2, R5: 4.7K ohm, rcl:R-US_R0805
- added S2: MOMENTARY-SWITCH-SPST-PTH-6.0MM, SparkFun-Switches:MOMENTARY-SWITCH-SPST-PTH-6.0MM
- added U4: H3LIS200DLTR, H3LIS200DLTR:H3LIS200DLTR
- added U5, U7: BS170F, BS170F:BS170F
Connections:
- removed net SX_DIO13: U1.GP22, U2.DOUT/DIO13
- new net N$3: S2.1, U1.GP22
- new net SDA1: R5.2
- net 3V3: now also C6.1, C7.1, GPS.4, R2.1, R5.1, U4.VDD, U4.VDD_IO
- net DROGUE: now also U5.G
- net GND: now also C6.2, C7.2, GPS.1, GPS.MP1, GPS.MP2, MOTOR.1, MOTOR.MP1, MOTOR.MP2, S2.2, SERIAL.1, SERIAL.MP1, SERIAL.MP2, U4.GND, U4.SDO/SA0, U5.S, U7.S
- net MAIN: now also U7.G
- net N$12: now also U5.D
- net N$13: now also U7.D
- net RX: now also GPS.3
- net SCL: now also U4.SCL/SPC
- net SCL0: now also MOTOR.3
- net SDA: now also U4.SDA/SDI/SDO
- net SDA0: now also MOTOR.2, R2.2
- net SER_RX: now also SERIAL.3
- net SER_TX: now also SERIAL.2
- net TX: now also GPS.2
Other:
- note added: "Push button for interfacing (Bad idea?)"

Commit message: Delete extra BMP
Parts:
- removed U$2: BMP280, BMP280:BMP280
Connections:
- removed net 3.3V: U$2.SDO
- net 3V3: no longer U$2.VCC
- net GND: no longer U$2.GND
- net SCL: no longer U$2.SCL
- net SDA: no longer U$2.SDA
Changed lines of the file:
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@@
 <part name="S1" library="SparkFun-Switches" deviceset="MOMENTARY-SWITCH-SPST" device="-PTH-6.0MM" override_package3d_urn="urn:adsk.eagle:package:40381829/2" override_package_urn="urn:adsk.eagle:footprint:40381830/1"/>
 <part name="BATTERY" library="XT30UPB-M" deviceset="XT30UPB-M" device="" override_package3d_urn="urn:adsk.eagle:package:40384065/5" override_package_urn="urn:adsk.eagle:footprint:40384066/1" override_locally_modified="yes"/>
-<part name="U$2" library="BMP280" deviceset="BMP280" device="" override_package3d_urn="urn:adsk.eagle:package:38477931/2" override_package_urn="urn:adsk.eagle:footprint:38477932/1"/>
 <part name="U2" library="XBP9B-XCST-021" deviceset="XBP9B-XCST-021" device=""/>
 <part name="R22" library="rcl" library_urn="urn:adsk.eagle:library:334" deviceset="R-US_" device="R0805" package3d_urn="urn:adsk.eagle:package:23553/2" value="4.7K ohm"/>
@@
 </plain>
 <instances>
-<instance part="U$1" gate="G$1" x="358.14" y="101.6" smashed="yes" rot="R270"/>
+<instance part="U$1" gate="G$1" x="358.14" y="81.28" smashed="yes" rot="R270"/>
 <instance part="U$3" gate="G$1" x="279.4" y="78.74" smashed="yes" rot="R90"/>
 <instance part="Q2" gate="G$1" x="309.88" y="152.4" smashed="yes">
@@
 <attribute name="NAME" x="327.152" y="228.6" size="1.778" layer="95" rot="R90"/>
 </instance>
-<instance part="U$2" gate="G$1" x="358.14" y="81.28" smashed="yes" rot="R270"/>
 <instance part="U2" gate="G$1" x="213.36" y="218.44" smashed="yes">
 <attribute name="NAME" x="190.4351" y="243.9121" size="1.2736" layer="95"/>
@@
 <segment>
 <pinref part="U$1" gate="G$1" pin="GND"/>
-<wire x1="342.9" y1="104.14" x2="335.28" y2="104.14" width="0.1524" layer="91"/>
-<label x="335.28" y="104.14" size="1.27" layer="95" rot="R180" xref="yes"/>
+<wire x1="342.9" y1="83.82" x2="335.28" y2="83.82" width="0.1524" layer="91"/>
+<label x="335.28" y="83.82" size="1.27" layer="95" rot="R180" xref="yes"/>
 </segment>
 <segment>
@@
 </segment>
 <segment>
-<pinref part="U$2" gate="G$1" pin="GND"/>
-<wire x1="342.9" y1="83.82" x2="335.28" y2="83.82" width="0.1524" layer="91"/>
-<label x="335.28" y="83.82" size="1.27" layer="95" rot="R180" xref="yes"/>
-</segment>
-<segment>
-<label x="335.28" y="93.98" size="1.27" layer="95" rot="R180" xref="yes"/>
+<label x="335.28" y="73.66" size="1.27" layer="95" rot="R180" xref="yes"/>
 <pinref part="U$1" gate="G$1" pin="SDO"/>
-<wire x1="342.9" y1="93.98" x2="335.28" y2="93.98" width="0.1524" layer="91"/>
+<wire x1="342.9" y1="73.66" x2="335.28" y2="73.66" width="0.1524" layer="91"/>
 </segment>
 <segment>
@@
 <segment>
 <pinref part="U$1" gate="G$1" pin="SCL"/>
-<wire x1="342.9" y1="101.6" x2="335.28" y2="101.6" width="0.1524" layer="91"/>
-<label x="335.28" y="101.6" size="1.4224" layer="95" rot="R180" xref="yes"/>
-<label x="335.28" y="101.6" size="1.4224" layer="95" rot="R180" xref="yes"/>
-<label x="335.28" y="101.6" size="1.4224" layer="95" rot="R180" xref="yes"/>
+<wire x1="342.9" y1="81.28" x2="335.28" y2="81.28" width="0.1524" layer="91"/>
+<label x="335.28" y="81.28" size="1.4224" layer="95" rot="R180" xref="yes"/>
+<label x="335.28" y="81.28" size="1.4224" layer="95" rot="R180" xref="yes"/>
+<label x="335.28" y="81.28" size="1.4224" layer="95" rot="R180" xref="yes"/>
 </segment>
 <segment>
@@
 </segment>
 <segment>
-<pinref part="U$2" gate="G$1" pin="SCL"/>
-<wire x1="342.9" y1="81.28" x2="335.28" y2="81.28" width="0.1524" layer="91"/>
-<label x="335.28" y="81.28" size="1.27" layer="95" rot="R180" xref="yes"/>
-</segment>
-<segment>
 <wire x1="340.36" y1="17.78" x2="335.28" y2="17.78" width="0.1524" layer="91"/>
 <label x="335.28" y="17.78" size="1.27" layer="95" rot="R180" xref="yes"/>
@@
 <segment>
 <pinref part="U$1" gate="G$1" pin="SDA"/>
-<wire x1="342.9" y1="99.06" x2="335.28" y2="99.06" width="0.1524" layer="91"/>
-<label x="335.28" y="99.06" size="1.4224" layer="95" rot="R180" xref="yes"/>
+<wire x1="342.9" y1="78.74" x2="335.28" y2="78.74" width="0.1524" layer="91"/>
+<label x="335.28" y="78.74" size="1.4224" layer="95" rot="R180" xref="yes"/>
 </segment>
 <segment>
@@
 </segment>
 <segment>
-<pinref part="U$2" gate="G$1" pin="SDA"/>
-<wire x1="342.9" y1="78.74" x2="335.28" y2="78.74" width="0.1524" layer="91"/>
-<label x="335.28" y="78.74" size="1.27" layer="95" rot="R180" xref="yes"/>
-</segment>
-<segment>
 <wire x1="340.36" y1="10.16" x2="335.28" y2="10.16" width="0.1524" layer="91"/>
 <label x="335.28" y="10.16" size="1.27" layer="95" rot="R180" xref="yes"/>
@@
 <segment>
 <pinref part="U$1" gate="G$1" pin="VCC"/>
-<wire x1="342.9" y1="106.68" x2="335.28" y2="106.68" width="0.1524" layer="91"/>
-<label x="335.28" y="106.68" size="1.27" layer="95" rot="R180" xref="yes"/>
+<wire x1="342.9" y1="86.36" x2="335.28" y2="86.36" width="0.1524" layer="91"/>
+<label x="335.28" y="86.36" size="1.27" layer="95" rot="R180" xref="yes"/>
 </segment>
 <segment>
@@
 <label x="208.28" y="134.62" size="1.27" layer="95" xref="yes"/>
 <wire x1="200.66" y1="134.62" x2="208.28" y2="134.62" width="0.1524" layer="91"/>
-</segment>
-<segment>
-<pinref part="U$2" gate="G$1" pin="VCC"/>
-<wire x1="342.9" y1="86.36" x2="335.28" y2="86.36" width="0.1524" layer="91"/>
-<label x="335.28" y="86.36" size="1.27" layer="95" rot="R180" xref="yes"/>
 </segment>
 <segment>
@@
 </segment>
 </net>
-<net name="3.3V" class="0">
-<segment>
-<label x="335.28" y="73.66" size="1.27" layer="95" rot="R180" xref="yes"/>
-<pinref part="U$2" gate="G$1" pin="SDO"/>
-<wire x1="335.28" y1="73.66" x2="342.9" y2="73.66" width="0.1524" layer="91"/>
-</segment>
-</net>

Commit message: Improve pyros
Parts:
- removed BATTERY, DROGUE, MAIN: XT30UPB-M, XT30UPB-M:XT30UPB-M
- removed MA_ARM: (no value), con-wago-500:W237-102
- removed Q1, Q2: IRF540NPBF, IRF540NPBF:IRF540NPBF
- removed R24, R26: 100K ohm, rcl:R-US_R0805
- added DROGUE_PYRO, J1, MAIN_PYRO: XT30PW-M, XT30PW-M:XT30PW-M
- added MAIN_ARM: (no value), con-wago-500:W237-102
- added R6: 4.7K, rcl:R-US_R0805
- added R7: 10 ohm, rcl:R-US_0207/10
- R11, R12: value 10 ohm -> 100K ohm; device rcl:R-US_0207/10 -> rcl:R-US_R0805
- R8: value 4.7K -> 10 ohm; device rcl:R-US_R0805 -> rcl:R-US_0207/10
- renumbered 3.3V_REGULATOR to BATTERY_REGULATOR3V3, 3.3V_REGULATOR1 to USB_REGULATOR3V3
Connections:
- removed net N$13: Q1.D, R11.2, R12.2, R24.1, U7.D
- removed net N$14: MAIN.-, MA_ARM-1.KL
- new net N$4: MAIN_PYRO.N, R7.1, R8.1
- new net N$5: R11.1, R7.2, R8.2, U7.D
- net 3V3: now also SERIAL.4
- net DROGUE: now also R1.2; no longer Q2.G, R1.1
- net GND: now also GPS.3, J1.N, R1.1, R12.2, R6.1; no longer BATTERY.-, GPS.1, Q1.S, Q2.S, R1.2, R26.2, R8.2
- net MAIN: now also R6.2; no longer Q1.G, R8.1
- net N$12: no longer Q2.D
- net N$2: now also DROGUE_PYRO.P, DR_ARM-2.KL; no longer DROGUE.-, DR_ARM-1.KL
- net N$6: now also MAIN_ARM-2.KL, MAIN_PYRO.P; no longer MAIN.+, R11.1, R12.1
- net N$7: now also DROGUE_PYRO.N; no longer DROGUE.+
- net RX: now also GPS.1; no longer GPS.3
- net SENSE_DROG: now also R23.2, R25.1; no longer R24.2, R26.1
- net SENSE_MAIN: now also R11.2, R12.1; no longer R23.2, R25.1
- net VCC: now also DR_ARM-1.KL, J1.P, MAIN_ARM-1.KL; no longer BATTERY.+, DR_ARM-2.KL, MA_ARM-2.KL
Other:
- note added: "Push button to reset pico (Bad idea, do not solder in actual board)"
- note removed: "Push button to reset pico (Bad idea)"
- moved on the sheet: DR_ARM-1, DR_ARM-2, LS1, R1, R10, R11, R12, R23, R25, R8, R9, U5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

Commit message: Cleanup main board and add motor controller
Parts:
- added H1, H2, H3, H4: MOUNT-PAD-ROUND3.0, holes:MOUNT-PAD-ROUND3.0
Connections:
- net MISO_0 renamed MISO0
- net MISO_1 renamed MISO1
- net MOSI_0 renamed MOSI0
- net MOSI_1 renamed MOSI1
- net SCK_0 renamed SCK0
- net SCK_1 renamed SCK1
- net SCL renamed SCL1
- removed net SDA: R3.2, U$1.SDA, U$4.SDA, U1.GP2, U3.SDA, U4.SDA/SDI/SDO
- new net AIR_DATA: U1.GP28
- new net AIR_SCK: U1.GP27
- net GND: now also H1.MOUNT, H2.MOUNT, H3.MOUNT, H4.MOUNT
- net SCL0: now also R5.2
- net SDA1: now also R3.2, U$1.SDA, U$4.SDA, U1.GP2, U3.SDA, U4.SDA/SDI/SDO; no longer R5.2
- net SENSE_DROG: no longer U1.GP27
- net SENSE_MAIN: no longer U1.GP28
Other:
- note added: "DATA LOGGING"
- note added: "MICROCONTOLLER AND PERIPHERALS"
- note added: "POWER AND PYROS"
- note added: "SENSORS"
- note added: "Sensors are on the I2C_1 bus (Except the ram air speed sensor)"
- note added: "TELEMETRY"
- moved on the sheet: BATTERY_REGULATOR3V3, C1, C2, C3, C4, C5, C6, C7, D1, D3, DROGUE_PYRO, DR_ARM-1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

Commit message: Start layout
Parts:
- added JP2: (no value), pinhead:PINHD-1X4
- renumbered J1 to POWER
Connections:
- net 3V3: now also JP2.4
- net AIR_DATA: now also JP2.3
- net AIR_SCK: now also JP2.2
- net GND: now also JP2.1
- net N$2: now also DROGUE_PYRO.N, DR_ARM-1.KL; no longer DROGUE_PYRO.P, DR_ARM-2.KL
- net N$7: now also DROGUE_PYRO.P; no longer DROGUE_PYRO.N
- net VCC: now also DR_ARM-2.KL; no longer DR_ARM-1.KL
Other:
- moved on the sheet: DROGUE_PYRO, DR_ARM-1, DR_ARM-2
Changed lines of the file:
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@@
 <part name="R2" library="rcl" library_urn="urn:adsk.eagle:library:334" deviceset="R-US_" device="R0805" package3d_urn="urn:adsk.eagle:package:23553/2" value="4.7K ohm"/>
 <part name="R5" library="rcl" library_urn="urn:adsk.eagle:library:334" deviceset="R-US_" device="R0805" package3d_urn="urn:adsk.eagle:package:23553/2" value="4.7K ohm"/>
-<part name="J1" library="XT30PW-M" deviceset="XT30PW-M" device=""/>
+<part name="POWER" library="XT30PW-M" deviceset="XT30PW-M" device=""/>
 <part name="DROGUE_PYRO" library="XT30PW-M" deviceset="XT30PW-M" device=""/>
 <part name="R6" library="rcl" library_urn="urn:adsk.eagle:library:334" deviceset="R-US_" device="R0805" package3d_urn="urn:adsk.eagle:package:23553/2" value="4.7K"/>
 <part name="R7" library="rcl" library_urn="urn:adsk.eagle:library:334" deviceset="R-US_" device="0207/10" package3d_urn="urn:adsk.eagle:package:23491/2" value="10 ohm"/>
 <part name="R8" library="rcl" library_urn="urn:adsk.eagle:library:334" deviceset="R-US_" device="0207/10" package3d_urn="urn:adsk.eagle:package:23491/2" value="10 ohm"/>
-<part name="MAIN_ARM" library="con-wago-500" library_urn="urn:adsk.eagle:library:195" deviceset="W237-102" device="" package3d_urn="urn:adsk.eagle:package:10688/1"/>
+<part name="MAIN_ARM" library="con-wago-500" library_urn="urn:adsk.eagle:library:195" deviceset="W237-102" device="" package3d_urn="urn:adsk.eagle:package:10688/1" override_package3d_urn="urn:adsk.eagle:package:42833995/2" override_package_urn="urn:adsk.eagle:footprint:10676/1"/>
 <part name="R11" library="rcl" library_urn="urn:adsk.eagle:library:334" deviceset="R-US_" device="R0805" package3d_urn="urn:adsk.eagle:package:23553/2" value="100K ohm"/>
 <part name="R12" library="rcl" library_urn="urn:adsk.eagle:library:334" deviceset="R-US_" device="R0805" package3d_urn="urn:adsk.eagle:package:23553/2" value="100K ohm"/>
@@
 <part name="H3" library="holes" library_urn="urn:adsk.eagle:library:237" deviceset="MOUNT-PAD-ROUND" device="3.0" package3d_urn="urn:adsk.eagle:package:14280/1"/>
 <part name="H4" library="holes" library_urn="urn:adsk.eagle:library:237" deviceset="MOUNT-PAD-ROUND" device="3.0" package3d_urn="urn:adsk.eagle:package:14280/1"/>
+<part name="JP2" library="pinhead" library_urn="urn:adsk.eagle:library:325" deviceset="PINHD-1X4" device="" package3d_urn="urn:adsk.eagle:package:22407/2"/>
 </parts>
 <sheets>
@@
 <attribute name="VALUE" x="29.21" y="222.758" size="1.778" layer="96"/>
 </instance>
-<instance part="DR_ARM" gate="-1" x="172.72" y="187.96" smashed="yes" rot="R180">
+<instance part="DR_ARM" gate="-1" x="172.72" y="182.88" smashed="yes" rot="R180">
+<attribute name="NAME" x="172.72" y="181.991" size="1.778" layer="95"/>
+</instance>
+<instance part="DR_ARM" gate="-2" x="172.72" y="187.96" smashed="yes" rot="R180">
+<attribute name="VALUE" x="175.26" y="191.643" size="1.778" layer="96" rot="R180"/>
 <attribute name="NAME" x="172.72" y="187.071" size="1.778" layer="95"/>
-</instance>
-<instance part="DR_ARM" gate="-2" x="172.72" y="182.88" smashed="yes" rot="R180">
-<attribute name="VALUE" x="175.26" y="186.563" size="1.778" layer="96" rot="R180"/>
-<attribute name="NAME" x="172.72" y="181.991" size="1.778" layer="95"/>
 </instance>
 <instance part="R23" gate="G$1" x="180.34" y="172.72" smashed="yes">
@@
 <attribute name="VALUE" x="110.49" y="33.782" size="1.778" layer="96" rot="R180"/>
 </instance>
-<instance part="J1" gate="G$1" x="246.38" y="243.84" smashed="yes">
+<instance part="POWER" gate="G$1" x="246.38" y="243.84" smashed="yes">
 <attribute name="NAME" x="238.76" y="247.142" size="1.778" layer="95"/>
 <attribute name="VALUE" x="238.76" y="236.22" size="1.778" layer="96"/>
 </instance>
-<instance part="DROGUE_PYRO" gate="G$1" x="137.16" y="177.8" smashed="yes">
-<attribute name="NAME" x="142.24" y="171.958" size="1.778" layer="95" rot="R180"/>
-<attribute name="VALUE" x="139.7" y="182.88" size="1.778" layer="96" rot="R180"/>
+<instance part="DROGUE_PYRO" gate="G$1" x="137.16" y="175.26" smashed="yes">
+<attribute name="NAME" x="142.24" y="169.418" size="1.778" layer="95" rot="R180"/>
+<attribute name="VALUE" x="139.7" y="180.34" size="1.778" layer="96" rot="R180"/>
 </instance>
 <instance part="R6" gate="G$1" x="208.28" y="208.28" smashed="yes" rot="R90">
@@
 <attribute name="VALUE" x="18.034" y="81.3562" size="1.778" layer="96"/>
 </instance>
+<instance part="JP2" gate="A" x="340.36" y="251.46" smashed="yes" rot="R180">
+<attribute name="NAME" x="346.71" y="243.205" size="1.778" layer="95" rot="R180"/>
+<attribute name="VALUE" x="346.71" y="259.08" size="1.778" layer="96" rot="R180"/>
+</instance>
 </instances>
 <busses>
@@
 <wire x1="251.46" y1="241.3" x2="259.08" y2="241.3" width="0.1524" layer="91"/>
 <label x="259.08" y="241.3" size="1.27" layer="95" xref="yes"/>
-<pinref part="J1" gate="G$1" pin="N"/>
+<pinref part="POWER" gate="G$1" pin="N"/>
 </segment>
 <segment>
@@
 <label x="7.62" y="78.74" size="1.27" layer="95" rot="R270" xref="yes"/>
 </segment>
+<segment>
+<pinref part="JP2" gate="A" pin="1"/>
+<wire x1="342.9" y1="246.38" x2="350.52" y2="246.38" width="0.1524" layer="91"/>
+<label x="350.52" y="246.38" size="1.27" layer="95" xref="yes"/>
+</segment>
 </net>
 <net name="VCC" class="0">
@@
 <label x="266.7" y="243.84" size="1.27" layer="95" xref="yes"/>
 <wire x1="266.7" y1="243.84" x2="251.46" y2="243.84" width="0.1524" layer="91"/>
-<pinref part="J1" gate="G$1" pin="P"/>
+<pinref part="POWER" gate="G$1" pin="P"/>
 </segment>
 <segment>
@@
 </segment>
 <segment>
-<pinref part="DR_ARM" gate="-1" pin="KL"/>
-<wire x1="167.64" y1="187.96" x2="152.4" y2="187.96" width="0.1524" layer="91"/>
-<label x="152.4" y="187.96" size="1.27" layer="95" rot="R180" xref="yes"/>
+<pinref part="DR_ARM" gate="-2" pin="KL"/>
+<wire x1="167.64" y1="187.96" x2="149.86" y2="187.96" width="0.1524" layer="91"/>
+<label x="149.86" y="187.96" size="1.27" layer="95" rot="R180" xref="yes"/>
 </segment>
 </net>
@@
 <label x="99.06" y="76.2" size="1.27" layer="95" xref="yes"/>
 </segment>
+<segment>
+<pinref part="JP2" gate="A" pin="4"/>
+<wire x1="342.9" y1="254" x2="350.52" y2="254" width="0.1524" layer="91"/>
+<label x="350.52" y="254" size="1.27" layer="95" xref="yes"/>
+</segment>
 </net>
 <net name="TX" class="0">
@@
 <pinref part="R9" gate="G$1" pin="1"/>
 <wire x1="149.86" y1="177.8" x2="152.4" y2="177.8" width="0.1524" layer="91"/>
+<pinref part="R10" gate="G$1" pin="1"/>
 <wire x1="149.86" y1="177.8" x2="149.86" y2="175.26" width="0.1524" layer="91"/>
-<pinref part="R10" gate="G$1" pin="1"/>
 <wire x1="149.86" y1="175.26" x2="149.86" y2="172.72" width="0.1524" layer="91"/>
 <wire x1="149.86" y1="172.72" x2="152.4" y2="172.72" width="0.1524" layer="91"/>
-<pinref part="DROGUE_PYRO" gate="G$1" pin="N"/>
+<pinref part="DROGUE_PYRO" gate="G$1" pin="P"/>
 <wire x1="142.24" y1="175.26" x2="149.86" y2="175.26" width="0.1524" layer="91"/>
 <junction x="149.86" y="175.26"/>
@@
 <net name="N$2" class="0">
 <segment>
-<pinref part="DROGUE_PYRO" gate="G$1" pin="P"/>
-<wire x1="142.24" y1="177.8" x2="144.78" y2="177.8" width="0.1524" layer="91"/>
-<wire x1="144.78" y1="177.8" x2="144.78" y2="182.88" width="0.1524" layer="91"/>
-<pinref part="DR_ARM" gate="-2" pin="KL"/>
+<pinref part="DR_ARM" gate="-1" pin="KL"/>
 <wire x1="144.78" y1="182.88" x2="167.64" y2="182.88" width="0.1524" layer="91"/>
+<pinref part="DROGUE_PYRO" gate="G$1" pin="N"/>
+<wire x1="142.24" y1="172.72" x2="144.78" y2="172.72" width="0.1524" layer="91"/>
+<wire x1="144.78" y1="172.72" x2="144.78" y2="182.88" width="0.1524" layer="91"/>
 </segment>
 </net>
@@
 <pinref part="U1" gate="G$1" pin="GP28"/>
 </segment>
+<segment>
+<pinref part="JP2" gate="A" pin="3"/>
+<wire x1="342.9" y1="251.46" x2="350.52" y2="251.46" width="0.1524" layer="91"/>
+<label x="350.52" y="251.46" size="1.27" layer="95" xref="yes"/>
+</segment>
 </net>
 <net name="AIR_SCK" class="0">
@@
 <label x="215.9" y="58.42" size="1.27" layer="95" xref="yes"/>
 </segment>
-</net>
+<segment>
+<pinref part="JP2" gate="A" pin="2"/>
+<wire x1="342.9" y1="248.92" x2="350.52" y2="248.92" width="0.1524" layer="91"/>
+<label x="350.52" y="248.92" size="1.27" layer="95" xref="yes"/>
+</segment>
+</net>

Commit message: uart xbee
Connections:
- removed net ATTN: U1.GP21, U2.AD1/DIO1/SPI_NATTN
- new net CTS: U1.GP21, U2.NCTS/DIO7
- new net SEX_RX: U2.DIN/NCONFIG/DIO14
- net MISO0: no longer U2.DIO12/SPI_MISO
- net MOSI0: no longer U2.DIO4/SPI_MOSI
- net SER_TX: now also U2.DOUT/DIO13
Changed lines of the file:
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@@
 <pinref part="U1" gate="G$1" pin="GP19"/>
-</segment>
-<segment>
-<pinref part="U2" gate="G$1" pin="DIO4/SPI_MOSI"/>
-<wire x1="40.64" y1="195.58" x2="33.02" y2="195.58" width="0.1524" layer="91"/>
-<label x="33.02" y="195.58" size="1.27" layer="95" rot="R180" xref="yes"/>
 </segment>
 </net>
@@
 <pinref part="R16" gate="G$1" pin="1"/>
 </segment>
-<segment>
-<pinref part="U2" gate="G$1" pin="DIO12/SPI_MISO"/>
-<wire x1="40.64" y1="205.74" x2="33.02" y2="205.74" width="0.1524" layer="91"/>
-<label x="33.02" y="205.74" size="1.27" layer="95" rot="R180" xref="yes"/>
-</segment>
 </net>
 <net name="CS_FLASH" class="0">
@@
 <label x="99.06" y="71.12" size="1.27" layer="95" xref="yes"/>
 </segment>
+<segment>
+<pinref part="U2" gate="G$1" pin="DOUT/DIO13"/>
+<wire x1="40.64" y1="210.82" x2="33.02" y2="210.82" width="0.1524" layer="91"/>
+<label x="33.02" y="210.82" size="1.016" layer="95" rot="R180" xref="yes"/>
+</segment>
 </net>
 <net name="SER_RX" class="0">
@@
 <wire x1="172.72" y1="33.02" x2="165.1" y2="33.02" width="0.1524" layer="91"/>
 <label x="165.1" y="33.02" size="1.27" layer="95" rot="R180" xref="yes"/>
-</segment>
-</net>
-<net name="ATTN" class="0">
-<segment>
-<pinref part="U2" gate="G$1" pin="AD1/DIO1/SPI_NATTN"/>
-<wire x1="40.64" y1="182.88" x2="33.02" y2="182.88" width="0.1524" layer="91"/>
-<label x="33.02" y="182.88" size="1.27" layer="95" rot="R180" xref="yes"/>
-</segment>
-<segment>
-<pinref part="U1" gate="G$1" pin="GP21"/>
-<wire x1="208.28" y1="45.72" x2="215.9" y2="45.72" width="0.1524" layer="91"/>
-<label x="215.9" y="45.72" size="1.27" layer="95" xref="yes"/>
 </segment>
 </net>
@@
 </segment>
 </net>
+<net name="SEX_RX" class="0">
+<segment>
+<pinref part="U2" gate="G$1" pin="DIN/NCONFIG/DIO14"/>
+<wire x1="40.64" y1="208.28" x2="33.02" y2="208.28" width="0.1524" layer="91"/>
+<label x="33.02" y="208.28" size="1.016" layer="95" rot="R180" xref="yes"/>
+</segment>
+</net>
+<net name="CTS" class="0">
+<segment>
+<pinref part="U2" gate="G$1" pin="NCTS/DIO7"/>
+<wire x1="40.64" y1="193.04" x2="33.02" y2="193.04" width="0.1524" layer="91"/>
+<label x="33.02" y="193.04" size="1.016" layer="95" rot="R180" xref="yes"/>
+</segment>
+<segment>
+<pinref part="U1" gate="G$1" pin="GP21"/>
+<wire x1="208.28" y1="45.72" x2="215.9" y2="45.72" width="0.1524" layer="91"/>
+<label x="215.9" y="45.72" size="1.27" layer="95" xref="yes"/>
+</segment>
+</net>
