File: Eagle files/FLYTE 2.0/FLYTE-v2.sch (EAGLE design)
At the start: 58 parts, among them U2 XBP9B-XCST-021, U3 ADS1115IDGSR, U4 H3LIS200DLTR, U5 BS170F, U6 W25Q32JVSSIQ, U7 BS170F

Commit message: .
Parts:
- removed R13, R22: 4.7K ohm, rcl:R-US_R0805
Connections:
- removed net CS_SX: R13.1, U1.GP17, U2.AD3/DIO3/SPI_NSSEL
- removed net SCK0: U1.GP18, U2.AD2/DIO2/SPI_CLK
- removed net SX_RESET: R22.2, U1.GP26, U2.!RESET
- net 3V3: no longer R13.2, R22.1
- net CTS: no longer U1.GP21
Changed lines of the file:
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@@
 <part name="C2" library="SparkFun-Capacitors" deviceset="22UF" device="-0805-6.3V-20%" override_package3d_urn="urn:adsk.eagle:package:40331879/2" override_package_urn="urn:adsk.eagle:footprint:40331880/1" value="22uF"/>
 <part name="U6" library="W25Q32JVSSIQ" deviceset="W25Q32JVSSIQ" device="" override_package3d_urn="urn:adsk.eagle:package:40381730/2" override_package_urn="urn:adsk.eagle:footprint:40381731/1"/>
-<part name="R13" library="rcl" library_urn="urn:adsk.eagle:library:334" deviceset="R-US_" device="R0805" package3d_urn="urn:adsk.eagle:package:23553/2" value="4.7K ohm"/>
 <part name="R14" library="rcl" library_urn="urn:adsk.eagle:library:334" deviceset="R-US_" device="R0805" package3d_urn="urn:adsk.eagle:package:23553/2" value="4.7K ohm"/>
 <part name="R15" library="rcl" library_urn="urn:adsk.eagle:library:334" deviceset="R-US_" device="R0805" package3d_urn="urn:adsk.eagle:package:23553/2" value="4.7K ohm"/>
@@
 <part name="S1" library="SparkFun-Switches" deviceset="MOMENTARY-SWITCH-SPST" device="-PTH-6.0MM" override_package3d_urn="urn:adsk.eagle:package:40381829/2" override_package_urn="urn:adsk.eagle:footprint:40381830/1"/>
 <part name="U2" library="XBP9B-XCST-021" deviceset="XBP9B-XCST-021" device=""/>
-<part name="R22" library="rcl" library_urn="urn:adsk.eagle:library:334" deviceset="R-US_" device="R0805" package3d_urn="urn:adsk.eagle:package:23553/2" value="4.7K ohm"/>
 <part name="DR_ARM" library="con-wago-500" library_urn="urn:adsk.eagle:library:195" deviceset="W237-102" device="" package3d_urn="urn:adsk.eagle:package:10688/1"/>
 <part name="R23" library="rcl" library_urn="urn:adsk.eagle:library:334" deviceset="R-US_" device="R0805" package3d_urn="urn:adsk.eagle:package:23553/2" value="100K ohm"/>
@@
 <attribute name="NAME" x="358.3677" y="79.525" size="1.27268125" layer="95"/>
 </instance>
-<instance part="R13" gate="G$1" x="231.14" y="35.56" smashed="yes">
-<attribute name="NAME" x="227.33" y="37.0586" size="1.778" layer="95"/>
-<attribute name="VALUE" x="227.33" y="32.258" size="1.778" layer="96"/>
-</instance>
 <instance part="R14" gate="G$1" x="149.86" y="35.56" smashed="yes">
 <attribute name="NAME" x="146.05" y="37.0586" size="1.778" layer="95"/>
@@
 <attribute name="NAME" x="45.6551" y="226.1321" size="1.2736" layer="95"/>
 <attribute name="VALUE" x="45.6561" y="175.1891" size="1.27355" layer="96"/>
-</instance>
-<instance part="R22" gate="G$1" x="33.02" y="226.06" smashed="yes">
-<attribute name="NAME" x="29.21" y="227.5586" size="1.778" layer="95"/>
-<attribute name="VALUE" x="29.21" y="222.758" size="1.778" layer="96"/>
 </instance>
 <instance part="DR_ARM" gate="-1" x="172.72" y="182.88" smashed="yes" rot="R180">
@@
 </segment>
 <segment>
-<pinref part="R13" gate="G$1" pin="2"/>
-<wire x1="236.22" y1="35.56" x2="241.3" y2="35.56" width="0.1524" layer="91"/>
-<label x="241.3" y="35.56" size="1.27" layer="95" xref="yes"/>
-</segment>
-<segment>
 <pinref part="R14" gate="G$1" pin="1"/>
 <wire x1="144.78" y1="35.56" x2="142.24" y2="35.56" width="0.1524" layer="91"/>
@@
 <label x="309.88" y="177.8" size="1.27" layer="95" rot="R180" xref="yes"/>
 <pinref part="U$4" gate="G$1" pin="VIN"/>
-</segment>
-<segment>
-<pinref part="R22" gate="G$1" pin="1"/>
-<wire x1="27.94" y1="226.06" x2="25.4" y2="226.06" width="0.1524" layer="91"/>
-<label x="25.4" y="226.06" size="1.27" layer="95" rot="R180" xref="yes"/>
 </segment>
 <segment>
@@
 </segment>
 </net>
-<net name="CS_SX" class="0">
-<segment>
-<wire x1="208.28" y1="33.02" x2="213.36" y2="33.02" width="0.1524" layer="91"/>
-<label x="215.9" y="33.02" size="1.27" layer="95" xref="yes"/>
-<pinref part="U1" gate="G$1" pin="GP17"/>
-<wire x1="213.36" y1="33.02" x2="215.9" y2="33.02" width="0.1524" layer="91"/>
-<wire x1="213.36" y1="33.02" x2="213.36" y2="35.56" width="0.1524" layer="91"/>
-<junction x="213.36" y="33.02"/>
-<wire x1="213.36" y1="35.56" x2="226.06" y2="35.56" width="0.1524" layer="91"/>
-<pinref part="R13" gate="G$1" pin="1"/>
-</segment>
-<segment>
-<pinref part="U2" gate="G$1" pin="AD3/DIO3/SPI_NSSEL"/>
-<wire x1="40.64" y1="187.96" x2="33.02" y2="187.96" width="0.1524" layer="91"/>
-<label x="33.02" y="187.96" size="1.27" layer="95" rot="R180" xref="yes"/>
-</segment>
-</net>
 <net name="CS_SD" class="0">
 <segment>
@@
 <wire x1="167.64" y1="35.56" x2="154.94" y2="35.56" width="0.1524" layer="91"/>
 <pinref part="R14" gate="G$1" pin="2"/>
-</segment>
-</net>
-<net name="SX_RESET" class="0">
-<segment>
-<pinref part="U1" gate="G$1" pin="GP26"/>
-<wire x1="208.28" y1="55.88" x2="215.9" y2="55.88" width="0.1524" layer="91"/>
-<label x="215.9" y="55.88" size="1.27" layer="95" xref="yes"/>
-</segment>
-<segment>
-<pinref part="U2" gate="G$1" pin="!RESET"/>
-<wire x1="40.64" y1="218.44" x2="38.1" y2="218.44" width="0.1524" layer="91"/>
-<label x="33.02" y="218.44" size="1.27" layer="95" rot="R180" xref="yes"/>
-<wire x1="38.1" y1="218.44" x2="33.02" y2="218.44" width="0.1524" layer="91"/>
-<wire x1="38.1" y1="218.44" x2="38.1" y2="226.06" width="0.1524" layer="91"/>
-<junction x="38.1" y="218.44"/>
-<pinref part="R22" gate="G$1" pin="2"/>
 </segment>
 </net>
@@
 </segment>
 </net>
-<net name="SCK0" class="0">
-<segment>
-<wire x1="208.28" y1="38.1" x2="215.9" y2="38.1" width="0.1524" layer="91"/>
-<label x="215.9" y="38.1" size="1.27" layer="95" xref="yes"/>
-<pinref part="U1" gate="G$1" pin="GP18"/>
-</segment>
-<segment>
-<pinref part="U2" gate="G$1" pin="AD2/DIO2/SPI_CLK"/>
-<wire x1="40.64" y1="185.42" x2="33.02" y2="185.42" width="0.1524" layer="91"/>
-<label x="33.02" y="185.42" size="1.27" layer="95" rot="R180" xref="yes"/>
-</segment>
-</net>
 <net name="MISO0" class="0">
 <segment>
@@
 <label x="33.02" y="193.04" size="1.016" layer="95" rot="R180" xref="yes"/>
 </segment>
-<segment>
-<pinref part="U1" gate="G$1" pin="GP21"/>
-<wire x1="208.28" y1="45.72" x2="215.9" y2="45.72" width="0.1524" layer="91"/>
-<label x="215.9" y="45.72" size="1.27" layer="95" xref="yes"/>
-</segment>
-</net>
+</net>

Commit message: Finish layout for v2
Parts:
- added LED1, LED2: (no value), led:LEDCHIPLED_1206
- added R13: (no value), rcl:R-US_R0805
- R16: value 100K ohm -> (none)
Connections:
- removed net MISO0: R16.1, U1.GP16
- removed net MOSI0: U1.GP19
- removed net SEX_RX: U2.DIN/NCONFIG/DIO14
- new net LED1: R13.1, U1.GP19
- new net LED2: R16.1, U1.GP18
- new net N$14: LED1.C, R13.2
- new net N$15: LED2.C, R16.2
- net 3V3: now also LED1.A, LED2.A; no longer R16.2
- net AIR_DATA: now also U1.GP16; no longer U1.GP28
- net AIR_SCK: now also U1.GP17; no longer U1.GP27
- net CTS: now also U1.GP27
- net DROGUE: now also U1.GP28; no longer U1.GP15
- net N$3: now also U1.GP26; no longer U1.GP22
- net SER_RX: now also U2.DIN/NCONFIG/DIO14
Other:
- moved on the sheet: R16, S2
