File: Eagle files/FLYTE 2.0/FLYTE-v2.sch (EAGLE design)
At the start: 59 parts, among them U2 XBP9B-XCST-021, U3 ADS1115IDGSR, U4 H3LIS200DLTR, U5 BS170F, U6 W25Q32JVSSIQ, U7 BS170F

Commit message: .
Parts:
- added JP3: (no value), adafruit:PINHD-1X3
Connections:
- new net 20: JP3.1, U1.GP15
- new net 21: JP3.2, U1.GP21
- new net 22: JP3.3, U1.GP22
Changed lines of the file:
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@@
 <part name="R13" library="rcl" library_urn="urn:adsk.eagle:library:334" deviceset="R-US_" device="R0805" package3d_urn="urn:adsk.eagle:package:23553/2"/>
 <part name="R16" library="rcl" library_urn="urn:adsk.eagle:library:334" deviceset="R-US_" device="R0805" package3d_urn="urn:adsk.eagle:package:23553/2"/>
+<part name="JP3" library="adafruit" library_urn="urn:adsk.eagle:library:420" deviceset="PINHD-1X3" device="" package3d_urn="urn:adsk.eagle:package:6240710/1"/>
 </parts>
 <sheets>
@@
 <attribute name="VALUE" x="259.842" y="21.59" size="1.778" layer="96" rot="R90"/>
 </instance>
+<instance part="JP3" gate="A" x="284.48" y="48.26" smashed="yes">
+<attribute name="NAME" x="278.13" y="53.975" size="1.778" layer="95"/>
+<attribute name="VALUE" x="278.13" y="40.64" size="1.778" layer="96"/>
+</instance>
 </instances>
 <busses>
@@
 </segment>
 </net>
+<net name="22" class="0">
+<segment>
+<pinref part="U1" gate="G$1" pin="GP22"/>
+<wire x1="208.28" y1="50.8" x2="215.9" y2="50.8" width="0.1524" layer="91"/>
+<label x="215.9" y="50.8" size="1.778" layer="95" xref="yes"/>
+</segment>
+<segment>
+<pinref part="JP3" gate="A" pin="3"/>
+<wire x1="281.94" y1="45.72" x2="271.78" y2="45.72" width="0.1524" layer="91"/>
+<label x="271.78" y="45.72" size="1.778" layer="95" rot="R180" xref="yes"/>
+</segment>
+</net>
+<net name="21" class="0">
+<segment>
+<pinref part="U1" gate="G$1" pin="GP21"/>
+<wire x1="208.28" y1="45.72" x2="215.9" y2="45.72" width="0.1524" layer="91"/>
+<label x="215.9" y="45.72" size="1.778" layer="95" xref="yes"/>
+</segment>
+<segment>
+<pinref part="JP3" gate="A" pin="2"/>
+<wire x1="281.94" y1="48.26" x2="271.78" y2="48.26" width="0.1524" layer="91"/>
+<label x="271.78" y="48.26" size="1.778" layer="95" rot="R180" xref="yes"/>
+</segment>
+</net>
+<net name="20" class="0">
+<segment>
+<pinref part="U1" gate="G$1" pin="GP15"/>
+<wire x1="172.72" y1="30.48" x2="165.1" y2="30.48" width="0.1524" layer="91"/>
+<label x="165.1" y="30.48" size="1.778" layer="95" rot="R180" xref="yes"/>
+</segment>
+<segment>
+<pinref part="JP3" gate="A" pin="1"/>
+<wire x1="281.94" y1="50.8" x2="271.78" y2="50.8" width="0.1524" layer="91"/>
+<label x="271.78" y="50.8" size="1.778" layer="95" rot="R180" xref="yes"/>
+</segment>
+</net>
