File: Eagle files/FLYTE 2.0/FLYTE-v2.sch (EAGLE design)
At the start: 60 parts, among them U3 ADS1115IDGSR, U4 H3LIS200DLTR, U5 BS170F, U6 W25Q32JVSSIQ, U7 BS170F

Commit message: minor changes
Parts:
- JP3: device adafruit:PINHD-1X3 -> pinhead:PINHD-1X4
Connections:
- net GND: now also JP3.4
Changed lines of the file:
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@@
 <part name="R13" library="rcl" library_urn="urn:adsk.eagle:library:334" deviceset="R-US_" device="R0805" package3d_urn="urn:adsk.eagle:package:23553/2"/>
 <part name="R16" library="rcl" library_urn="urn:adsk.eagle:library:334" deviceset="R-US_" device="R0805" package3d_urn="urn:adsk.eagle:package:23553/2"/>
-<part name="JP3" library="adafruit" library_urn="urn:adsk.eagle:library:420" deviceset="PINHD-1X3" device="" package3d_urn="urn:adsk.eagle:package:6240710/1"/>
+<part name="JP3" library="pinhead" library_urn="urn:adsk.eagle:library:325" deviceset="PINHD-1X4" device="" package3d_urn="urn:adsk.eagle:package:22407/2"/>
 </parts>
 <sheets>
@@
 <label x="350.52" y="246.38" size="1.27" layer="95" xref="yes"/>
 </segment>
+<segment>
+<pinref part="JP3" gate="A" pin="4"/>
+<wire x1="281.94" y1="45.72" x2="271.78" y2="45.72" width="0.1524" layer="91"/>
+<label x="271.78" y="45.72" size="1.27" layer="95" rot="R180" xref="yes"/>
+</segment>
 </net>
 <net name="VCC" class="0">
@@
 <pinref part="U1" gate="G$1" pin="GP22"/>
 <wire x1="208.28" y1="50.8" x2="215.9" y2="50.8" width="0.1524" layer="91"/>
-<label x="215.9" y="50.8" size="1.778" layer="95" xref="yes"/>
+<label x="215.9" y="50.8" size="1.27" layer="95" xref="yes"/>
 </segment>
 <segment>
 <pinref part="JP3" gate="A" pin="3"/>
-<wire x1="281.94" y1="45.72" x2="271.78" y2="45.72" width="0.1524" layer="91"/>
-<label x="271.78" y="45.72" size="1.778" layer="95" rot="R180" xref="yes"/>
+<wire x1="281.94" y1="48.26" x2="271.78" y2="48.26" width="0.1524" layer="91"/>
+<label x="271.78" y="48.26" size="1.27" layer="95" rot="R180" xref="yes"/>
 </segment>
 </net>
@@
 <pinref part="U1" gate="G$1" pin="GP21"/>
 <wire x1="208.28" y1="45.72" x2="215.9" y2="45.72" width="0.1524" layer="91"/>
-<label x="215.9" y="45.72" size="1.778" layer="95" xref="yes"/>
+<label x="215.9" y="45.72" size="1.27" layer="95" xref="yes"/>
 </segment>
 <segment>
 <pinref part="JP3" gate="A" pin="2"/>
-<wire x1="281.94" y1="48.26" x2="271.78" y2="48.26" width="0.1524" layer="91"/>
-<label x="271.78" y="48.26" size="1.778" layer="95" rot="R180" xref="yes"/>
+<wire x1="281.94" y1="50.8" x2="271.78" y2="50.8" width="0.1524" layer="91"/>
+<label x="271.78" y="50.8" size="1.27" layer="95" rot="R180" xref="yes"/>
 </segment>
 </net>
@@
 <pinref part="U1" gate="G$1" pin="GP15"/>
 <wire x1="172.72" y1="30.48" x2="165.1" y2="30.48" width="0.1524" layer="91"/>
-<label x="165.1" y="30.48" size="1.778" layer="95" rot="R180" xref="yes"/>
+<label x="165.1" y="30.48" size="1.27" layer="95" rot="R180" xref="yes"/>
 </segment>
 <segment>
 <pinref part="JP3" gate="A" pin="1"/>
-<wire x1="281.94" y1="50.8" x2="271.78" y2="50.8" width="0.1524" layer="91"/>
-<label x="271.78" y="50.8" size="1.778" layer="95" rot="R180" xref="yes"/>
-</segment>
-</net>
+<wire x1="281.94" y1="53.34" x2="271.78" y2="53.34" width="0.1524" layer="91"/>
+<label x="271.78" y="53.34" size="1.27" layer="95" rot="R180" xref="yes"/>
+</segment>
+</net>

Commit message: idk
Parts:
- removed R14: 4.7K ohm, rcl:R-US_R0805
- removed U$3: SDREADER, SDREADER:SDREADER
- added C8: 100 nF, SparkFun-Capacitors:22UF-0805-6.3V-20%
- added D2: 1N4004, diode:1N4004
- added U2: W25Q32JVSSIQ, W25Q32JVSSIQ:W25Q32JVSSIQ
Connections:
- removed net CS_SD: R14.2, U$3.CS, U1.GP13
- net 3V3: now also C8.2, D2.C, U2.!HOLD!/!RESET!(IO3), U2.!WP!(IO2), U2.VCC; no longer R14.1, U$3.VCC
- net CS_FLASH: now also U2.!CS
- net GND: now also C8.1, U2.GND; no longer U$3.GND, U$4.RST
- net MISO1: now also U2.DO(IO1); no longer U$3.MISO
- net MOSI1: now also U2.DI(IO0); no longer U$3.MOSI
- net RX: now also U1.GP8; no longer U1.GP9
- net SCK1: now also U2.CLK; no longer U$3.CLK
- net SER_RX: now also U1.GP0; no longer U1.GP1
- net SER_TX: now also U1.GP1; no longer U1.GP0
- net TX: now also U1.GP9; no longer U1.GP8
- net VCC: now also D2.A
