File: Eagle files/FLYTE 2.0/FLYTE-v2.brd (EAGLE design)
At the start: 116 x 55 mm, 59 parts, among them U2 XBP9B-XCST-021, U3 ADS1115IDGSR, U4 H3LIS200DLTR, U5 BS170F, U6 W25Q32JVSSIQ, U7 BS170F

Commit message: Thoda aur
Routing:
- net 3V3: track 343.0 -> 341.9 mm
Changed lines of the file:
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@@
 <setting verticaltext="up"/>
 </settings>
-<grid distance="1" unitdist="mil" unit="mil" style="lines" multiple="1" display="no" altdistance="1" altunitdist="mil" altunit="mil"/>
+<grid distance="1" unitdist="mil" unit="mm" style="lines" multiple="1" display="no" altdistance="1" altunitdist="mil" altunit="mm"/>
 <layers>
 <layer number="1" name="Top" color="4" fill="1" visible="yes" active="yes"/>
@@
 <wire x1="34.72" y1="36.345" x2="38.172" y2="32.893" width="0.4064" layer="16"/>
 <wire x1="38.172" y1="32.893" x2="43.1546" y2="32.893" width="0.4064" layer="16"/>
-<wire x1="87.9701" y1="46.31605" x2="87.54025" y2="46.7459" width="0.4064" layer="16"/>
-<wire x1="87.9701" y1="38.9761" x2="88.347" y2="38.5992" width="0.4064" layer="16"/>
-<wire x1="87.9701" y1="46.31605" x2="87.9701" y2="38.9761" width="0.4064" layer="16"/>
+<wire x1="88.3003" y1="44.13165" x2="85.68605" y2="46.7459" width="0.4064" layer="16"/>
+<wire x1="88.3003" y1="38.6459" x2="88.347" y2="38.5992" width="0.4064" layer="16"/>
+<wire x1="88.3003" y1="44.13165" x2="88.3003" y2="38.6459" width="0.4064" layer="16"/>
 <wire x1="89.0412" y1="43.70130625" x2="89.0412" y2="43.7042" width="0.4064" layer="1"/>
 <wire x1="89.0412" y1="43.7042" x2="89.9356" y2="44.5986" width="0.4064" layer="1"/>
@@
 <wire x1="86.1568" y1="21.0862" x2="87.9094" y2="22.8388" width="0.4064" layer="16"/>
 <wire x1="75.1029" y1="46.7459" x2="75" y2="46.643" width="0.4064" layer="16"/>
-<wire x1="87.54025" y1="46.7459" x2="75.1029" y2="46.7459" width="0.4064" layer="16"/>
+<wire x1="85.68605" y1="46.7459" x2="75.1029" y2="46.7459" width="0.4064" layer="16"/>
 <wire x1="77.4224" y1="23.129" x2="77.4224" y2="22.0948" width="0.254" layer="16"/>
 <wire x1="77.4224" y1="22.0948" x2="77.6224" y2="21.8948" width="0.254" layer="16"/>

Commit message: .
Parts:
- added JP3: (no value), adafruit:1X03
Connections:
- new net 20: JP3.1, U1.P$20
- new net 21: JP3.2, U1.P$27
- new net 22: JP3.3, U1.P$29
Changed lines of the file:
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@@
 <attribute name="VALUE" x="56.0832" y="7.6454" size="1.27" layer="27"/>
+</element>
+<element name="JP3" library="adafruit" library_urn="urn:adsk.eagle:library:420" package="1X03" package3d_urn="urn:adsk.eagle:package:6240710/1" value="" x="3.175" y="-8.89" smashed="yes">
+<attribute name="NAME" x="-0.7112" y="-7.0612" size="1.27" layer="25" ratio="10"/>
+<attribute name="VALUE" x="-0.635" y="-12.065" size="1.27" layer="27"/>
 </element>
 </elements>
@@
 <wire x1="60.5054" y1="10.1854" x2="60.5308" y2="10.16" width="0.254" layer="1"/>
 </signal>
+<signal name="22">
+<contactref element="U1" pad="P$29"/>
+<contactref element="JP3" pad="3"/>
+<wire x1="5.715" y1="-8.89" x2="50.96" y2="22.86" width="0" layer="19" extent="16-16"/>
+</signal>
+<signal name="21">
+<contactref element="U1" pad="P$27"/>
+<contactref element="JP3" pad="2"/>
+<wire x1="3.175" y1="-8.89" x2="50.96" y2="17.78" width="0" layer="19" extent="16-16"/>
+</signal>
+<signal name="20">
+<contactref element="U1" pad="P$20"/>
+<contactref element="JP3" pad="1"/>
+<wire x1="0.635" y1="-8.89" x2="70.96" y2="2.54" width="0" layer="19" extent="16-16"/>
+</signal>
 </signals>
