File: Eagle files/FLYTE 2.0/FLYTE-v2.brd (EAGLE design)
At the start: 116 x 55 mm, 60 parts, among them U3 ADS1115IDGSR, U4 H3LIS200DLTR, U5 BS170F, U6 W25Q32JVSSIQ, U7 BS170F

Commit message: minor changes
Parts:
- JP3: device adafruit:1X03 -> pinhead:1X04
- moved JP3 44.4 mm to (39.0, 17.3), turned to 90 degrees
- moved XBEE 3.91 mm to (24.1, 11.5)
Connections:
- net GND: now also JP3.4
Routing:
- net 20: track 0.00 -> 44.6 mm, vias 0 -> 2
- net 22: track 0.00 -> 14.7 mm, vias 0 -> 1
- net 21: track 0.00 -> 12.6 mm, vias 0 -> 1
- net 3V3: track 342.0 -> 349.8 mm
- net SER_TX: track 84.4 -> 88.3 mm
- net SER_RX: track 70.6 -> 74.5 mm
- net CTS: track 48.0 -> 51.6 mm
Other:
- board text added: "20"
- board text added: "21"
- board text added: "22"
- board text added: "G"
- board text added: "INT"
- board text removed: "INTERFACE"

Commit message: Minor changes
Parts:
- moved POWER 1.24 mm to (33.0, 51.8)
- moved DROGUE_PYRO 1.17 mm to (3.17, 36.9)
- moved R10 1.13 mm to (16.3, 38.2)
- moved R23 1.13 mm to (17.0, 41.7)
- moved R9 1.13 mm to (19.3, 38.2)
- moved U5 1.13 mm to (17.5, 37.8)
- moved MAIN_PYRO 1.09 mm to (112.9, 37.0)
- moved DR_ARM 0.94 mm to (15.5, 51.1)
- moved MAIN_ARM 0.94 mm to (100.5, 51.1)
- moved R1 0.88 mm to (21.3, 37.3)
- moved R25 0.88 mm to (21.7, 41.7)
- moved GPS 0.15 mm to (71.0, 53.3)
- moved MOTOR 0.15 mm to (87.0, 53.3)
- moved SERIAL 0.15 mm to (55.0, 53.3)
Routing:
- net N$2: track 11.8 -> 10.4 mm
- net N$6: track 11.6 -> 10.3 mm
- net SENSE_DROG: track 71.5 -> 70.4 mm
- net DROGUE: track 40.4 -> 39.3 mm
- net N$4: track 7.75 -> 6.66 mm
- net VCC: track 121.6 -> 120.8 mm
Other:
- board text added: "+"
- board text added: "-"

Commit message: Minor changes
Parts:
- moved R7 1.27 mm to (98.8, 38.6)
- moved R10 0.89 mm to (17.2, 38.2)
- moved R9 0.69 mm to (19.9, 38.2)
- moved R8 0.51 mm to (96.2, 38.6)
- moved R25 0.38 mm to (22.1, 41.7)
Routing:
- net N$7: track 6.63 -> 7.31 mm
- net N$4: track 6.66 -> 7.16 mm
