File: Eagle files/FLYTE 2.0/motor_controller_1.0.brd (EAGLE design)
At the start: 160 x 100 mm, 21 parts, among them J1 XT60PW-F

Commit message: .
Parts:
- moved H3 137.6 mm to (61.0, 5.08)
- moved JP4 132.4 mm to (61.0, 16.5), turned to 90 degrees
- moved JP3 120.4 mm to (61.0, 25.4), turned to 90 degrees
- moved D1 117.4 mm to (45.7, 27.9)
- moved D2 117.0 mm to (47.0, 38.1)
- moved JP2 108.6 mm to (61.0, 34.3), turned to 90 degrees
- moved J1 103.8 mm to (48.4, 58.8)
- moved JP1 96.9 mm to (61.0, 43.2), turned to 90 degrees
- moved R2 93.5 mm to (47.0, 17.8), flipped to the bottom
- moved R3 92.5 mm to (47.0, 21.6), flipped to the bottom
- moved R4 92.5 mm to (41.9, 21.6), flipped to the bottom
- moved R1 85.4 mm to (41.9, 17.8), flipped to the bottom
- moved H2 82.7 mm to (5.08, 5.08)
- moved H4 80.5 mm to (61.0, 55.9)
- moved D3 74.8 mm to (43.2, 38.1)
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Routing:
- net 5V: track 0.00 -> 107.5 mm
- net N$5: track 0.00 -> 84.4 mm, vias 0 -> 3
- net N$6: track 0.00 -> 62.0 mm, vias 0 -> 3
- net N$4: track 0.00 -> 46.3 mm
- net N$1: track 0.00 -> 38.1 mm
- net SERVO1: track 0.00 -> 36.3 mm, vias 0 -> 2
- net SERVO2: track 0.00 -> 33.3 mm, vias 0 -> 2
- net SCL0: track 0.00 -> 30.1 mm
- net SERVO4: track 0.00 -> 28.9 mm, vias 0 -> 3
- net SDA0: track 0.00 -> 27.8 mm
- net SERVO3: track 0.00 -> 27.7 mm, vias 0 -> 2
- net N$7: track 0.00 -> 16.8 mm, vias 0 -> 1
- net N$8: track 0.00 -> 16.2 mm, vias 0 -> 1
- net N$2: track 0.00 -> 14.0 mm
- net SER_RX: track 0.00 -> 12.0 mm
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- added copper zone on layer 1, net GND
- added copper zone on layer 16, net GND
Other:
- board size 160 x 100 mm -> 66 x 61.9 mm
- board text added: "5v"
- board text added: "GND"
