File: Eagle files/FLYTE 2.0/layout version/FLYTE-v2.brd (EAGLE design)
At the start: 116 x 55 mm, 58 parts, among them U2 XBP9B-XCST-021, U3 ADS1115IDGSR, U4 H3LIS200DLTR, U5 BS170F, U6 W25Q32JVSSIQ, U7 BS170F

Commit message: layout done
Parts:
- removed R13, R22: 4.7K ohm, rcl:R0805
- moved S2 0.26 mm to (45.1, 15.7), flipped to the bottom
Connections:
- removed net ATTN: U1.P$27, U2.19
- removed net CS_SX: R13.1, U1.P$22, U2.17
- removed net SCK0: U1.P$24, U2.18
- removed net SX_RESET: R22.2, U1.P$31, U2.5
- new net CTS: U2.12
- new net SEX_RX: U2.3
- net 3V3: no longer R13.2, R22.1
- net MISO0: no longer U2.4
- net MOSI0: no longer U2.11
- net SER_TX: now also U2.2
Routing:
- net GND: track 497.4 -> 136.9 mm, vias 15 -> 13
- net 3V3: track 415.3 -> 314.7 mm, vias 4 -> 5
- net MAIN: track 163.7 -> 65.7 mm, vias 3 -> 2
- net SER_TX: track 21.5 -> 79.4 mm, vias 1 -> 2
- net SENSE_MAIN: track 63.2 -> 35.9 mm, vias 4 -> 2
- net TX: track 52.0 -> 27.9 mm, vias 4 -> 1
- net VCC: track 159.6 -> 139.5 mm, vias 2 -> 5
- net N$3: track 5.51 -> 23.1 mm, vias 0 -> 1
- net SENSE_DROG: track 79.3 -> 70.4 mm
- net SCL0: track 30.4 -> 39.0 mm, vias 3 -> 1
- net SDA0: track 23.7 -> 29.0 mm
- net CS_SX: track 4.82 -> 0.00 mm
- net SCL1: track 38.8 -> 34.0 mm
- net N$8: track 5.91 -> 9.52 mm, vias 0 -> 1
- net N$5: track 10.2 -> 13.8 mm
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