File: Eagle files/FLYTE 2.0/reefing/reefingBrd.brd (EAGLE design)
At the start: 40 x 80 mm, 19 parts, among them U1 RASPBERRY_PICOSMD, U2 GY-521MPU6050, U7 BS170F

Commit message: .
Parts:
- moved MAIN_ARM 4.37 mm to (19.8, 75.7)
- renumbered MAIN_PYRO to PYRO
Routing:
- net VCC: track 41.5 -> 46.0 mm
- net N$6: track 9.22 -> 11.4 mm
Other:
- board text added: "+ MAIN ARM -"
- board text added: "C:/Users/ASUS/Desktop/FLYTE/Bitmaps/RT logo.bmp"
- board text added: "REEFING BOARD"
