File: Payload/Payload.sch (EAGLE design)
At the start: 18 parts, among them CON1 XT30UPB-M

Commit message: payload sch 408 mc board
Parts:
- removed BATTERY_REGULATOR3V3: AMS1117-3.3, AMS1117-3.3:AMS1117-3.3
- removed U$2: VCNL4040, VCNL4040:VCNL4040
- added U$4: LTR390, LTR390:LTR390
- added U2: AMS1117-5.0, AMS1117-5.0:AMS1117-5.0
- U$1: value LM398LIB -> VCNL4040; device LTR390symbol:LM398LIB -> VCNL4040:VCNL4040
Connections:
- new net 5V: C1.2, D1.A, U$5.5, U$6.1, U2.VOUT
- net 3V3: now also U$4.3V3, U1.3V3(OUT); no longer BATTERY_REGULATOR3V3.VOUT, C1.2, D1.A, U$2.VCC
- net GND: now also U$4.GND, U2.GND/ADJ; no longer BATTERY_REGULATOR3V3.ADJ/GND, U$2.GND
- net N$1: now also U1.VBUS; no longer U1.VSYS
- net SCL0: now also U$1.SCL; no longer U$2.SCL
- net SCL1: now also U$4.SCL; no longer U$1.SCL
- net SDA0: now also U$1.SDA; no longer U$2.SDA
- net SDA1: now also U$4.SDA; no longer U$1.SDA
- net VCC: now also U2.VIN; no longer BATTERY_REGULATOR3V3.VIN, U$5.5, U$6.1
Other:
- moved on the sheet: CON1, D1

Commit message: payload. yet to be verified
Parts:
- removed CON1: XT30UPB-M, amass:XT30UPB-M
- removed LS1: KPEG106-HS, KPEG106-HS:KPEG106-HS
- added J1: XT60-M, XT60-M:XT60-M
- added LS2: BUZZER-PTH, SparkFun-Electromechanical:BUZZER-PTH
- added R5, R6: 330 ohm, rcl:R-US_R0805
- added R8: 100k ohm, rcl:R-US_R0805
- added R9: 301k ohm, rcl:R-US_R0805
- C1, C2: value 22uF -> 10 uF; device SparkFun-Capacitors:22UF-0805-6.3V-20% -> microbuilder:CAP_TANTALUMA/3216_WAVE
- U2: value AMS1117-5.0 -> MIC29302WU-TRTO-263-5_MCH-M; device AMS1117-5.0:AMS1117-5.0 -> MIC29302WU:MIC29302WU-TRTO-263-5_MCH-M
Connections:
- removed net N$2: LS1.POS, U1.GP6
- removed net VCC: C2.2, CON1.+, U2.VIN
- new net 7.4V: C1.+, J1.POS, U2.EN, U2.IN
- new net BUZZER: LS2.1, U1.GP6
- new net N$14: R8.1, R9.1, U2.ADJ
- new net N$5: LED1.A, R5.2
- new net N$6: R6.1, U1.GP20
- net 3V3: now also U$4.VIN; no longer U$4.3V3
- net 5V: now also C2.+, R9.2, U2.OUT; no longer C1.2, U2.VOUT
- net GND: now also C1.-, C2.-, J1.NEG, LS2.2, R8.2, U2.6, U2.GND; no longer C1.1, C2.1, CON1.-, LS1.NEG, U2.GND/ADJ
- net N$1: now also U1.VSYS; no longer U1.VBUS
- net N$3: now also R5.1; no longer LED1.A
- net N$4: now also R6.2; no longer U1.GP20
- net RX: now also U$5.1; no longer U$5.2
- net TX: now also U$5.2; no longer U$5.1
Other:
- moved on the sheet: D1, LED1, LED2
