File: Eagle files/FLYTE 2.1/FLYTE-v2_1.brd (EAGLE design)
At the start: 116 x 55 mm, 68 parts, among them Q1 IRF540NPBF, Q2 IRF540NPBF, U3 ADS1115IDGSR, U4 H3LIS200DLTR, U6 W25Q32JVSSIQ

Commit message: motor controller re design
Parts:
- removed C6: 10 uF, SparkFun-Capacitors:0805
- removed C7: 100 nF, SparkFun-Capacitors:0805
- removed U4: H3LIS200DLTR, H3LIS200DLTR:PQFN50P300X300X100-16N
- added U$2: KX134-BREAKOUT, KX134_Breakout:KX134-BREAKOUT
Connections:
- new net CS_KX134: U$2.!CS
- new net INT1_KX134: U$2.INT1
- new net INT2_KX134: U$2.INT2
- new net TRIG_KX134: U$2.TRIG
- net 3V3: now also U$2.3V3; no longer C6.1, C7.1, U4.1, U4.14, U4.15
- net GND: now also U$2.ADDR, U$2.GND; no longer C6.2, C7.2, U4.10, U4.12, U4.13, U4.16, U4.5, U4.7
- net SCL1: now also U$2.SCL; no longer U4.4
- net SDA1: now also U$2.SDA; no longer U4.6

Commit message: Schematics of FC and motor controller
Parts:
- moved C9 6.84 mm to (104.1, 7.62), turned to 0 degrees
Changed lines of the file:
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@@
 <attribute name="VALUE" x="101.219" y="10.16" size="0.6096" layer="28" font="vector" ratio="20" rot="MR270" align="top-center"/>
 </element>
-<element name="C9" library="SparkFun-Capacitors" package="0805" override_package3d_urn="urn:adsk.eagle:package:40331879/2" override_package_urn="urn:adsk.eagle:footprint:40331880/1" value="10 uF" x="97.79" y="10.16" smashed="yes" rot="MR270">
-<attribute name="NAME" x="96.901" y="10.16" size="0.6096" layer="26" font="vector" ratio="20" rot="MR270" align="bottom-center"/>
-<attribute name="PROD_ID" value="CAP-08402" x="222.25" y="-72.39" size="1.778" layer="28" rot="MR270" display="off"/>
-<attribute name="VALUE" x="98.679" y="10.16" size="0.6096" layer="28" font="vector" ratio="20" rot="MR270" align="top-center"/>
+<element name="C9" library="SparkFun-Capacitors" package="0805" override_package3d_urn="urn:adsk.eagle:package:40331879/2" override_package_urn="urn:adsk.eagle:footprint:40331880/1" value="10 uF" x="104.14" y="7.62" smashed="yes" rot="MR0">
+<attribute name="NAME" x="104.14" y="8.509" size="0.6096" layer="26" font="vector" ratio="20" rot="MR0" align="bottom-center"/>
+<attribute name="PROD_ID" value="CAP-08402" x="21.59" y="-116.84" size="1.778" layer="28" rot="MR0" display="off"/>
+<attribute name="VALUE" x="104.14" y="6.731" size="0.6096" layer="28" font="vector" ratio="20" rot="MR0" align="top-center"/>
 </element>
 <element name="D1" library="diode" library_urn="urn:adsk.eagle:library:210" package="DO41-10" package3d_urn="urn:adsk.eagle:package:43336/1" override_package3d_urn="urn:adsk.eagle:package:40381849/2" override_package_urn="urn:adsk.eagle:footprint:43094/1" value="1N4004" x="62.23" y="41.91" smashed="yes" rot="R270">
@@
 <wire x1="90.01" y1="21.59" x2="94.98" y2="24.13" width="0" layer="19" extent="16-16"/>
 <wire x1="94.98" y1="13.97" x2="90.01" y2="21.59" width="0" layer="19" extent="16-16"/>
-<wire x1="97.79" y1="11.06" x2="94.98" y2="13.97" width="0" layer="19" extent="16-16"/>
-<wire x1="100.33" y1="11.06" x2="97.79" y2="11.06" width="0" layer="19" extent="16-16"/>
-<wire x1="93.98" y1="5.08" x2="97.79" y2="11.06" width="0" layer="19" extent="16-16"/>
+<wire x1="105.04" y1="7.62" x2="94.98" y2="13.97" width="0" layer="19" extent="16-16"/>
+<wire x1="100.33" y1="11.06" x2="105.04" y2="7.62" width="0" layer="19" extent="16-16"/>
+<wire x1="93.98" y1="5.08" x2="105.04" y2="7.62" width="0" layer="19" extent="16-16"/>
 <wire x1="90.01" y1="8.89" x2="93.98" y2="5.08" width="0" layer="19" extent="16-16"/>
 <wire x1="83.82" y1="9.84" x2="90.01" y2="8.89" width="0" layer="19" extent="1-16"/>
@@
 <wire x1="103.505" y1="10.37" x2="104.775" y2="10.37" width="0" layer="19" extent="16-16"/>
 <wire x1="100.33" y1="9.26" x2="103.505" y2="10.37" width="0" layer="19" extent="16-16"/>
-<wire x1="97.79" y1="9.26" x2="100.33" y2="9.26" width="0" layer="19" extent="16-16"/>
-<wire x1="94.93" y1="8.89" x2="97.79" y2="9.26" width="0" layer="19" extent="16-16"/>
+<wire x1="103.24" y1="7.62" x2="100.33" y2="9.26" width="0" layer="19" extent="16-16"/>
+<wire x1="94.93" y1="8.89" x2="103.24" y2="7.62" width="0" layer="19" extent="16-16"/>
 <wire x1="94.93" y1="11.43" x2="94.93" y2="8.89" width="0" layer="19" extent="16-16"/>
 <wire x1="101.6" y1="5.08" x2="100.33" y2="9.26" width="0" layer="19" extent="16-16"/>

Commit message: Schem of fc and mc
Parts:
- removed DROGUE_PYRO, MAIN_PYRO: XT30UPB-M, XT30UPB-M:XT30UPB-M
- removed R10, R8: 10 ohm, rcl:0207/10
- added DROGUE, MAIN: XT30UPB-M, XT30UPB-M:XT30UPB-M
- moved U$2 71.3 mm to (67.3, 0.25), turned to 90 degrees
- moved U$4 46.8 mm to (21.7, 27.3), turned to 0 degrees
- moved H2 32.3 mm to (37.3, 5.00)
- moved JP3 29.5 mm to (37.0, 17.8), turned to 270 degrees
- moved LS1 15.3 mm to (57.8, 33.5), turned to 180 degrees
- moved C5 10.8 mm to (54.0, 15.9)
- moved C10 10.0 mm to (57.0, 13.0)
- moved U3 9.93 mm to (52.7, 13.0)
- moved Q1 9.02 mm to (12.6, 37.0)
- moved R1 9.02 mm to (12.6, 42.0)
- moved R11 8.98 mm to (111.8, 30.5), turned to 0 degrees
- moved R23 8.44 mm to (4.83, 29.7)
- moved R25 8.08 mm to (8.38, 28.7)
- moved D2 7.75 mm to (57.8, 45.7), turned to 0 degrees
- moved R9 7.24 mm to (8.00, 37.1)
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Connections:
- net N$11: no longer R8.2
- net N$12: no longer R10.2
- net N$2: now also DROGUE.P$2; no longer DROGUE_PYRO.P$2
- net N$4: now also MAIN.P$2; no longer MAIN_PYRO.P$2, R8.1
- net N$6: now also MAIN.P$1; no longer MAIN_PYRO.P$1
- net N$7: now also DROGUE.P$1; no longer DROGUE_PYRO.P$1, R10.1

Commit message: payload pushed
Routing:
- net N$3: track 0.00 -> 9.10 mm
Changed lines of the file:
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@@
 <drawing>
 <settings>
-<setting alwaysvectorfont="yes"/>
+<setting alwaysvectorfont="no"/>
 <setting verticaltext="up"/>
 </settings>
-<grid distance="0.127" unitdist="mm" unit="mm" style="lines" multiple="1" display="no" altdistance="5" altunitdist="mil" altunit="mm"/>
+<grid distance="1" unitdist="mil" unit="mil" style="lines" multiple="1" display="no" altdistance="0.025" altunitdist="mil" altunit="mil"/>
 <layers>
 <layer number="1" name="Top" color="4" fill="1" visible="yes" active="yes"/>
@@
 </layers>
 <board>
-<fusionsync huburn="a.YnVzaW5lc3M6aWl0YjUzNQ" projecturn="a.YnVzaW5lc3M6aWl0YjUzNSNEMjAyMjA3MjU1NDIwMjEzNzY" f3durn="urn:adsk.wipprod:dm.lineage:jQ7C4NV9RB6eI30_qBJzBA" pcbguid="8cd1458f-768b-48ed-a8b8-6d023e6b69b8" lastpulledtime="" lastsyncedchangeguid="" latestrevisionid="2a022255-9a1d-48d5-bbbf-c881e8a3bf04" lastsyncedrevisionid="2a022255-9a1d-48d5-bbbf-c881e8a3bf04" lastboardhashguid="c37a480a-631b-47b4-54b2-87c3bbc9a39c" lastpushedtime="2024-05-01T03:43:34Z" linktopcb3d="true"/>
+<fusionsync huburn="a.YnVzaW5lc3M6aWl0YjUzNQ" projecturn="a.YnVzaW5lc3M6aWl0YjUzNSNEMjAyMjA3MjU1NDIwMjEzNzY" f3durn="urn:adsk.wipprod:dm.lineage:jQ7C4NV9RB6eI30_qBJzBA" pcbguid="" lastpulledtime="" lastsyncedchangeguid="" latestrevisionid="2a022255-9a1d-48d5-bbbf-c881e8a3bf04" lastsyncedrevisionid="2a022255-9a1d-48d5-bbbf-c881e8a3bf04" lastboardhashguid="c37a480a-631b-47b4-54b2-87c3bbc9a39c" lastpushedtime="2024-05-01T03:43:34Z" linktopcb3d="false"/>
 <plain>
 <wire x1="0" y1="0" x2="116" y2="0" width="0" layer="20"/>
@@
 <contactref element="INTERFACE" pad="3"/>
 <contactref element="INTERFACE" pad="1"/>
-<wire x1="73.569" y1="43.71" x2="73.569" y2="52.81" width="0" layer="19" extent="1-1"/>
+<wire x1="73.569" y1="52.81" x2="73.569" y2="43.71" width="0.254" layer="1"/>
 <wire x1="70.01" y1="29.21" x2="73.569" y2="43.71" width="0" layer="19" extent="1-16"/>
 </signal>

Commit message: mc 1.0
Parts:
- moved C10 0.66 mm to (57.7, 12.9)
Routing:
- net 3V3: track 0.00 -> 148.4 mm
- net VCC: track 0.00 -> 94.2 mm, vias 0 -> 3
- net BNO_INT: track 0.00 -> 75.3 mm, vias 0 -> 1
- net SENSE_MAIN: track 0.00 -> 67.4 mm, vias 0 -> 4
- net GPS_TX: track 0.00 -> 59.7 mm, vias 0 -> 1
- net GPS_RX: track 0.00 -> 54.7 mm, vias 0 -> 1
- net N$8: track 0.00 -> 32.8 mm, vias 0 -> 1
- net AIR_DATA: track 0.00 -> 30.5 mm
- net AIR_SCK: track 0.00 -> 28.4 mm
- net N$3: track 9.10 -> 26.9 mm, vias 0 -> 1
- net N$6: track 0.00 -> 14.1 mm
- net SDA1: track 0.00 -> 11.8 mm
- net LED2: track 0.00 -> 10.2 mm, vias 0 -> 1
- net N$4: track 0.00 -> 9.54 mm
- net N$11: track 0.00 -> 6.69 mm
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- added copper zone on layer 1, net GND
- added copper zone on layer 16, net GND

Commit message: mc2.0
Parts:
- moved R25 2.71 mm to (6.17, 30.3)
- moved R23 2.62 mm to (2.59, 31.1)
- moved XBEE 2.11 mm to (15.1, 14.6)
Routing:
- net 3V3: track 148.4 -> 296.2 mm, vias 0 -> 7
- net TELE_TX: track 0.00 -> 76.8 mm, vias 0 -> 1
- net TELE_RX: track 0.00 -> 74.9 mm
- net SDA1: track 11.8 -> 81.4 mm, vias 0 -> 3
- net 20: track 0.00 -> 63.1 mm, vias 0 -> 1
- net SCL1: track 0.00 -> 61.8 mm, vias 0 -> 4
- net CTS: track 0.00 -> 55.7 mm, vias 0 -> 3
- net MAIN: track 3.12 -> 48.0 mm
- net SDA0: track 2.50 -> 42.3 mm, vias 0 -> 4
- net VCC: track 94.2 -> 133.0 mm, vias 3 -> 4
- net 22: track 0.00 -> 38.0 mm, vias 0 -> 2
- net 21: track 0.00 -> 35.2 mm, vias 0 -> 2
- net SCL0: track 2.57 -> 33.8 mm, vias 0 -> 2
- net BUZZER: track 0.00 -> 30.6 mm
- net MOSI1: track 0.00 -> 21.4 mm, vias 0 -> 2
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
Commit message: mc done
Routing:
- net VBUS_REG: track 10.5 -> 95.4 mm, vias 0 -> 5
- net SENSE_DROG: track 2.69 -> 67.6 mm, vias 0 -> 2
- net TELE_TX: track 76.8 -> 138.8 mm, vias 1 -> 5
- net TELE_RX: track 74.9 -> 136.5 mm, vias 0 -> 3
- net DROGUE: track 2.60 -> 62.7 mm, vias 0 -> 5
- net 3V3: track 296.2 -> 354.7 mm, vias 7 -> 13
- net SCL1: track 61.8 -> 108.6 mm, vias 4 -> 12
- net SDA1: track 81.4 -> 119.7 mm, vias 3 -> 6
- net VCC: track 133.0 -> 165.3 mm, vias 4 -> 6
- net GND: track 0.00 -> 15.6 mm, vias 0 -> 5

Commit message: flyte done
Parts:
- removed JP1: (no value), pinhead:1X02
- removed JP2: (no value), pinhead:1X04
- added RAM_AIR: (no value), pinhead:1X04
- added U$10: (no value), vcc_label:VCC0
- added U$11, U$26: (no value), vbus_label:VBUS0
- added U$12: (no value), main_label:MAIN0
- added U$13: (no value), drogue_label:DROGUE0
- added U$14: (no value), lipo_1s_label:LIPO_1S0
- added U$15, U$3: (no value), gnd_label:GND0
- added U$16: (no value), scl_label:SCL0
- added U$17: (no value), sda_label:SDA0
- added U$18, U$21: (no value), gnd_small_label:GND0
- added U$19, U$20: (no value), 3v3_small_label:3V30
- added U$22, U$23: (no value), rx_small_label:RX0
- added U$24, U$25: (no value), tx_small_label:TX0
- added U$27: (no value), flyte_label:FLYTE_V2#10
- added U$5: (no value), 3v3_label:3V30
- added U$6: (no value), 20_label:200
- added U$7: (no value), 21_label:210
- added U$8: (no value), 22_label:220
- added U$9: (no value), status_label:STATUS0
- added VBUS_CONN: (no value), pinhead:1X02
- moved R23 50.5 mm to (49.8, 49.0)
- moved LIPO_POWER 50.3 mm to (105.0, 70.1)
- moved Q2 50.2 mm to (150.2, 54.7)
- moved R17 50.2 mm to (141.1, 29.7)
- moved C10 50.2 mm to (104.5, 30.8)
- moved C3 50.2 mm to (104.0, 61.1)
- moved R15 50.2 mm to (141.1, 27.4)
- moved 3V3_LED 50.2 mm to (130.7, 21.7)
- moved C1 50.2 mm to (92.6, 61.1)
- moved C2 50.2 mm to (96.4, 61.1)
- moved C8 50.2 mm to (148.2, 29.2)
- moved D1 50.2 mm to (105.3, 59.8)
- moved D2 50.2 mm to (104.6, 63.6), flipped to the top, turned to 180 degrees
- moved D3 50.2 mm to (113.2, 64.9)
- moved DROGUE 50.2 mm to (50.3, 55.8)
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Connections:
- net 3V3: now also RAM_AIR.4; no longer JP2.4
- net AIR_DATA: now also RAM_AIR.3; no longer JP2.3
- net AIR_SCK: now also RAM_AIR.2; no longer JP2.2
- net GND: now also RAM_AIR.1; no longer JP2.1
- net VBUS: now also VBUS_CONN.1; no longer JP1.1
- net VBUS_REG: now also VBUS_CONN.2; no longer JP1.2
Routing:
- net TELE_RX: track 136.5 -> 133.6 mm
- net CTS: track 55.7 -> 56.5 mm
