File: Eagle files/FLYTE 2.1/FLYTE-v2_1.sch (EAGLE design)
At the start: 68 parts, among them Q1 IRF540NPBF, Q2 IRF540NPBF, U3 ADS1115IDGSR, U4 H3LIS200DLTR, U6 W25Q32JVSSIQ

Commit message: motor controller re design
Parts:
- removed C6: 10 uF, SparkFun-Capacitors:22UF-0805-6.3V-20%
- removed C7: 100 nF, SparkFun-Capacitors:22UF-0805-6.3V-20%
- removed U4: H3LIS200DLTR, H3LIS200DLTR:H3LIS200DLTR
- added U$2: KX134-BREAKOUT, KX134_Breakout:KX134-BREAKOUT
Connections:
- new net CS_KX134: U$2.!CS
- new net INT1_KX134: U$2.INT1
- new net INT2_KX134: U$2.INT2
- new net TRIG_KX134: U$2.TRIG
- net 3V3: now also U$2.3V3; no longer C6.1, C7.1, U4.VDD, U4.VDD_IO
- net GND: now also U$2.ADDR, U$2.GND; no longer C6.2, C7.2, U4.GND, U4.SDO/SA0
- net SCL1: now also U$2.SCL; no longer U4.SCL/SPC
- net SDA1: now also U$2.SDA; no longer U4.SDA/SDI/SDO
Changed lines of the file:
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@@
 <part name="C5" library="SparkFun-Capacitors" deviceset="22UF" device="-0805-6.3V-20%" override_package3d_urn="urn:adsk.eagle:package:40331879/2" override_package_urn="urn:adsk.eagle:footprint:40331880/1" value="100 nF"/>
 <part name="U$4" library="BNO055" deviceset="BNO055" device="" override_package3d_urn="urn:adsk.eagle:package:43006369/2" override_package_urn="urn:adsk.eagle:footprint:43006370/1"/>
-<part name="U4" library="H3LIS200DLTR" deviceset="H3LIS200DLTR" device="" override_package3d_urn="urn:adsk.eagle:package:43006487/2" override_package_urn="urn:adsk.eagle:footprint:43006488/1"/>
-<part name="C6" library="SparkFun-Capacitors" deviceset="22UF" device="-0805-6.3V-20%" override_package3d_urn="urn:adsk.eagle:package:40331879/2" override_package_urn="urn:adsk.eagle:footprint:40331880/1" value="10 uF"/>
-<part name="C7" library="SparkFun-Capacitors" deviceset="22UF" device="-0805-6.3V-20%" override_package3d_urn="urn:adsk.eagle:package:40331879/2" override_package_urn="urn:adsk.eagle:footprint:40331880/1" value="100 nF"/>
 <part name="R2" library="rcl" library_urn="urn:adsk.eagle:library:334" deviceset="R-US_" device="R0805" package3d_urn="urn:adsk.eagle:package:23553/2" value="4.7K ohm"/>
 <part name="R5" library="rcl" library_urn="urn:adsk.eagle:library:334" deviceset="R-US_" device="R0805" package3d_urn="urn:adsk.eagle:package:23553/2" value="4.7K ohm"/>
@@
 <part name="INTERFACE" library="TS04-66-95-BK-100-SMT" deviceset="TS04-66-95-BK-100-SMT" device=""/>
 <part name="R15" library="rcl" library_urn="urn:adsk.eagle:library:334" deviceset="R-US_" device="R0805" package3d_urn="urn:adsk.eagle:package:23553/2" value="4.7K ohm"/>
+<part name="U$2" library="KX134_Breakout" deviceset="KX134-BREAKOUT" device=""/>
 </parts>
 <sheets>
@@
 </instance>
 <instance part="U$4" gate="G$1" x="320.04" y="157.48" smashed="yes" rot="R270"/>
-<instance part="U4" gate="G$1" x="340.36" y="106.68" smashed="yes" rot="R180">
-<attribute name="NAME" x="353.0693" y="93.9707" size="1.779309375" layer="95" rot="R180"/>
-<attribute name="VALUE" x="353.0645" y="121.9254" size="1.77863125" layer="96" rot="R180"/>
-</instance>
-<instance part="C6" gate="G$1" x="317.5" y="104.14" smashed="yes" rot="R180">
-<attribute name="NAME" x="315.341" y="100.076" size="1.778" layer="95" font="vector" rot="R270"/>
-<attribute name="VALUE" x="315.341" y="112.776" size="1.778" layer="96" font="vector" rot="R270"/>
-</instance>
-<instance part="C7" gate="G$1" x="312.42" y="104.14" smashed="yes" rot="R180">
-<attribute name="NAME" x="310.261" y="100.076" size="1.778" layer="95" font="vector" rot="R270"/>
-<attribute name="VALUE" x="310.261" y="112.776" size="1.778" layer="96" font="vector" rot="R270"/>
-</instance>
 <instance part="R2" gate="G$1" x="109.22" y="22.86" smashed="yes" rot="R180">
 <attribute name="NAME" x="115.57" y="21.3614" size="1.778" layer="95" rot="R180"/>
@@
 <attribute name="VALUE" x="135.89" y="34.798" size="1.778" layer="96"/>
 </instance>
+<instance part="U$2" gate="A" x="350.52" y="96.52" smashed="yes" rot="R90"/>
 </instances>
 <busses>
@@
 <wire x1="332.74" y1="220.98" x2="327.66" y2="220.98" width="0.1524" layer="91"/>
 <label x="327.66" y="220.98" size="1.27" layer="95" rot="R180" xref="yes"/>
-</segment>
-<segment>
-<pinref part="U4" gate="G$1" pin="GND"/>
-<wire x1="322.58" y1="116.84" x2="317.5" y2="116.84" width="0.1524" layer="91"/>
-<label x="309.88" y="116.84" size="1.27" layer="95" rot="R180" xref="yes"/>
-<pinref part="C6" gate="G$1" pin="2"/>
-<wire x1="317.5" y1="116.84" x2="312.42" y2="116.84" width="0.1524" layer="91"/>
-<wire x1="312.42" y1="116.84" x2="309.88" y2="116.84" width="0.1524" layer="91"/>
-<wire x1="317.5" y1="106.68" x2="317.5" y2="116.84" width="0.1524" layer="91"/>
-<junction x="317.5" y="116.84"/>
-<pinref part="C7" gate="G$1" pin="2"/>
-<wire x1="312.42" y1="106.68" x2="312.42" y2="116.84" width="0.1524" layer="91"/>
-<junction x="312.42" y="116.84"/>
-</segment>
-<segment>
-<pinref part="U4" gate="G$1" pin="SDO/SA0"/>
-<wire x1="358.14" y1="109.22" x2="363.22" y2="109.22" width="0.1524" layer="91"/>
-<label x="363.22" y="109.22" size="1.27" layer="95" xref="yes"/>
 </segment>
 <segment>
@@
 <label x="386.08" y="63.5" size="1.27" layer="95" rot="R270" xref="yes"/>
 </segment>
+<segment>
+<pinref part="U$2" gate="A" pin="ADDR"/>
+<wire x1="355.6" y1="116.84" x2="360.68" y2="116.84" width="0.1524" layer="91"/>
+<label x="360.68" y="116.84" size="1.27" layer="95" xref="yes"/>
+</segment>
+<segment>
+<pinref part="U$2" gate="A" pin="GND"/>
+<wire x1="355.6" y1="96.52" x2="360.68" y2="96.52" width="0.1524" layer="91"/>
+<label x="360.68" y="96.52" size="1.27" layer="95" xref="yes"/>
+</segment>
 </net>
 <net name="VCC" class="0">
@@
 </segment>
 <segment>
-<pinref part="U4" gate="G$1" pin="SCL/SPC"/>
-<wire x1="358.14" y1="104.14" x2="363.22" y2="104.14" width="0.1524" layer="91"/>
-<label x="363.22" y="104.14" size="1.27" layer="95" xref="yes"/>
+<pinref part="U$2" gate="A" pin="SCL"/>
+<wire x1="355.6" y1="111.76" x2="360.68" y2="111.76" width="0.1524" layer="91"/>
+<label x="360.68" y="111.76" size="1.27" layer="95" xref="yes"/>
 </segment>
 </net>
@@
 </segment>
 <segment>
-<pinref part="U4" gate="G$1" pin="VDD_IO"/>
-<wire x1="322.58" y1="96.52" x2="320.04" y2="96.52" width="0.1524" layer="91"/>
-<label x="309.88" y="96.52" size="1.27" layer="95" rot="R180" xref="yes"/>
-<pinref part="U4" gate="G$1" pin="VDD"/>
-<wire x1="320.04" y1="96.52" x2="317.5" y2="96.52" width="0.1524" layer="91"/>
-<wire x1="317.5" y1="96.52" x2="312.42" y2="96.52" width="0.1524" layer="91"/>
-<wire x1="312.42" y1="96.52" x2="309.88" y2="96.52" width="0.1524" layer="91"/>
-<wire x1="322.58" y1="99.06" x2="320.04" y2="99.06" width="0.1524" layer="91"/>
-<wire x1="320.04" y1="99.06" x2="320.04" y2="96.52" width="0.1524" layer="91"/>
-<junction x="320.04" y="96.52"/>
-<pinref part="C6" gate="G$1" pin="1"/>
-<wire x1="317.5" y1="96.52" x2="317.5" y2="99.06" width="0.1524" layer="91"/>
-<junction x="317.5" y="96.52"/>
-<pinref part="C7" gate="G$1" pin="1"/>
-<wire x1="312.42" y1="96.52" x2="312.42" y2="99.06" width="0.1524" layer="91"/>
-<junction x="312.42" y="96.52"/>
-</segment>
-<segment>
 <wire x1="114.3" y1="22.86" x2="116.84" y2="22.86" width="0.1524" layer="91"/>
 <label x="116.84" y="22.86" size="1.27" layer="95" xref="yes"/>
@@
 <wire x1="134.62" y1="38.1" x2="132.08" y2="38.1" width="0.1524" layer="91"/>
 <label x="132.08" y="38.1" size="1.27" layer="95" rot="R180" xref="yes"/>
+</segment>
+<segment>
+<pinref part="U$2" gate="A" pin="3V3"/>
+<wire x1="355.6" y1="101.6" x2="360.68" y2="101.6" width="0.1524" layer="91"/>
+<label x="360.68" y="101.6" size="1.27" layer="95" xref="yes"/>
 </segment>
 </net>
@@
 </segment>
 <segment>
-<pinref part="U4" gate="G$1" pin="SDA/SDI/SDO"/>
-<wire x1="358.14" y1="106.68" x2="363.22" y2="106.68" width="0.1524" layer="91"/>
-<label x="363.22" y="106.68" size="1.27" layer="95" xref="yes"/>
+<pinref part="U$2" gate="A" pin="SDA"/>
+<wire x1="355.6" y1="106.68" x2="360.68" y2="106.68" width="0.1524" layer="91"/>
+<label x="360.68" y="106.68" size="1.27" layer="95" xref="yes"/>
 </segment>
 </net>
@@
 </segment>
 </net>
+<net name="CS_KX134" class="0">
+<segment>
+<pinref part="U$2" gate="A" pin="!CS"/>
+<wire x1="355.6" y1="121.92" x2="360.68" y2="121.92" width="0.1524" layer="91"/>
+<label x="360.68" y="121.92" size="1.27" layer="95" xref="yes"/>
+</segment>
+</net>
+<net name="TRIG_KX134" class="0">
+<segment>
+<pinref part="U$2" gate="A" pin="TRIG"/>
+<wire x1="320.04" y1="114.3" x2="317.5" y2="114.3" width="0.1524" layer="91"/>
+<label x="317.5" y="114.3" size="1.27" layer="95" rot="R180" xref="yes"/>
+</segment>
+</net>
+<net name="INT1_KX134" class="0">
+<segment>
+<pinref part="U$2" gate="A" pin="INT1"/>
+<wire x1="320.04" y1="109.22" x2="317.5" y2="109.22" width="0.1524" layer="91"/>
+<label x="317.5" y="109.22" size="1.27" layer="95" rot="R180" xref="yes"/>
+</segment>
+</net>
+<net name="INT2_KX134" class="0">
+<segment>
+<pinref part="U$2" gate="A" pin="INT2"/>
+<wire x1="320.04" y1="104.14" x2="317.5" y2="104.14" width="0.1524" layer="91"/>
+<label x="317.5" y="104.14" size="1.27" layer="95" rot="R180" xref="yes"/>
+</segment>
+</net>

Commit message: Schem of fc and mc
Parts:
- removed R10, R8: 10 ohm, rcl:R-US_0207/10
- renumbered DROGUE_PYRO to DROGUE, MAIN_PYRO to MAIN
Connections:
- net N$11: no longer R8.2
- net N$12: no longer R10.2
- net N$4: no longer R8.1
- net N$7: no longer R10.1

Commit message: flyte done
Parts:
- renumbered JP1 to VBUS_CONN, JP2 to RAM_AIR
Changed lines of the file:
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@@
 <part name="C3" library="SparkFun-Capacitors" deviceset="22UF" device="-0805-6.3V-20%" override_package3d_urn="urn:adsk.eagle:package:40331879/2" override_package_urn="urn:adsk.eagle:footprint:40331880/1" value="22uF"/>
 <part name="C4" library="SparkFun-Capacitors" deviceset="22UF" device="-0805-6.3V-20%" override_package3d_urn="urn:adsk.eagle:package:40331879/2" override_package_urn="urn:adsk.eagle:footprint:40331880/1" value="22uF"/>
-<part name="JP1" library="pinhead" library_urn="urn:adsk.eagle:library:325" deviceset="PINHD-1X2" device="" package3d_urn="urn:adsk.eagle:package:22435/2"/>
+<part name="VBUS_CONN" library="pinhead" library_urn="urn:adsk.eagle:library:325" deviceset="PINHD-1X2" device="" package3d_urn="urn:adsk.eagle:package:22435/2"/>
 <part name="U3" library="ADS1115IDGSR" deviceset="ADS1115IDGSR" device="" override_package3d_urn="urn:adsk.eagle:package:43006505/2" override_package_urn="urn:adsk.eagle:footprint:43006506/1"/>
 <part name="C5" library="SparkFun-Capacitors" deviceset="22UF" device="-0805-6.3V-20%" override_package3d_urn="urn:adsk.eagle:package:40331879/2" override_package_urn="urn:adsk.eagle:footprint:40331880/1" value="100 nF"/>
@@
 <part name="H3" library="holes" library_urn="urn:adsk.eagle:library:237" deviceset="MOUNT-PAD-ROUND" device="3.0" package3d_urn="urn:adsk.eagle:package:14280/1" override_package3d_urn="urn:adsk.eagle:package:43006545/2" override_package_urn="urn:adsk.eagle:footprint:14251/1"/>
 <part name="H4" library="holes" library_urn="urn:adsk.eagle:library:237" deviceset="MOUNT-PAD-ROUND" device="3.0" package3d_urn="urn:adsk.eagle:package:14280/1" override_package3d_urn="urn:adsk.eagle:package:43006542/2" override_package_urn="urn:adsk.eagle:footprint:14251/1"/>
-<part name="JP2" library="pinhead" library_urn="urn:adsk.eagle:library:325" deviceset="PINHD-1X4" device="" package3d_urn="urn:adsk.eagle:package:22407/2" override_package3d_urn="urn:adsk.eagle:package:43006558/3" override_package_urn="urn:adsk.eagle:footprint:22258/1"/>
+<part name="RAM_AIR" library="pinhead" library_urn="urn:adsk.eagle:library:325" deviceset="PINHD-1X4" device="" package3d_urn="urn:adsk.eagle:package:22407/2" override_package3d_urn="urn:adsk.eagle:package:43006558/3" override_package_urn="urn:adsk.eagle:footprint:22258/1"/>
 <part name="LED1" library="led" library_urn="urn:adsk.eagle:library:259" deviceset="LED" device="CHIPLED_1206" package3d_urn="urn:adsk.eagle:package:15823/2"/>
 <part name="LED2" library="led" library_urn="urn:adsk.eagle:library:259" deviceset="LED" device="CHIPLED_1206" package3d_urn="urn:adsk.eagle:package:15823/2"/>
@@
 <part name="C9" library="SparkFun-Capacitors" deviceset="22UF" device="-0805-6.3V-20%" override_package3d_urn="urn:adsk.eagle:package:40331879/2" override_package_urn="urn:adsk.eagle:footprint:40331880/1" value="10 uF"/>
 <part name="C10" library="SparkFun-Capacitors" deviceset="22UF" device="-0805-6.3V-20%" override_package3d_urn="urn:adsk.eagle:package:40331879/2" override_package_urn="urn:adsk.eagle:footprint:40331880/1" value="10 uF"/>
-<part name="Q1" library="IRF540NPBF" deviceset="IRF540NPBF" device=""/>
-<part name="Q2" library="IRF540NPBF" deviceset="IRF540NPBF" device=""/>
-<part name="SERIAL_CONN" library="B4B-XH-AM__LF__SN_" deviceset="B4B-XH-AM_(LF)(SN)" device=""/>
-<part name="GPS_CONN" library="B4B-XH-AM__LF__SN_" deviceset="B4B-XH-AM_(LF)(SN)" device=""/>
-<part name="MOTOR_CONN" library="B4B-XH-AM__LF__SN_" deviceset="B4B-XH-AM_(LF)(SN)" device=""/>
+<part name="Q1" library="IRF540NPBF" deviceset="IRF540NPBF" device="" override_package3d_urn="urn:adsk.eagle:package:44252858/3" override_package_urn="urn:adsk.eagle:footprint:44252859/1"/>
+<part name="Q2" library="IRF540NPBF" deviceset="IRF540NPBF" device="" override_package3d_urn="urn:adsk.eagle:package:44252853/2" override_package_urn="urn:adsk.eagle:footprint:44252854/1"/>
+<part name="SERIAL_CONN" library="B4B-XH-AM__LF__SN_" deviceset="B4B-XH-AM_(LF)(SN)" device="" override_package3d_urn="urn:adsk.eagle:package:44252846/2" override_package_urn="urn:adsk.eagle:footprint:44252847/1"/>
+<part name="GPS_CONN" library="B4B-XH-AM__LF__SN_" deviceset="B4B-XH-AM_(LF)(SN)" device="" override_package3d_urn="urn:adsk.eagle:package:44252849/2" override_package_urn="urn:adsk.eagle:footprint:44252850/1"/>
+<part name="MOTOR_CONN" library="B4B-XH-AM__LF__SN_" deviceset="B4B-XH-AM_(LF)(SN)" device="" override_package3d_urn="urn:adsk.eagle:package:44252851/2" override_package_urn="urn:adsk.eagle:footprint:44252852/1"/>
 <part name="3V3_LED" library="led" library_urn="urn:adsk.eagle:library:259" deviceset="LED" device="CHIPLED_1206" package3d_urn="urn:adsk.eagle:package:15823/2"/>
 <part name="VCC_LED" library="led" library_urn="urn:adsk.eagle:library:259" deviceset="LED" device="CHIPLED_1206" package3d_urn="urn:adsk.eagle:package:15823/2"/>
@@
 <part name="VBUS_LED" library="led" library_urn="urn:adsk.eagle:library:259" deviceset="LED" device="CHIPLED_1206" package3d_urn="urn:adsk.eagle:package:15823/2"/>
 <part name="R19" library="rcl" library_urn="urn:adsk.eagle:library:334" deviceset="R-US_" device="R0805" package3d_urn="urn:adsk.eagle:package:23553/2" value="330 ohm"/>
-<part name="USB_REG" library="AMS1117-3.3" deviceset="AMS1117-3.3" device=""/>
-<part name="LIPO_REG" library="AMS1117-3.3" deviceset="AMS1117-3.3" device=""/>
-<part name="RESET" library="TS04-66-95-BK-100-SMT" deviceset="TS04-66-95-BK-100-SMT" device=""/>
-<part name="INTERFACE" library="TS04-66-95-BK-100-SMT" deviceset="TS04-66-95-BK-100-SMT" device=""/>
+<part name="USB_REG" library="AMS1117-3.3" deviceset="AMS1117-3.3" device="" override_package3d_urn="urn:adsk.eagle:package:44252891/2" override_package_urn="urn:adsk.eagle:footprint:44252892/1"/>
+<part name="LIPO_REG" library="AMS1117-3.3" deviceset="AMS1117-3.3" device="" override_package3d_urn="urn:adsk.eagle:package:44252876/2" override_package_urn="urn:adsk.eagle:footprint:44252877/1"/>
+<part name="RESET" library="TS04-66-95-BK-100-SMT" deviceset="TS04-66-95-BK-100-SMT" device="" override_package3d_urn="urn:adsk.eagle:package:44253003/2" override_package_urn="urn:adsk.eagle:footprint:44253004/1"/>
+<part name="INTERFACE" library="TS04-66-95-BK-100-SMT" deviceset="TS04-66-95-BK-100-SMT" device="" override_package3d_urn="urn:adsk.eagle:package:44252924/2" override_package_urn="urn:adsk.eagle:footprint:44252925/1"/>
 <part name="R15" library="rcl" library_urn="urn:adsk.eagle:library:334" deviceset="R-US_" device="R0805" package3d_urn="urn:adsk.eagle:package:23553/2" value="4.7K ohm"/>
 <part name="U$2" library="KX134_Breakout" deviceset="KX134-BREAKOUT" device=""/>
-<part name="MAIN" library="XT30UPB-M" deviceset="XT30UPB-M" device=""/>
-<part name="LIPO_POWER" library="XT30UPB-M" deviceset="XT30UPB-M" device=""/>
-<part name="DROGUE" library="XT30UPB-M" deviceset="XT30UPB-M" device=""/>
+<part name="MAIN" library="XT30UPB-M" deviceset="XT30UPB-M" device="" override_package3d_urn="urn:adsk.eagle:package:44252914/2" override_package_urn="urn:adsk.eagle:footprint:44252915/1"/>
+<part name="LIPO_POWER" library="XT30UPB-M" deviceset="XT30UPB-M" device="" override_package3d_urn="urn:adsk.eagle:package:44252894/2" override_package_urn="urn:adsk.eagle:footprint:44252895/1"/>
+<part name="DROGUE" library="XT30UPB-M" deviceset="XT30UPB-M" device="" override_package3d_urn="urn:adsk.eagle:package:44252903/2" override_package_urn="urn:adsk.eagle:footprint:44252904/1"/>
 </parts>
 <sheets>
@@
 <attribute name="VALUE" x="245.364" y="185.801" size="1.778" layer="96" font="vector"/>
 </instance>
-<instance part="JP1" gate="G$1" x="233.68" y="101.6" smashed="yes" rot="R90">
+<instance part="VBUS_CONN" gate="G$1" x="233.68" y="101.6" smashed="yes" rot="R90">
 <attribute name="NAME" x="227.965" y="95.25" size="1.778" layer="95" rot="R90"/>
 <attribute name="VALUE" x="238.76" y="95.25" size="1.778" layer="96" rot="R90"/>
@@
 <attribute name="VALUE" x="18.034" y="81.3562" size="1.778" layer="96"/>
 </instance>
-<instance part="JP2" gate="A" x="340.36" y="251.46" smashed="yes" rot="R180">
+<instance part="RAM_AIR" gate="A" x="340.36" y="251.46" smashed="yes" rot="R180">
 <attribute name="NAME" x="346.71" y="243.205" size="1.778" layer="95" rot="R180"/>
 <attribute name="VALUE" x="346.71" y="259.08" size="1.778" layer="96" rot="R180"/>
@@
 </segment>
 <segment>
-<pinref part="JP2" gate="A" pin="1"/>
+<pinref part="RAM_AIR" gate="A" pin="1"/>
 <wire x1="342.9" y1="246.38" x2="350.52" y2="246.38" width="0.1524" layer="91"/>
 <label x="350.52" y="246.38" size="1.27" layer="95" xref="yes"/>
@@
 </segment>
 <segment>
-<pinref part="JP2" gate="A" pin="4"/>
+<pinref part="RAM_AIR" gate="A" pin="4"/>
 <wire x1="342.9" y1="254" x2="350.52" y2="254" width="0.1524" layer="91"/>
 <label x="350.52" y="254" size="1.27" layer="95" xref="yes"/>
@@
 <label x="223.52" y="88.9" size="1.27" layer="95" rot="R90" xref="yes"/>
 <wire x1="231.14" y1="88.9" x2="231.14" y2="99.06" width="0.1524" layer="91"/>
-<pinref part="JP1" gate="G$1" pin="1"/>
+<pinref part="VBUS_CONN" gate="G$1" pin="1"/>
 </segment>
 </net>
 <net name="VBUS_REG" class="0">
 <segment>
-<pinref part="JP1" gate="G$1" pin="2"/>
+<pinref part="VBUS_CONN" gate="G$1" pin="2"/>
 <wire x1="233.68" y1="99.06" x2="233.68" y2="91.44" width="0.1524" layer="91"/>
 <wire x1="233.68" y1="91.44" x2="238.76" y2="91.44" width="0.1524" layer="91"/>
@@
 <net name="AIR_DATA" class="0">
 <segment>
-<pinref part="JP2" gate="A" pin="3"/>
+<pinref part="RAM_AIR" gate="A" pin="3"/>
 <wire x1="342.9" y1="251.46" x2="350.52" y2="251.46" width="0.1524" layer="91"/>
 <label x="350.52" y="251.46" size="1.27" layer="95" xref="yes"/>
@@
 <net name="AIR_SCK" class="0">
 <segment>
-<pinref part="JP2" gate="A" pin="2"/>
+<pinref part="RAM_AIR" gate="A" pin="2"/>
 <wire x1="342.9" y1="248.92" x2="350.52" y2="248.92" width="0.1524" layer="91"/>
 <label x="350.52" y="248.92" size="1.27" layer="95" xref="yes"/>
