File: Eagle files/FLYTE 2.1/FLYTE-v2_1.sch (EAGLE design)
At the start: 65 parts, among them J1 B6B-XH-A(LF)(SN), Q1 IRF540NPBF, Q2 IRF540NPBF, U3 ADS1115IDGSR, U6 W25Q32JVSSIQ

Commit message: oof
Parts:
- removed C1, C2, C3, C4: 22uF, SparkFun-Capacitors:22UF-0805-6.3V-20%
- removed D2: 1N4004, diode:1N4004
- removed JP3: (no value), pinhead:PINHD-1X4
- removed LIPO_REG, USB_REG: AMS1117-3.3, AMS1117-3.3:AMS1117-3.3
- added C11, C6: 10uF, microbuilder:CAP_TANTALUMA/3216_WAVE
- added C12, C7: 10 uF, microbuilder:CAP_TANTALUMA/3216_WAVE
- added Q3: (no value), microbuilder:MOSFET-PWIDE
- added R10, R21: 165K ohm, rcl:R-US_R0805
- added R20, R8: 100K ohm, rcl:R-US_R0805
- added R22, R24: 4.7K ohm, rcl:R-US_R0805
- added U2, U4: MIC29302WU-TR, MIC29302WU:MIC29302WU-TR
- J1: value B6B-XH-A(LF)(SN) -> B5B-XH-A(LF)(SN); device B6B-XH-A_LF__SN_:B6B-XH-A(LF)(SN) -> B5B-XH-A_LF__SN_:B5B-XH-A(LF)(SN)
Connections:
- removed net 20: JP3.1, U1.GP15
- removed net 21: JP3.2, U1.GP21
- removed net TEMP_VOUT: J1.5
- new net MISO0: J1.5, U1.GP16
- new net N$10: R10.2, R8.1, U2.ADJ
- new net N$5: R20.1, R21.2, U4.ADJ
- new net SCK0: J1.3, U1.GP18
- new net VCC_EN: Q3.D, R22.2, U4.EN
- net 3V3: now also C12.+, C7.+, J1.2, R10.1, R21.1, U2.OUT, U4.OUT; no longer C1.2, C3.2, D2.C, J1.6, LIPO_REG.VOUT, USB_REG.VOUT
- net AIR_DATA: now also U1.GP15; no longer U1.GP16
- net AIR_SCK: now also U1.GP14; no longer U1.GP17
- net BNO_INT: now also U1.GP22; no longer U1.GP14
- net CS_TEMP: now also J1.4, U1.GP17; no longer J1.2, JP3.3, U1.GP22
- net GND: now also C11.-, C12.-, C6.-, C7.-, J1.1, R20.2, R22.1, R24.1, R8.2, U2.6, U2.GND, U4.6, U4.GND; no longer C1.1, C2.1, C3.1, C4.1, J1.4, JP3.4, LIPO_REG.ADJ/GND, USB_REG.ADJ/GND
- net LED1: now also U1.GP21; no longer U1.GP19
- net LED2: now also U1.GP19; no longer U1.GP18
- net MISO1: no longer J1.3
- net SCK1: no longer J1.1
- net VBUS_REG: now also C6.+, Q3.G, R24.2, U2.EN, U2.IN; no longer C4.2, USB_REG.VIN
- net VCC: now also C11.+, Q3.S, U4.IN; no longer C2.2, D2.A, LIPO_REG.VIN
