File: Eagle files/FLYTE 2.1/reefingBrd.brd (EAGLE design)
At the start: 160 x 100 mm, 37 parts, among them U1 RASPBERRY_PICOSMD, U2 GY-521MPU6050, U7 IRF540NPBF

Commit message: reefing
Parts:
- removed BATTERY_REGULATOR3V3, USB_REGULATOR: AMS1117-3.3, AMS1117-3.3:SOT229P700X180-4N
- removed C1, C2, C3, C4: 22uF, SparkFun-Capacitors:0805
- removed D2: 1N4004, diode:DO41-10
- added C11, C6: 10uF, microbuilder:EIA3216-18/A-W
- added C12, C7: 10 uF, microbuilder:EIA3216-18/A-W
- added Q3: (no value), microbuilder:SOT23-WIDE
- added R14, R20: 100K ohm, rcl:R0805
- added R15, R21: 165K ohm, rcl:R0805
- added R22, R24: 4.7K ohm, rcl:R0805
- added U3, U4: MIC29302WU-TR, MIC29302WU:TO-263-5_MCH
Connections:
- new net N$10: R14.1, R15.2, U3.5
- new net N$3: R20.1, R21.2, U4.5
- new net VCC_EN: Q3.3, R22.2, U4.1
- net 3V3: now also C12.+, C7.+, R15.1, R21.1, U3.4, U4.4; no longer BATTERY_REGULATOR3V3.2, C1.2, C4.1, D2.C, USB_REGULATOR.2
- net GND: now also C11.-, C12.-, C6.-, C7.-, R14.2, R20.2, R22.1, R24.1, U3.3, U3.6, U4.3, U4.6; no longer BATTERY_REGULATOR3V3.1, C1.1, C2.1, C3.1, C4.2, USB_REGULATOR.1
- net VBUS_REG: now also C6.+, Q3.1, R24.2, U3.1, U3.2; no longer C3.2, USB_REGULATOR.3
- net VCC: now also C11.+, Q3.2, U4.2; no longer BATTERY_REGULATOR3V3.3, C2.2, D2.A

Commit message: .
Parts:
- moved R20 168.1 mm to (66.4, 49.6), flipped to the bottom
- moved R15 164.4 mm to (58.1, 43.1), flipped to the bottom
- moved C11 159.8 mm to (6.15, 67.7)
- moved R22 157.6 mm to (61.6, 54.6), turned to 180 degrees
- moved R21 155.4 mm to (64.4, 43.1), flipped to the bottom
- moved C12 153.2 mm to (3.99, 58.5)
- moved Q3 153.1 mm to (15.4, 73.5), turned to 180 degrees
- moved C7 150.2 mm to (3.70, 62.5)
- moved R24 147.9 mm to (14.6, 65.8), flipped to the bottom, turned to 270 degrees
- moved C6 145.7 mm to (10.5, 54.4)
- moved R14 111.9 mm to (17.8, 65.4), flipped to the bottom, turned to 90 degrees
- moved U3 106.9 mm to (62.4, 30.1), turned to 180 degrees
- moved U4 104.3 mm to (12.4, 41.8), flipped to the bottom, turned to 270 degrees
- moved H1 87.8 mm to (67.2, 4.08)
- moved H2 83.1 mm to (5.08, 74.9)
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Routing:
- net VCC: track 0.00 -> 165.2 mm, vias 0 -> 2
- net 3V3: track 0.00 -> 162.8 mm, vias 0 -> 6
- net VBUS_REG: track 0.00 -> 99.8 mm, vias 0 -> 5
- net VCC_EN: track 0.00 -> 92.0 mm, vias 0 -> 5
- net SDA1: track 0.00 -> 74.1 mm, vias 0 -> 5
- net SDA0: track 0.00 -> 72.7 mm, vias 0 -> 5
- net VBUS: track 0.00 -> 65.6 mm, vias 0 -> 1
- net SCL0: track 0.00 -> 65.6 mm, vias 0 -> 1
- net N$10: track 0.00 -> 57.4 mm, vias 0 -> 3
- net N$3: track 0.00 -> 54.3 mm, vias 0 -> 2
- net SENSE_MAIN: track 0.00 -> 53.5 mm, vias 0 -> 5
- net SCL1: track 0.00 -> 48.7 mm, vias 0 -> 4
- net BUZZER: track 0.00 -> 45.7 mm, vias 0 -> 2
- net MAIN: track 0.00 -> 34.6 mm, vias 0 -> 3
- net N$13: track 0.00 -> 33.4 mm, vias 0 -> 1
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- added copper zone on layer 1, net GND
- added copper zone on layer 16, net GND
Other:
- board size 160 x 100 mm -> 72 x 80 mm

Commit message: .
Other:
- board text added: "10"
- board text added: "100"
- board text added: "165"
- board text added: "330"
- board text added: "3v3"
- board text added: "4.7"
- board text added: "Gnd"
- board text added: "bzzr"
- board text added: "inta"
- board text added: "power"
- board text added: "pyro"
- board text added: "vcc"
