File: Eagle files/FLYTE 2.1/reefingBrd.brd (EAGLE design)
At the start: 61 x 73 mm, 41 parts, among them U1 RASPBERRY_PICOSMD, U2 GY-521MPU6050, U3 MIC29302WU-TR, U4 MIC29302WU-TR, U7 IRF540NPBF

Commit message: new reef
Routing:
- net GND: track 4.28 -> 10.6 mm, vias 1 -> 2
Changed lines of the file:
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@@
 <grid distance="1" unitdist="mil" unit="mil" style="lines" multiple="1" display="no" altdistance="0.25" altunitdist="mil" altunit="mil"/>
 <layers>
-<layer number="1" name="Top" color="4" fill="1" visible="no" active="yes"/>
+<layer number="1" name="Top" color="4" fill="1" visible="yes" active="yes"/>
 <layer number="2" name="Route2" color="16" fill="1" visible="no" active="no"/>
 <layer number="3" name="Route3" color="17" fill="1" visible="no" active="no"/>
@@
 <layer number="19" name="Unrouted" color="6" fill="1" visible="yes" active="yes"/>
 <layer number="20" name="Dimension" color="24" fill="1" visible="yes" active="yes"/>
-<layer number="21" name="tPlace" color="7" fill="1" visible="no" active="yes"/>
+<layer number="21" name="tPlace" color="7" fill="1" visible="yes" active="yes"/>
 <layer number="22" name="bPlace" color="7" fill="1" visible="yes" active="yes"/>
 <layer number="23" name="tOrigins" color="15" fill="1" visible="yes" active="yes"/>
 <layer number="24" name="bOrigins" color="15" fill="1" visible="yes" active="yes"/>
-<layer number="25" name="tNames" color="7" fill="1" visible="no" active="yes"/>
+<layer number="25" name="tNames" color="7" fill="1" visible="yes" active="yes"/>
 <layer number="26" name="bNames" color="7" fill="1" visible="yes" active="yes"/>
-<layer number="27" name="tValues" color="7" fill="1" visible="no" active="yes"/>
+<layer number="27" name="tValues" color="7" fill="1" visible="yes" active="yes"/>
 <layer number="28" name="bValues" color="7" fill="1" visible="yes" active="yes"/>
 <layer number="29" name="tStop" color="7" fill="3" visible="no" active="yes"/>
@@
 </element>
 <element name="R15" library="rcl" library_urn="urn:adsk.eagle:library:334" package="R0805" package3d_urn="urn:adsk.eagle:package:23553/2" value="165K ohm" x="12.23" y="28.42" smashed="yes" rot="MR180">
+<attribute name="NAME" x="20.7898" y="31.2902" size="1.27" layer="26" rot="MR180"/>
 <attribute name="POPULARITY" value="85" x="63.03" y="140.18" size="1.778" layer="28" rot="MR180" display="off"/>
 <attribute name="SPICEPREFIX" value="R" x="63.03" y="140.18" size="1.778" layer="28" rot="MR180" display="off"/>
@@
 <attribute name="POPULARITY" value="85" x="-58.889" y="-85.492" size="1.778" layer="28" rot="MR0" display="off"/>
 <attribute name="SPICEPREFIX" value="R" x="-58.889" y="-85.492" size="1.778" layer="28" rot="MR0" display="off"/>
-<attribute name="VALUE" x="14.3374" y="26.9196" size="1.27" layer="28" rot="MR180"/>
+<attribute name="VALUE" x="12.866" y="23.728" size="1.27" layer="28" rot="MR0"/>
 </element>
 <element name="R22" library="rcl" library_urn="urn:adsk.eagle:library:334" package="R0805" package3d_urn="urn:adsk.eagle:package:23553/2" value="4.7K ohm" x="20.38" y="58.68" smashed="yes" rot="MR90">
@@
 <vertex x="60.96" y="73.025"/>
 </polygon>
-<wire x1="54.6608" y1="32.7698" x2="54.7732" y2="32.8822" width="0.4064" layer="16"/>
 <wire x1="54.7732" y1="32.8822" x2="54.841" y2="32.95" width="0.4064" layer="16"/>
 <wire x1="54.621" y1="28.9191" x2="54.621" y2="31.253" width="0.4064" layer="1"/>
@@
 <wire x1="54.6608" y1="31.2928" x2="54.7732" y2="31.4052" width="0.4064" layer="16"/>
 <wire x1="54.7732" y1="31.4052" x2="54.7732" y2="32.8822" width="0.4064" layer="16"/>
+<wire x1="54.841" y1="32.95" x2="55.6514" y2="33.7604" width="0.4064" layer="16"/>
+<wire x1="55.6514" y1="33.7604" x2="55.6514" y2="36.4236" width="0.4064" layer="16"/>
+<via x="55.6514" y="36.4236" extent="1-16" drill="0.35"/>
+<wire x1="54.7578" y1="38.6723" x2="54.7578" y2="37.3172" width="0.4064" layer="1"/>
+<wire x1="54.7578" y1="37.3172" x2="55.6514" y2="36.4236" width="0.4064" layer="1"/>
 </signal>
 <signal name="3V3">
