File: Eagle files/FLYTE 2.1/reefingBrd.sch (EAGLE design)
At the start: 65 parts, among them J1 B6B-XH-A(LF)(SN), Q1 IRF540NPBF, Q2 IRF540NPBF, U3 ADS1115IDGSR, U6 W25Q32JVSSIQ

Commit message: reefing
Parts:
- removed 3V3_LED, VBUS_LED, VCC_LED: (no value), led:LEDCHIPLED_1206
- removed C10, C9: 10 uF, SparkFun-Capacitors:22UF-0805-6.3V-20%
- removed C5, C8: 100 nF, SparkFun-Capacitors:22UF-0805-6.3V-20%
- removed DROGUE, LIPO_POWER, MAIN: XT30UPB-M, XT30UPB-M:XT30UPB-M
- removed DR_ARM: (no value), con-wago-500:W237-102
- removed GPS_CONN, MOTOR_CONN, SERIAL_CONN: B4B-XH-AM_(LF)(SN), B4B-XH-AM__LF__SN_:B4B-XH-AM_(LF)(SN)
- removed H3, H4: MOUNT-PAD-ROUND3.0, holes:MOUNT-PAD-ROUND3.0
- removed INTERFACE, RESET: TS04-66-95-BK-100-SMT, TS04-66-95-BK-100-SMT:TS04-66-95-BK-100-SMT
- removed J1: B6B-XH-A(LF)(SN), B6B-XH-A_LF__SN_:B6B-XH-A(LF)(SN)
- removed JP3, RAM_AIR: (no value), pinhead:PINHD-1X4
- removed LIPO_REG, USB_REG: AMS1117-3.3, AMS1117-3.3:AMS1117-3.3
- removed Q1, Q2: IRF540NPBF, IRF540NPBF:IRF540NPBF
- removed R14, R16, R18, R19: 330 ohm, rcl:R-US_R0805
- removed R15: 4.7K ohm, rcl:R-US_R0805
- removed R17, R23, R25: 100K ohm, rcl:R-US_R0805
- removed U$4: BNO055, BNO055:BNO055
- removed U3: ADS1115IDGSR, ADS1115IDGSR:ADS1115IDGSR
- removed U6: W25Q32JVSSIQ, W25Q32JVSSIQ:W25Q32JVSSIQ
- removed VBUS_CONN: (no value), pinhead:PINHD-1X2
- removed XBEE: XBP9B-XCST-021, XBP9B-XCST-021:XBP9B-XCST-021
- added BATTERY_REGULATOR3V3, USB_REGULATOR: AMS1117-3.3, AMS1117-3.3:AMS1117-3.3
- added JP1: (no value), pinhead:PINHD-1X2
- added LED3, LED4, LED5: (no value), led:LEDCHIPLED_1206
- added POWER, PYRO: XT30PW-M, XT30PW-M:XT30PW-M
- added R10: 330 ohm, rcl:R-US_R0805
- added R8: 100K, rcl:R-US_R0805
- added U2: GY-521MPU6050, gy-87:GY-521MPU6050
- added U7: IRF540NPBF, IRF540NPBF:IRF540NPBF
- R11, R12: value 100K ohm -> 330 ohm
- R5: value 4.7K ohm -> 100K
- R6: value 4.7K ohm -> 4.7K
- R9: value 10 ohm -> 330 ohm; device rcl:R-US_0207/10 -> rcl:R-US_R0805
- U$2: value KX134-BREAKOUT -> BMP280; device KX134_Breakout:KX134-BREAKOUT -> BMP280:BMP280
- U1: value (none) -> RASPBERRY_PICOSMD; device RpiPico:RASPBERRY_PICO-NO_DEBUG -> RpiPico:RASPBERRY_PICOSMD
Connections:
- removed net 20: JP3.1, U1.GP15
- removed net 21: JP3.2, U1.GP21
- removed net AIR_DATA: RAM_AIR.3, U1.GP16
- removed net AIR_SCK: RAM_AIR.2, U1.GP17
- removed net BNO_INT: U$4.INT, U1.GP14
- removed net CS_FLASH: R15.2, U1.GP13, U6.!CS
- removed net CS_KX134: U$2.!CS
- removed net CS_TEMP: J1.2, JP3.3, U1.GP22
- removed net CTS: U1.GP27, XBEE.NCTS/DIO7
- removed net DROGUE: Q1.G, R1.2, U1.GP28
- removed net GPS_RX: GPS_CONN.1, U1.GP8
- removed net GPS_TX: GPS_CONN.2, U1.GP9
- removed net INT1_KX134: U$2.INT1
- removed net INT2_KX134: U$2.INT2
- removed net MISO1: J1.3, R17.2, U1.GP12, U6.DO(IO1)
- removed net MOSI1: U1.GP11, U6.DI(IO0)
- removed net N$16: 3V3_LED.C, R14.2
- removed net N$18: R18.2, VCC_LED.C
- removed net N$2 (its old number): DROGUE.-, DR_ARM-1.KL
- removed net N$3: INTERFACE.2, U1.GP26
- removed net N$7: DROGUE.+, R23.1, R9.1
- removed net N$8: RESET.2, U1.RUN
- removed net SCK1: J1.1, U1.GP10, U6.CLK
- removed net SENSE_DROG: R23.2, R25.1, U3.AIN1
- removed net TELE_RX: SERIAL_CONN.3, U1.GP0, XBEE.DIN/NCONFIG/DIO14
- removed net TELE_TX: SERIAL_CONN.2, U1.GP1, XBEE.DOUT/DIO13
- removed net TEMP_VOUT: J1.5
- removed net TRIG_KX134: U$2.TRIG
- new net N$5: R7.2, U7.D
- net 3V3: now also BATTERY_REGULATOR3V3.VOUT, C4.1, R1.1, U$2.SDO, U$2.VCC, U2.3V3, USB_REGULATOR.VOUT; no longer 3V3_LED.A, C10.1, C3.2, C5.1, C8.2, C9.2, GPS_CONN.4, J1.6, LED1.A, LIPO_REG.VOUT, LS1.1, R15.1, R17.1, R5.1, RAM_AIR.4, SERIAL_CONN.4, U$2.3V3, U$4.RST, U$4.VIN, U3.AIN2, U3.VDD, U6.!HOLD!/!RESET!(IO3), U6.!WP!(IO2), U6.VCC, USB_REG.VOUT, XBEE.VCC
- net BUZZER: now also LS1.1, U1.GP19; no longer LS1.2, U1.GP6
- net GND: now also BATTERY_REGULATOR3V3.ADJ/GND, C4.2, LS1.2, POWER.N, R10.1, R11.1, R12.1, R13.1, R8.1, R9.1, U2.GND, U7.S, USB_REGULATOR.ADJ/GND; no longer C10.2, C4.1, C5.2, C8.1, C9.1, GPS_CONN.3, H3.MOUNT, H4.MOUNT, INTERFACE.4, J1.4, JP3.4, LIPO_POWER.-, LIPO_REG.ADJ/GND, MOTOR_CONN.1, Q1.S, Q2.S, R1.1, R12.2, R14.1, R18.1, R19.1, R25.2, RAM_AIR.1, RESET.4, SERIAL_CONN.1, U$2.ADDR, U$4.ADR, U$4.GND, U$4.PS0, U$4.PS1, U3.ADDR, U3.GND, U6.GND, USB_REG.ADJ/GND, XBEE.GND
- net LED1: now also LED4.A, U1.GP17; no longer R13.1, U1.GP19
- net LED2: now also LED5.A, U1.GP16; no longer R16.1, U1.GP18
- net MAIN: now also U7.G; no longer Q2.G
- net N$11: now also LED1.C, R9.2; no longer Q2.D, R7.2
- net N$12: now also LED2.C, R10.2; no longer Q1.D, R9.2
- net N$13: now also LED3.C, R11.2; no longer R19.2, VBUS_LED.C
- net N$14: now also LED4.C, R12.2; no longer LED1.C, R13.2
- net N$15: now also LED5.C, R13.2; no longer LED2.C, R16.2
- net N$4: now also PYRO.N, R5.2; no longer MAIN.-, R11.1
- net N$6: now also PYRO.P; no longer MAIN.+
- net SCL0: now also R2.2, U2.SCL; no longer MOTOR_CONN.3, R5.2
- net SCL1: no longer U$4.SCL, U3.SCL
- net SDA0: now also R1.2; no longer MOTOR_CONN.2, R2.2
- net SDA1: now also U2.SDA; no longer U$4.SDA, U3.SDA
- net SENSE_MAIN: now also R5.1, R8.2, U1.GP28; no longer R11.2, R12.1, U3.AIN0
- net VBUS: now also JP1.2, LED3.A; no longer VBUS_CONN.1
- net VBUS_REG: now also C3.2, JP1.1, USB_REGULATOR.VIN; no longer C4.2, USB_REG.VIN, VBUS_CONN.2, VBUS_LED.A
- net VCC: now also BATTERY_REGULATOR3V3.VIN, LED1.A, POWER.P; no longer DR_ARM-2.KL, LIPO_POWER.+, LIPO_REG.VIN, U3.AIN3, VCC_LED.A
Other:
- note removed: "All CS lines have a pullup resistor to initialize all components as inactive If this is not done, garbage values may cause trouble Similarly, all MISO lines are pulled up as they are only used when slave components are in use. They might float otherwise"
- note removed: "DATA LOGGING"
- note removed: "Data logging components communicate with pico on SPI1 bus"
- note removed: "MICROCONTOLLER AND PERIPHERALS"
- note removed: "POWER AND PYROS"
- note removed: "PS0 and PS1 are tied to GND to select I2C"
- note removed: "Push button for interfacing (Bad idea?)"
- note removed: "Push button to reset pico (Bad idea, do not solder in actual board)"
- note removed: "Reset Pin is ACTIVE LOW"
- note removed: "SENSORS"
- note removed: "Sensors are on the I2C_1 bus (Except the ram air speed sensor)"
- note removed: "TELEMETRY"
- note removed: "Telemetry communicates with pico on SPI0 bus"
- moved on the sheet: C1, C2, C3, C4, D1, D2, D3, H1, H2, LED1, LED2, LS1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

Commit message: oof
Parts:
- removed U$1, U$2: BMP280, BMP280:BMP280
Connections:
- net 3V3: no longer U$1.VCC, U$2.SDO, U$2.VCC
- net GND: no longer U$1.GND, U$1.SDO, U$2.GND
- net SCL1: no longer U$1.SCL, U$2.SCL
- net SDA1: no longer U$1.SDA, U$2.SDA
Changed lines of the file:
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@@
 <part name="R3" library="rcl" library_urn="urn:adsk.eagle:library:334" deviceset="R-US_" device="R0805" package3d_urn="urn:adsk.eagle:package:23553/2" value="4.7K ohm"/>
 <part name="R4" library="rcl" library_urn="urn:adsk.eagle:library:334" deviceset="R-US_" device="R0805" package3d_urn="urn:adsk.eagle:package:23553/2" value="4.7K ohm"/>
-<part name="U$1" library="BMP280" deviceset="BMP280" device="" override_package3d_urn="urn:adsk.eagle:package:38477931/2" override_package_urn="urn:adsk.eagle:footprint:38477932/1"/>
-<part name="U$2" library="BMP280" deviceset="BMP280" device="" override_package3d_urn="urn:adsk.eagle:package:38477931/2" override_package_urn="urn:adsk.eagle:footprint:38477932/1"/>
 <part name="POWER" library="XT30PW-M" deviceset="XT30PW-M" device="" override_package3d_urn="urn:adsk.eagle:package:43074490/2" override_package_urn="urn:adsk.eagle:footprint:43074491/1"/>
 <part name="R6" library="rcl" library_urn="urn:adsk.eagle:library:334" deviceset="R-US_" device="R0805" package3d_urn="urn:adsk.eagle:package:23553/2" value="4.7K"/>
@@
 <attribute name="VALUE" x="29.21" y="11.938" size="1.778" layer="96"/>
 </instance>
-<instance part="U$1" gate="G$1" x="-45.72" y="43.18" smashed="yes"/>
-<instance part="U$2" gate="G$1" x="-25.4" y="43.18" smashed="yes"/>
 <instance part="POWER" gate="G$1" x="33.02" y="43.18" smashed="yes">
 <attribute name="NAME" x="25.4" y="46.482" size="1.778" layer="95"/>
@@
 <label x="119.38" y="-43.18" size="1.27" layer="95" xref="yes"/>
 <pinref part="U1" gate="U$1" pin="GND"/>
-</segment>
-<segment>
-<pinref part="U$1" gate="G$1" pin="GND"/>
-<wire x1="-48.26" y1="27.94" x2="-48.26" y2="20.32" width="0.1524" layer="91"/>
-<label x="-48.26" y="20.32" size="1.27" layer="95" rot="R270" xref="yes"/>
-</segment>
-<segment>
-<label x="-38.1" y="20.32" size="1.27" layer="95" rot="R270" xref="yes"/>
-<pinref part="U$1" gate="G$1" pin="SDO"/>
-<wire x1="-38.1" y1="27.94" x2="-38.1" y2="20.32" width="0.1524" layer="91"/>
-</segment>
-<segment>
-<pinref part="U$2" gate="G$1" pin="GND"/>
-<wire x1="-27.94" y1="27.94" x2="-27.94" y2="20.32" width="0.1524" layer="91"/>
-<label x="-27.94" y="20.32" size="1.27" layer="95" rot="R270" xref="yes"/>
 </segment>
 <segment>
@@
 <label x="50.8" y="15.24" size="1.27" layer="95" xref="yes"/>
 </segment>
-<segment>
-<pinref part="U$1" gate="G$1" pin="SCL"/>
-<wire x1="-45.72" y1="27.94" x2="-45.72" y2="20.32" width="0.1524" layer="91"/>
-<label x="-45.72" y="20.32" size="1.4224" layer="95" rot="R270" xref="yes"/>
-<label x="-45.72" y="20.32" size="1.4224" layer="95" rot="R270" xref="yes"/>
-<label x="-45.72" y="20.32" size="1.4224" layer="95" rot="R270" xref="yes"/>
-</segment>
-<segment>
-<pinref part="U$2" gate="G$1" pin="SCL"/>
-<wire x1="-25.4" y1="27.94" x2="-25.4" y2="20.32" width="0.1524" layer="91"/>
-<label x="-25.4" y="20.32" size="1.4224" layer="95" rot="R270" xref="yes"/>
-<label x="-25.4" y="20.32" size="1.4224" layer="95" rot="R270" xref="yes"/>
-<label x="-25.4" y="20.32" size="1.4224" layer="95" rot="R270" xref="yes"/>
-</segment>
 </net>
 <net name="3V3" class="0">
@@
 <label x="129.54" y="25.4" size="1.27" layer="95" xref="yes"/>
 <wire x1="121.92" y1="25.4" x2="129.54" y2="25.4" width="0.1524" layer="91"/>
-</segment>
-<segment>
-<pinref part="U$1" gate="G$1" pin="VCC"/>
-<wire x1="-50.8" y1="27.94" x2="-50.8" y2="20.32" width="0.1524" layer="91"/>
-<label x="-50.8" y="20.32" size="1.27" layer="95" rot="R270" xref="yes"/>
-</segment>
-<segment>
-<pinref part="U$2" gate="G$1" pin="VCC"/>
-<wire x1="-30.48" y1="27.94" x2="-30.48" y2="20.32" width="0.1524" layer="91"/>
-<label x="-30.48" y="20.32" size="1.27" layer="95" rot="R270" xref="yes"/>
 </segment>
 <segment>
@@
 </segment>
 <segment>
-<label x="-17.78" y="20.32" size="1.27" layer="95" rot="R270" xref="yes"/>
-<pinref part="U$2" gate="G$1" pin="SDO"/>
-<wire x1="-17.78" y1="27.94" x2="-17.78" y2="20.32" width="0.1524" layer="91"/>
-</segment>
-<segment>
 <pinref part="R1" gate="G$1" pin="1"/>
 <wire x1="40.64" y1="5.08" x2="12.7" y2="5.08" width="0.1524" layer="91"/>
@@
 </segment>
 <segment>
-<pinref part="U$2" gate="G$1" pin="SDA"/>
-<wire x1="-22.86" y1="27.94" x2="-22.86" y2="20.32" width="0.1524" layer="91"/>
-<label x="-22.86" y="20.32" size="1.4224" layer="95" rot="R270" xref="yes"/>
-</segment>
-<segment>
-<pinref part="U$1" gate="G$1" pin="SDA"/>
-<wire x1="-43.18" y1="27.94" x2="-43.18" y2="20.32" width="0.1524" layer="91"/>
-<label x="-43.18" y="20.32" size="1.4224" layer="95" rot="R270" xref="yes"/>
-</segment>
-<segment>

Commit message: reefing
Parts:
- removed BATTERY_REGULATOR3V3, USB_REGULATOR: AMS1117-3.3, AMS1117-3.3:AMS1117-3.3
- removed C1, C2, C3, C4: 22uF, SparkFun-Capacitors:22UF-0805-6.3V-20%
- removed D2: 1N4004, diode:1N4004
- added C11, C6: 10uF, microbuilder:CAP_TANTALUMA/3216_WAVE
- added C12, C7: 10 uF, microbuilder:CAP_TANTALUMA/3216_WAVE
- added Q3: (no value), microbuilder:MOSFET-PWIDE
- added R14, R20: 100K ohm, rcl:R-US_R0805
- added R15, R21: 165K ohm, rcl:R-US_R0805
- added R22, R24: 4.7K ohm, rcl:R-US_R0805
- added U3, U4: MIC29302WU-TR, MIC29302WU:MIC29302WU-TR
Connections:
- new net N$10: R14.1, R15.2, U3.ADJ
- new net N$3: R20.1, R21.2, U4.ADJ
- new net VCC_EN: Q3.D, R22.2, U4.EN
- net 3V3: now also C12.+, C7.+, R15.1, R21.1, U3.OUT, U4.OUT; no longer BATTERY_REGULATOR3V3.VOUT, C1.2, C4.1, D2.C, USB_REGULATOR.VOUT
- net GND: now also C11.-, C12.-, C6.-, C7.-, R14.2, R20.2, R22.1, R24.1, U3.6, U3.GND, U4.6, U4.GND; no longer BATTERY_REGULATOR3V3.ADJ/GND, C1.1, C2.1, C3.1, C4.2, USB_REGULATOR.ADJ/GND
- net VBUS_REG: now also C6.+, Q3.G, R24.2, U3.EN, U3.IN; no longer C3.2, USB_REGULATOR.VIN
- net VCC: now also C11.+, Q3.S, U4.IN; no longer BATTERY_REGULATOR3V3.VIN, C2.2, D2.A

Commit message: .
Connections:
- net SDA0: now also U2.SDA
- net SDA1: no longer U2.SDA
Changed lines of the file:
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@@
 <label x="48.26" y="17.78" size="1.27" layer="95" xref="yes"/>
-</segment>
-<segment>
-<pinref part="U2" gate="G$1" pin="SDA"/>
-<wire x1="-30.48" y1="-20.32" x2="-25.4" y2="-20.32" width="0.1524" layer="91"/>
-<label x="-25.4" y="-20.32" size="1.27" layer="95" xref="yes"/>
 </segment>
 </net>
@@
 <label x="68.58" y="-10.16" size="1.27" layer="95" rot="R180" xref="yes"/>
 </segment>
+<segment>
+<pinref part="U2" gate="G$1" pin="SDA"/>
+<wire x1="-30.48" y1="-20.32" x2="-25.4" y2="-20.32" width="0.1524" layer="91"/>
+<label x="-25.4" y="-20.32" size="1.27" layer="95" xref="yes"/>
+</segment>
 </net>

Commit message: new reef
Parts:
- removed R3, R4: 4.7K ohm, rcl:R-US_R0805
Connections:
- removed net SCL1: R4.2, U1.GP3
- removed net SDA1: R3.2, U1.GP2
- net 3V3: no longer R3.1, R4.1
Changed lines of the file:
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@@
 <parts>
 <part name="D1" library="diode" library_urn="urn:adsk.eagle:library:210" deviceset="1N4004" device="" package3d_urn="urn:adsk.eagle:package:43336/1" override_package3d_urn="urn:adsk.eagle:package:40381849/2" override_package_urn="urn:adsk.eagle:footprint:43094/1"/>
-<part name="R3" library="rcl" library_urn="urn:adsk.eagle:library:334" deviceset="R-US_" device="R0805" package3d_urn="urn:adsk.eagle:package:23553/2" value="4.7K ohm"/>
-<part name="R4" library="rcl" library_urn="urn:adsk.eagle:library:334" deviceset="R-US_" device="R0805" package3d_urn="urn:adsk.eagle:package:23553/2" value="4.7K ohm"/>
 <part name="POWER" library="XT30PW-M" deviceset="XT30PW-M" device="" override_package3d_urn="urn:adsk.eagle:package:43074490/2" override_package_urn="urn:adsk.eagle:footprint:43074491/1"/>
 <part name="R6" library="rcl" library_urn="urn:adsk.eagle:library:334" deviceset="R-US_" device="R0805" package3d_urn="urn:adsk.eagle:package:23553/2" value="4.7K"/>
@@
 <attribute name="NAME" x="119.38" y="22.3774" size="1.778" layer="95" rot="R180"/>
 </instance>
-<instance part="R3" gate="G$1" x="20.32" y="10.16" smashed="yes">
-<attribute name="NAME" x="19.05" y="14.1986" size="1.778" layer="95"/>
-<attribute name="VALUE" x="16.51" y="11.938" size="1.778" layer="96"/>
-</instance>
-<instance part="R4" gate="G$1" x="33.02" y="7.62" smashed="yes">
-<attribute name="NAME" x="31.75" y="14.1986" size="1.778" layer="95"/>
-<attribute name="VALUE" x="29.21" y="11.938" size="1.778" layer="96"/>
-</instance>
 <instance part="POWER" gate="G$1" x="33.02" y="43.18" smashed="yes">
 <attribute name="NAME" x="25.4" y="46.482" size="1.778" layer="95"/>
@@
 </segment>
 </net>
-<net name="SCL1" class="0">
-<segment>
-<wire x1="38.1" y1="7.62" x2="50.8" y2="7.62" width="0.1524" layer="91"/>
-<pinref part="R4" gate="G$1" pin="2"/>
-<pinref part="U1" gate="U$1" pin="GP3"/>
-<wire x1="50.8" y1="7.62" x2="76.2" y2="7.62" width="0.1524" layer="91"/>
-<wire x1="50.8" y1="7.62" x2="50.8" y2="15.24" width="0.1524" layer="91"/>
-<junction x="50.8" y="7.62"/>
-<label x="50.8" y="15.24" size="1.27" layer="95" xref="yes"/>
-</segment>
-</net>
 <net name="3V3" class="0">
-<segment>
-<wire x1="15.24" y1="10.16" x2="12.7" y2="10.16" width="0.1524" layer="91"/>
-<label x="12.7" y="10.16" size="1.27" layer="95" rot="R180" xref="yes"/>
-<pinref part="R3" gate="G$1" pin="1"/>
-</segment>
-<segment>
-<wire x1="27.94" y1="7.62" x2="12.7" y2="7.62" width="0.1524" layer="91"/>
-<label x="12.7" y="7.62" size="1.27" layer="95" rot="R180" xref="yes"/>
-<pinref part="R4" gate="G$1" pin="1"/>
-</segment>
 <segment>
 <pinref part="D1" gate="1" pin="A"/>
@@
 </segment>
 </net>
-<net name="SDA1" class="0">
-<segment>
-<wire x1="25.4" y1="10.16" x2="48.26" y2="10.16" width="0.1524" layer="91"/>
-<pinref part="R3" gate="G$1" pin="2"/>
-<pinref part="U1" gate="U$1" pin="GP2"/>
-<wire x1="48.26" y1="10.16" x2="76.2" y2="10.16" width="0.1524" layer="91"/>
-<wire x1="48.26" y1="10.16" x2="48.26" y2="17.78" width="0.1524" layer="91"/>
-<junction x="48.26" y="10.16"/>
-<label x="48.26" y="17.78" size="1.27" layer="95" xref="yes"/>
-</segment>
-</net>
