File: Eagle files/FLYTE 2.1/reef1.0/reefingBrd.brd (EAGLE design)
At the start: 72 x 80 mm, 43 parts, among them U1 RASPBERRY_PICOSMD, U2 GY-521MPU6050, U3 MIC29302WU-TR, U4 MIC29302WU-TR, U7 IRF540NPBF

Commit message: .
Connections:
- net SDA0: now also U2.SDA
- net SDA1: no longer U2.SDA
Routing:
- net SDA0: track 72.7 -> 97.1 mm, vias 5 -> 7
- net SDA1: track 74.1 -> 56.2 mm
Changed lines of the file:
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@@
 <drawing>
 <settings>
-<setting alwaysvectorfont="yes"/>
+<setting alwaysvectorfont="no"/>
 <setting verticaltext="up"/>
 </settings>
 <grid distance="1" unitdist="mil" unit="mil" style="lines" multiple="1" display="no" altdistance="0.025" altunitdist="mil" altunit="mil"/>
 <layers>
-<layer number="1" name="Top" color="4" fill="1" visible="no" active="yes"/>
-<layer number="16" name="Bottom" color="1" fill="1" visible="no" active="yes"/>
+<layer number="1" name="Top" color="4" fill="1" visible="yes" active="yes"/>
+<layer number="16" name="Bottom" color="1" fill="1" visible="yes" active="yes"/>
 <layer number="17" name="Pads" color="2" fill="1" visible="yes" active="yes"/>
 <layer number="18" name="Vias" color="2" fill="1" visible="yes" active="yes"/>
@@
 <contactref element="R3" pad="2"/>
 <contactref element="U1" pad="P$4"/>
-<contactref element="U2" pad="SDA"/>
-<wire x1="21.8342" y1="24.6419" x2="22.3969" y2="24.0792" width="0.254" layer="1"/>
-<wire x1="22.3969" y1="24.0792" x2="39.5478" y2="24.0792" width="0.254" layer="1"/>
 <via x="39.5478" y="24.0792" extent="1-16" drill="0.35"/>
 <wire x1="39.5478" y1="24.0792" x2="43.7134" y2="19.9136" width="0.254" layer="16"/>
@@
 <wire x1="30.9372" y1="41.783" x2="31.417" y2="41.3032" width="0.254" layer="16"/>
 <wire x1="31.417" y1="41.3032" x2="31.417" y2="39.5154" width="0.254" layer="16"/>
+<contactref element="U2" pad="SDA"/>
+<via x="31.6484" y="32.7152" extent="1-16" drill="0.35"/>
+<wire x1="21.8342" y1="24.6419" x2="24.3106" y2="27.1183" width="0.254" layer="1"/>
+<wire x1="28.94793125" y1="29.1728" x2="29.9752" y2="30.20006875" width="0.254" layer="1"/>
+<wire x1="29.9752" y1="30.20006875" x2="29.9752" y2="31.042" width="0.254" layer="1"/>
+<wire x1="29.9752" y1="31.042" x2="31.6484" y2="32.7152" width="0.254" layer="1"/>
+<wire x1="24.3106" y1="27.1183" x2="24.3106" y2="27.98573125" width="0.254" layer="1"/>
+<wire x1="24.3106" y1="27.98573125" x2="25.49766875" y2="29.1728" width="0.254" layer="1"/>
+<wire x1="25.49766875" y1="29.1728" x2="28.94793125" y2="29.1728" width="0.254" layer="1"/>
+<wire x1="31.6484" y1="32.7152" x2="32.639" y2="31.7246" width="0.254" layer="16"/>
+<via x="37.1348" y="35.687" extent="1-16" drill="0.35"/>
+<wire x1="33.83973125" y1="31.7246" x2="37.1348" y2="35.01966875" width="0.254" layer="16"/>
+<wire x1="37.1348" y1="35.01966875" x2="37.1348" y2="35.687" width="0.254" layer="16"/>
+<wire x1="37.1348" y1="35.687" x2="36.79" y2="36.0318" width="0.254" layer="1"/>
+<wire x1="36.79" y1="36.0318" x2="34.9006" y2="36.0318" width="0.254" layer="1"/>
+<wire x1="32.639" y1="31.7246" x2="33.83973125" y2="31.7246" width="0.254" layer="16"/>
 </signal>
 <signal name="SCL0">
