File: Eagle files/FLYTE 3/FLYTE 3.01/FLYTE 3.01.sch (EAGLE design)
At the start: 307 parts, among them IC1 BMP280, IC2 MPXV5100DP, IC3 AS179-92LF, IC4 AS179-92LF, IC6 MAX8574EUT+T, IC8 MCP73843-420I_MS, IC9 MCP73844-840I_MS, J10 B2B-XH-A(LF)(SN), J11 B2B-XH-A(LF)(SN), J12 CON-SMA-EDGE-S, J13 282834-2, J2 282834-2, J3 282834-2, J4 282834-2, J5 282834-2, J6 503182-1852, J7 XT60-M, J8 CON-SMA-EDGE-S, J9 282834-2, Q1 SI7625DN-T1-GE3, Q6 SI7625DN-T1-GE3, Q7 SI7625DN-T1-GE3, U1 BNO055, U2 CJ3400, U3 CJ3400, U5 CJ3400, U6 ADS1115IDGSR, U7 CJ3400, U9 ADS1115IDGSR, X6 USB Type C, Y1 FC-135_32.7680KA-A0

Commit message: FLYTE 3.02
Parts:
- removed 1S_POW: V60D60C-M3_I, V60D60C-M3_I:V60D60C-M3_I
- removed 32XO: ASE, crystal:ASE
- removed AOA, SS, TVC_1, TVC_2, TVC_3, TVC_4: 03-JST-B3B-XH-A, bt_con-jst-xh (1):03-JST-B3B-XH-A
- removed C102, C106, C68, C75, C82, C89: 10 uF, standardparts:CAPACITOR.0603
- removed C103, C109, C69, C76, C83, C90: 4.7 uF, standardparts:CAPACITOR.0603
- removed C104: 1.2 nF, standardparts:CAPACITOR.0603
- removed C105, C111, C64, C71, C78, C85, C92: 22 nF, standardparts:CAPACITOR.0603
- removed C107, C108, C113, C114, C66, C67, C73, C74, C80, C81, C87, C88, C94, C95: 0.22 uF, standardparts:CAPACITOR.0603
- removed C110, C70, C77, C84, C91: 1.8 nF, standardparts:CAPACITOR.0603
- removed C112: 100 uF, standardparts:CAPACITOR.1210
- removed C65: 220 uF, standardparts:CAPACITOR.1210
- removed C72, C79, C86, C93: 100 uF, standardparts:CAPACITOR.1206
- removed C96, C98: 10uF, microbuilder:CAP_TANTALUMA/3216_WAVE
- removed C97: 0.1 uF, standardparts:CAPACITOR.0603
- removed CHG_BST, REG_3V3, REG_5V, REG_CAM, REG_FIN_1, REG_FIN_2, REG_TVC_1, REG_TVC_2: LT3120JV#PBF, LT3120JV#PBF:LT3120JV#PBF
- removed D3, D9: (no value), standardparts:LED.0603
- removed D8: RSX501LAM20TR, RSX501LAM20TR:RSX501LAM20TR
- removed H1: MOUNT-PAD-ROUND3.0, holes:MOUNT-PAD-ROUND3.0
- removed IC4: AS179-92LF, AS179-92LF:AS179-92LF
- removed IC8: MCP73843-420I_MS, MCP73843-420I_MS:MCP73843-420I_MS
- removed J12: CON-SMA-EDGE-S, CON-SMA-EDGE-S:CON-SMA-EDGE-S
- removed L10, L11, L12, L13, L14, L15, L16, L9: 4.7 uH, standardparts:RF-INDUCTOR.0603
- removed L2: 2.7 nH, standardparts:RF-INDUCTOR.0603
- removed L3, L4: 5.6 nH, standardparts:RF-INDUCTOR.0603
- removed L5: 33 nH, standardparts:RF-INDUCTOR.0603
- removed Q6, Q7: SI7625DN-T1-GE3, SI7625DN-T1-GE3:SI7625DN-T1-GE3
- removed SX1272: SX1272IMLTRT, SX1272IMLTRT:SX1272IMLTRT
- removed U$11: XT30UPB-M, XT30UPB-M:XT30UPB-M
- removed U$2: SN74LVC1G04DBVR, SN74LVC1G04DBVR:SN74LVC1G04DBVR
- added J1: 282834-2, 282834-2:282834-2
- added R100, R98, R99: 0 ohm, standardparts:RESISTOR.0603
- added R101, R93, R94, R95, R96: 10k ohm, standardparts:RESISTOR.0603
- added R102: (no value), standardparts:RESISTOR.0805
- added R12, R57, R71, R91: 100k ohm, standardparts:RESISTOR.0603
- added R90, R92: 140k ohm, standardparts:RESISTOR.0603
- added R97: (no value), standardparts:RESISTOR.0603
- added U10, U4: LM1117-3.3, LM1117-3.3:LM1117-3.3
- added U11, U12, U13, U14, U8: MIC29302WU-TR, MIC29302WU:MIC29302WU-TR
- added U15, U16: ADS1115IDGSR, ADS1115IDGSR:ADS1115IDGSR
- added U17: CP2102, CP2102:CP2102
- added VR1: XL6009, XL6009:XL6009
- added XBEE: XBP9B-XCST-021, XBP9B-XCST-021:XBP9B-XCST-021
- C1: value 10 uF -> (none)
- C18: value 10 uF -> 10uF; device standardparts:CAPACITOR.0603 -> microbuilder:CAP_TANTALUMA/3216_WAVE
- C34: value 3.3 nF -> 47pF
- C35: value 22 nF -> (none)
- C38: value 24 pF -> (none)
- C39: value 24 pF -> 1uF
- C4: value 4.7 uF -> (none)
- C40: value 100 nF -> 10uF
- C41, C43: value 100 nF -> 10uF; device standardparts:CAPACITOR.0603 -> microbuilder:CAP_TANTALUMA/3216_WAVE
- C42: value 100 nF -> 10 uF; device standardparts:CAPACITOR.0603 -> microbuilder:CAP_TANTALUMA/3216_WAVE
- C44, C49: value 3.3 pF -> 10 uF; device standardparts:CAPACITOR.0603 -> microbuilder:CAP_TANTALUMA/3216_WAVE
- C45: value 47 pF -> 10uF; device standardparts:CAPACITOR.0603 -> microbuilder:CAP_TANTALUMA/3216_WAVE
- C46, C48: value 8.2 pF -> 10 uF; device standardparts:CAPACITOR.0603 -> microbuilder:CAP_TANTALUMA/3216_WAVE
- C47: value 22 pF -> 10uF; device standardparts:CAPACITOR.0603 -> microbuilder:CAP_TANTALUMA/3216_WAVE
- C50: value 1.5 pF -> 0.1 uF
- C51: value 10 nF -> 0.1 uF
- C52: value 47 pF -> 100 uF; device standardparts:CAPACITOR.0603 -> standardparts:CAPACITOR.1206
- C53: value 47 pF -> 1 uF
- C58: device standardparts:CAPACITOR.0805 -> standardparts:CAPACITOR.1206
- C59: value 0.22 uF -> 1 uF
- C60: value 0.22 uF -> 100 uF; device standardparts:CAPACITOR.0603 -> standardparts:CAPACITOR.1206
- C61: value 10 uF -> 100 nF
- C63: value 1.8 nF -> 1 uF
- J8: value CON-SMA-EDGE-S -> SMA_CONNECTOR; device CON-SMA-EDGE-S:CON-SMA-EDGE-S -> SMA_CONNECTOR (1):SMA_CONNECTOR
- L1: value 10 nH -> 33 uH; device standardparts:RF-INDUCTOR.0603 -> SRR1260-330M:SRR1260-330M
- R16: value 412k ohm -> 365k ohm
- R17: value 100k ohm -> 57.6k ohm
- R18: value 137k ohm -> 100k ohm
- R22, R53: value 46.4k ohm -> 100k ohm
- R23: value 158k ohm -> 301k ohm
- R24: value 523k ohm -> 0.1 ohm
- R25, R37: value 100k ohm -> 0.13 ohm
- R27: value 10k ohm -> 301k ohm
- R28: value 105 ohm -> 100k ohm
- R30: value 316k ohm -> 301k ohm
- R32: value 46.4k ohm -> 301k ohm
- R33: value 158k ohm -> 100k ohm
- R35: value 523k ohm -> 301k ohm
- R38, R45, R49: value 46.4k ohm -> 0.13 ohm
- R39, R42, R46, R50: value 158k ohm -> 0.13 ohm
- R40, R47, R51: value 402k ohm -> 0.13 ohm
- R41: value 21k ohm -> 0.13 ohm
- R44, R48, R52: value 50k ohm -> 0.13 ohm
- R54, R67, R86, R88: value 158k ohm -> 140k ohm
- R55: value 402k ohm -> 100k ohm
- R56: value 50k ohm -> 140k ohm
- R60: value 0.1 ohm -> 140k ohm
- R61: value 158 ohm -> 100k ohm
- R62, R69: value 100k ohm -> 140k ohm
- R68: value 1.3M ohm -> 100k ohm
- R74: value 36.5k ohm -> 140k ohm
- R76: value 43k ohm -> 140k ohm
- R78: value 28k ohm -> 140k ohm
Connections:
- removed net 1S_ADC: R78.2, R79.1, U6.AIN1
- removed net 1S_POW: 1S_POW.A_1, D3.1, Q7.D_1, Q7.D_2, Q7.D_3, Q7.D_4, Q7.D_5, Q7.D_6, Q7.D_7
- removed net 2S_ADC: R16.2, R17.1, U6.AIN0
- removed net 2S_POW: 1S_POW.A_2, D4.1, Q6.D_1, Q6.D_2, Q6.D_3, Q6.D_4, Q6.D_5, Q6.D_6, Q6.D_7
- removed net AIN2: R88.2, R89.1, U6.AIN2
- removed net AIN3: R86.2, R87.1, U6.AIN3
- removed net AOA_ADC: AOA-3.1, U9.AIN0
- removed net CS_SX: R27.1, RP2040.GPIO21, SX1272.NSS
- removed net F1: R30.1, R31.2, REG_3V3.FB
- removed net F2: R35.1, R37.2, REG_5V.FB
- removed net F3: R40.1, R44.2, REG_FIN_1.FB
- removed net F4: R47.1, R48.2, REG_FIN_2.FB
- removed net F5: R51.1, R52.2, REG_TVC_1.FB
- removed net F6: R55.1, R56.2, REG_TVC_2.FB
- removed net F7: CHG_BST.FB, R68.1, R69.2
- removed net F8: R24.1, R25.2, REG_CAM.FB
- removed net N$100: IC8.SENSE, Q3.S, R60.2
- removed net N$101: D9.2, R61.1
- removed net N$102: IC8.STAT1, R61.2
- removed net N$103: IC8.EN, R62.1
- removed net N$104: IC8.DRV, Q3.G
- removed net N$106: C97.2, IC8.TIMER
- removed net N$111: CHG_BST.VC, R66.2
- removed net N$112: C104.2, R66.1
- removed net N$113: CHG_BST.RT, R67.2
- removed net N$114: C105.2, CHG_BST.BST3
- removed net N$115: C107.2, CHG_BST.SW2_1, CHG_BST.SW2_2, L15.1
- removed net N$116: C108.1, CHG_BST.SW1_1, CHG_BST.SW1_2, L15.2
- removed net N$117: C107.1, CHG_BST.BST2
- removed net N$118: C108.2, CHG_BST.BST1
- removed net N$119: R23.2, REG_CAM.RT
- removed net N$120: C111.2, REG_CAM.BST3
- removed net N$122: C113.2, L16.1, REG_CAM.SW2_1, REG_CAM.SW2_2
- removed net N$123: C114.1, L16.2, REG_CAM.SW1_1, REG_CAM.SW1_2
- removed net N$124: C113.1, REG_CAM.BST2
- removed net N$125: C114.2, REG_CAM.BST1
- removed net N$46: R42.2, REG_3V3.RT
- removed net N$47: C35.2, REG_3V3.BST3
- removed net N$48: C60.1, L9.2, REG_3V3.SW1_1, REG_3V3.SW1_2
- removed net N$49: C59.1, REG_3V3.BST2
- removed net N$52: D3.2, R28.2
- removed net N$56: C60.2, REG_3V3.BST1
- removed net N$57: R32.2, REG_5V.VC
- removed net N$58: C63.2, R32.1
- removed net N$59: R33.2, REG_5V.RT
- removed net N$60: C64.2, REG_5V.BST3
- removed net N$61: C66.2, L10.1, REG_5V.SW2_1, REG_5V.SW2_2
- removed net N$62: C67.1, L10.2, REG_5V.SW1_1, REG_5V.SW1_2
- removed net N$63: C66.1, REG_5V.BST2
- removed net N$64: C67.2, REG_5V.BST1
- removed net N$65: R38.2, REG_FIN_1.VC
- removed net N$66: C70.2, R38.1
- removed net N$67: R39.2, REG_FIN_1.RT
- removed net N$68: C71.2, REG_FIN_1.BST3
- removed net N$69: C73.2, L11.1, REG_FIN_1.SW2_1, REG_FIN_1.SW2_2
- removed net N$70: C74.1, L11.2, REG_FIN_1.SW1_1, REG_FIN_1.SW1_2
- removed net N$71: C73.1, REG_FIN_1.BST2
- removed net N$72: C74.2, REG_FIN_1.BST1
- removed net N$73: R45.2, REG_FIN_2.VC
- removed net N$74: C77.2, R45.1
- removed net N$75: R46.2, REG_FIN_2.RT
- removed net N$76: C78.2, REG_FIN_2.BST3
- removed net N$77: C80.2, L12.1, REG_FIN_2.SW2_1, REG_FIN_2.SW2_2
- removed net N$78: C81.1, L12.2, REG_FIN_2.SW1_1, REG_FIN_2.SW1_2
- removed net N$79: C80.1, REG_FIN_2.BST2
- removed net N$80: C81.2, REG_FIN_2.BST1
- removed net N$81: R49.2, REG_TVC_1.VC
- removed net N$82: C84.2, R49.1
- removed net N$83: R50.2, REG_TVC_1.RT
- removed net N$84: C85.2, REG_TVC_1.BST3
- removed net N$85: C87.2, L13.1, REG_TVC_1.SW2_1, REG_TVC_1.SW2_2
- removed net N$86: C88.1, L13.2, REG_TVC_1.SW1_1, REG_TVC_1.SW1_2
- removed net N$87: C87.1, REG_TVC_1.BST2
- removed net N$88: C88.2, REG_TVC_1.BST1
- removed net N$89: R53.2, REG_TVC_2.VC
- removed net N$90: C91.2, R53.1
- removed net N$91: R54.2, REG_TVC_2.RT
- removed net N$92: C92.2, REG_TVC_2.BST3
- removed net N$93: C94.2, L14.1, REG_TVC_2.SW2_1, REG_TVC_2.SW2_2
- removed net N$94: C95.1, L14.2, REG_TVC_2.SW1_1, REG_TVC_2.SW1_2
- removed net N$95: C94.1, REG_TVC_2.BST2
- removed net N$96: C95.2, REG_TVC_2.BST1
- removed net N$99: C96.+, D8.K, D9.1, IC8.VDD, R60.1, R62.2
- removed net N_RXTX: IC4.V2, U$2.Y
- removed net P1: C4.1, REG_3V3.MPPC, REG_3V3.PROG, REG_3V3.VCC
- removed net P2: C62.1, REG_5V.MPPC, REG_5V.PROG, REG_5V.VCC
- removed net P3: C69.1, REG_FIN_1.MPPC, REG_FIN_1.PROG, REG_FIN_1.VCC
- removed net P4: C76.1, REG_FIN_2.MPPC, REG_FIN_2.PROG, REG_FIN_2.VCC
- removed net P5: C83.1, REG_TVC_1.MPPC, REG_TVC_1.PROG, REG_TVC_1.VCC
- removed net P6: C90.1, REG_TVC_2.MPPC, REG_TVC_2.PROG, REG_TVC_2.VCC
- removed net P7: C103.1, CHG_BST.MPPC, CHG_BST.PROG, CHG_BST.VCC
- removed net P8: C109.1, REG_CAM.MPPC, REG_CAM.PROG, REG_CAM.VCC
- removed net RXTX: IC4.V1, SX1272.RXTX, U$2.A
- removed net SS_ADC: SS-3.1, U9.AIN1
- removed net TVC_1: RP2040.GPIO7, TVC_1-3.1
- removed net TVC_2: RP2040.GPIO6, TVC_2-3.1
- removed net TVC_3: RP2040.GPIO13, TVC_3-3.1
- removed net TVC_4: RP2040.GPIO4, TVC_4-3.1
- removed net VCC_CTRL: 1S_POW.COMMON_K, C68.1, C75.1, C82.1, C89.1, Q1.S_1, Q1.S_2, Q1.S_3, REG_FIN_1.PVIN_1, REG_FIN_1.PVIN_2, REG_FIN_1.PVIN_3, REG_FIN_1.VIN, REG_FIN_2.PVIN_1, REG_FIN_2.PVIN_2, REG_FIN_2.PVIN_3, REG_FIN_2.VIN, REG_TVC_1.PVIN_1, REG_TVC_1.PVIN_2, REG_TVC_1.PVIN_3, REG_TVC_1.VIN, REG_TVC_2.PVIN_1, REG_TVC_2.PVIN_2, REG_TVC_2.PVIN_3, REG_TVC_2.VIN
- removed net V_TVC_1: C85.1, C86.2, R51.2, R86.1, REG_TVC_1.ISN, REG_TVC_1.ISP, REG_TVC_1.PVOUT_1, REG_TVC_1.PVOUT_2, TVC_1-2.1, TVC_2-2.1
- removed net V_TVC_2: C92.1, C93.2, R55.2, REG_TVC_2.ISN, REG_TVC_2.ISP, REG_TVC_2.PVOUT_1, REG_TVC_2.PVOUT_2, TVC_3-2.1, TVC_4-2.1
- removed net XIN1: 32XO.OUT, C38.2, SX1272.XTA
- removed net XOUT1: 32XO.TRI, C39.2, SX1272.XTB
- removed net XT30+: C98.+, IC8.VBAT, Q3.D, Q7.S_1, Q7.S_2, Q7.S_3, R78.1, U$11.+
- new net 3V3_OP: AC1.IO_VDD, AC1.NCS, AC1.SDO/ADDR, AC1.VDD, C10.2, C11.2, C115.2, C12.2, C13.2, C14.2, C15.2, C16.2, C19.2, C20.1, C21.1, C25.1, C30.2, C31.2, C32.2, C5.1, C61.2, C9.2, FLASH.VCC, IC1.VDD, IC1.VDDIO, J6.VDD, L6.1, Q3.D, R0.2, R10.2, R13.2, R14.1, R43.1, R72.2, R73.2, R80.2, R81.2, R82.2, R83.2, R84.2, R85.2, RP2040.ADC_AVDD, RP2040.IOVDD0, RP2040.IOVDD1, RP2040.IOVDD2, RP2040.IOVDD3, RP2040.IOVDD4, RP2040.IOVDD5, RP2040.RUN, RP2040.USB_VDD, RP2040.VREG_IN, U$1.NC, U$1.VCC, U1.NBOOT_LOAD_PIN, U1.VDD, U1.VDDIO, U16.AIN3
- new net 3V3_SET: C62.1, J1.2, Q3.G, R101.2, U17.VDD
- new net CTS: R98.1, XBEE.NCTS/DIO7
- new net D+1: R102.2, U17.D+
- new net D1: FIN_1-2.1, R25.2, R37.2, R38.2, R39.2, R55.1
- new net D2: FIN_2-2.1, R45.2, R46.2, R47.2, R48.2, R68.1
- new net D3: FIN_3-2.1, R40.2, R41.2, R42.2, R44.2, R77.1
- new net D4: FIN_4-2.1, R49.2, R50.2, R51.2, R52.2, R89.1
- new net DTR: R100.1, XBEE.NDTR/SLEEP_RQ/DIO8
- new net N$13: R28.1, R30.2, U11.ADJ
- new net N$18: D10.A, L1.1, VR1.SW
- new net N$20: R55.2, R56.1, U6.AIN1
- new net N$5: R12.1, R27.2, U8.ADJ
- new net RSSI: RP2040.GPIO23, XBEE.DIO10/PWM0
- new net RTS: R99.1, XBEE.NRTS/DIO6
- new net TEL_RST: RP2040.GPIO22, XBEE.!RESET
- new net TEL_RX: R93.1, RP2040.GPIO24, U17.TXD, XBEE.DIN/NCONFIG/DIO14
- new net TEL_TX: R94.1, RP2040.GPIO25, U17.RXD, XBEE.DOUT/DIO13
- new net V_FIN_3: C46.+, R32.1, R40.1, R41.1, R42.1, R44.1, R75.1, U12.OUT
- new net V_FIN_4: C48.+, R35.1, R49.1, R50.1, R51.1, R52.1, R87.1, U13.OUT
- net 3V3: now also C34.2, C39.2, C4.2, J1.1, Q3.S, R93.2, R94.2, U4.VOUT, U4.VOUT_2, XBEE.VCC; no longer AC1.IO_VDD, AC1.NCS, AC1.SDO/ADDR, AC1.VDD, AOA-2.1, C10.2, C11.2, C115.2, C12.2, C13.2, C14.2, C15.2, C16.2, C17.1, C19.2, C20.1, C21.1, C25.1, C29.1, C30.2, C31.2, C32.2, C35.1, C41.2, C5.1, C58.2, C9.2, FLASH.VCC, IC1.VDD, IC1.VDDIO, J6.VDD, L6.1, R0.2, R10.2, R13.2, R14.1, R27.2, R30.2, R43.1, R72.2, R73.2, R80.2, R81.2, R82.2, R83.2, R84.2, R85.2, REG_3V3.ISN, REG_3V3.ISP, REG_3V3.PVOUT_1, REG_3V3.PVOUT_2, RP2040.IOVDD0, RP2040.IOVDD1, RP2040.IOVDD2, RP2040.IOVDD3, RP2040.IOVDD4, RP2040.IOVDD5, RP2040.RUN, RP2040.USB_VDD, RP2040.VREG_IN, SS-2.1, SX1272.VBAT1, SX1272.VBAT2, U$1.NC, U$1.VCC, U$2.NC, U$2.VCC, U1.NBOOT_LOAD_PIN, U1.VDD, U1.VDDIO, U6.VDD, U9.ADDR, U9.VDD
- net 5V: now also C17.1, C29.1, C38.2, C50.1, C51.1, U10.VOUT, U10.VOUT_2, U15.VDD, U16.VDD, U6.VDD, U9.ADDR, U9.VDD; no longer C64.1, C65.2, R35.2, REG_5V.ISN, REG_5V.ISP, REG_5V.PVOUT_1, REG_5V.PVOUT_2
- net BUZZER: now also RP2040.GPIO14; no longer RP2040.GPIO11
- net CAM: now also RP2040.GPIO8, U14.EN; no longer REG_CAM.EN/UVLO, RP2040.GPIO23
- net CS_SD: now also RP2040.GPIO1; no longer RP2040.GPIO5
- net CTRL: now also RP2040.GPIO9, U11.EN, U12.EN, U13.EN, U8.EN; no longer REG_FIN_1.EN/UVLO, REG_FIN_2.EN/UVLO, REG_TVC_1.EN/UVLO, REG_TVC_2.EN/UVLO, RP2040.GPIO24
- net D+: now also R102.1
- net D-: now also U17.D-
- net DROGUE: now also RP2040.GPIO21; no longer RP2040.GPIO0
- net FIN_1: now also RP2040.GPIO4; no longer RP2040.GPIO10
- net FIN_2: now also RP2040.GPIO5; no longer RP2040.GPIO12
- net FIN_3: now also RP2040.GPIO6; no longer RP2040.GPIO8
- net FIN_4: now also RP2040.GPIO7; no longer RP2040.GPIO9
- net GND: now also C1.1, C18.-, C35.1, C4.1, C41.-, C42.-, C43.-, C44.-, C45.-, C46.-, C47.-, C48.-, C49.-, C50.2, C52.1, C53.1, C59.1, C60.1, C61.1, C63.2, R101.1, R12.2, R22.2, R28.2, R31.2, R33.2, R54.2, R56.2, R60.2, R62.2, R67.2, R69.2, R74.2, R76.2, R78.2, R86.2, R88.2, R90.2, R92.2, R95.1, R97.2, U10.ADJ/GND, U11.6, U11.GND, U12.6, U12.GND, U13.6, U13.GND, U14.6, U14.GND, U15.GND, U16.GND, U17.GND, U4.ADJ/GND, U8.6, U8.GND, VR1.GND, XBEE.GND; no longer 32XO.GND, 32XO.VDD, AOA-1.1, C1.2, C102.2, C103.2, C104.1, C106.1, C109.2, C110.1, C112.1, C18.2, C4.2, C41.1, C42.1, C43.1, C44.2, C46.2, C48.2, C49.2, C52.2, C61.2, C63.1, C65.1, C68.2, C69.2, C70.1, C72.1, C75.2, C76.2, C77.1, C79.1, C82.2, C83.2, C84.1, C86.1, C89.2, C90.2, C91.1, C93.1, C96.-, C97.1, C98.-, CHG_BST.GND_1, CHG_BST.GND_2, CHG_BST.GND_3, CHG_BST.GND_4, CHG_BST.PGND, CHG_BST.SYNC/MODE, H1.MOUNT, IC4.GND, IC8.VSS, J12.2, R23.1, R25.1, R28.1, R31.1, R33.1, R37.1, R39.1, R42.1, R44.1, R46.1, R48.1, R50.1, R52.1, R54.1, R56.1, R67.1, R69.1, R75.2, R77.2, R79.2, R87.2, R89.2, REG_3V3.GND_1, REG_3V3.GND_2, REG_3V3.GND_3, REG_3V3.GND_4, REG_3V3.PGND, REG_3V3.SYNC/MODE, REG_5V.GND_1, REG_5V.GND_2, REG_5V.GND_3, REG_5V.GND_4, REG_5V.PGND, REG_5V.SYNC/MODE, REG_CAM.GND_1, REG_CAM.GND_2, REG_CAM.GND_3, REG_CAM.GND_4, REG_CAM.PGND, REG_CAM.SYNC/MODE, REG_FIN_1.GND_1, REG_FIN_1.GND_2, REG_FIN_1.GND_3, REG_FIN_1.GND_4, REG_FIN_1.PGND, REG_FIN_1.SYNC/MODE, REG_FIN_2.GND_1, REG_FIN_2.GND_2, REG_FIN_2.GND_3, REG_FIN_2.GND_4, REG_FIN_2.PGND, REG_FIN_2.SYNC/MODE, REG_TVC_1.GND_1, REG_TVC_1.GND_2, REG_TVC_1.GND_3, REG_TVC_1.GND_4, REG_TVC_1.PGND, REG_TVC_1.SYNC/MODE, REG_TVC_2.GND_1, REG_TVC_2.GND_2, REG_TVC_2.GND_3, REG_TVC_2.GND_4, REG_TVC_2.PGND, REG_TVC_2.SYNC/MODE, SS-1.1, SX1272.GND, TVC_1-1.1, TVC_2-1.1, TVC_3-1.1, TVC_4-1.1, U$11.-, U$2.GND
- net GPS_RX: now also RP2040.GPIO12; no longer RP2040.GPIO16
- net GPS_TX: now also RP2040.GPIO13; no longer RP2040.GPIO17
- net IGN1: now also RP2040.GPIO18; no longer RP2040.GPIO3
- net IGN2: now also RP2040.GPIO19; no longer RP2040.GPIO2
- net LED: now also RP2040.GPIO15; no longer RP2040.GPIO25
- net MAIN: now also RP2040.GPIO20; no longer RP2040.GPIO1
- net MISO: now also RP2040.GPIO0; no longer RP2040.GPIO20, SX1272.MISO
- net MOS: now also D4.1
- net MOSI: now also RP2040.GPIO3; no longer RP2040.GPIO19, SX1272.MOSI
- net N$14: now also R31.1, R32.2, U12.ADJ; no longer R74.2, R75.1, U9.AIN2
- net N$16: now also R22.1, R23.2, U14.ADJ; no longer R22.2, REG_CAM.VC
- net N$17: now also R33.1, R35.2, U13.ADJ; no longer R76.2, R77.1, U9.AIN3
- net N$19: now also R16.2, R17.1, VR1.FB; no longer C110.2, R22.1
- net N$21: now also R53.2, R54.1, U6.AIN0; no longer C59.2, L9.1, REG_3V3.SW2_1, REG_3V3.SW2_2
- net N$29: now also R57.2, R60.1, U6.AIN2; no longer C42.2, SX1272.VR_ANA
- net N$30: now also R61.2, R62.1, U6.AIN3; no longer C43.2, SX1272.VR_DIG
- net N$31: now also R66.2, R67.1, U9.AIN0; no longer C44.1, C45.2, L1.2
- net N$32: now also R68.2, R69.1, U9.AIN1; no longer C45.1, IC4.J2
- net N$33: now also R71.2, R74.1, U9.AIN2; no longer L2.1, SX1272.PA_BOOST
- net N$34: now also R75.2, R76.1, U15.AIN0; no longer L1.1, SX1272.RFI
- net N$35: now also R77.2, R78.1, U15.AIN1; no longer C46.1, C47.2, L2.2, L5.2
- net N$36: now also R79.2, R86.1, U15.AIN2; no longer C47.1, L3.1
- net N$37: now also R87.2, R88.1, U16.AIN0; no longer C48.1, C50.2, L3.2, L4.1
- net N$38: now also R89.2, R90.1, U16.AIN1; no longer C49.1, C50.1, IC4.J3, L4.2
- net N$39: now also R91.2, R92.1, U16.AIN2; no longer C51.1, C52.1, L5.1, SX1272.VR_PA
- net N$40: now also R96.2, U17.!RST; no longer C53.2, IC4.J1
- net N$41: now also R97.1, U17.!SUSPEND; no longer C53.1, J12.1
- net N$42: now also R98.2, U17.CTS; no longer C99.+, D10.K, D11.1, IC9.VDD, R63.1, R65.2
- net N$43: now also R99.2, U17.RTS; no longer R41.2, REG_3V3.VC
- net N$44: now also R24.1
- net N$45: now also R100.2, U17.DTR; no longer C34.2, R41.1
- net PYRO_DROGUE: now also R71.1
- net PYRO_IGN1: now also R79.1
- net PYRO_IGN2: now also R91.1
- net PYRO_MAIN: now also R57.1
- net S: now also RP2040.GPIO16; no longer RP2040.GPIO22
- net SCK: now also RP2040.GPIO2; no longer RP2040.GPIO18, SX1272.SCK
- net SCL: now also RP2040.GPIO11, U15.ADDR, U15.SCL, U16.SCL; no longer RP2040.GPIO15
- net SDA: now also RP2040.GPIO10, U15.SDA, U16.ADDR, U16.SDA; no longer RP2040.GPIO14
- net USB+: now also C56.1, IC6.!SHDN, IC6.VCC
- net USB_BST: now also C58.2, C59.2, C60.2, C99.+, D10.K, D11.1, IC9.VDD, R16.1, R24.2, R63.1, R65.2; no longer C105.1, C106.2, CHG_BST.ISN, CHG_BST.ISP, CHG_BST.PVOUT_1, CHG_BST.PVOUT_2, D10.A, D8.A, Q6.G, Q7.G, R68.2
- net USB_CHG: now also C52.2, C53.2, L1.2, R95.2, VR1.EN, VR1.VIN; no longer C102.1, CHG_BST.EN/UVLO, CHG_BST.PVIN_1, CHG_BST.PVIN_2, CHG_BST.PVIN_3, CHG_BST.VIN
- net VBUS: now also C63.1, R96.1, U17.REGIN, U17.VBUS; no longer C56.1, IC6.!SHDN, IC6.VCC
- net VCC: now also C1.2, C18.+, C35.2, U10.VIN, U14.IN, U4.VIN; no longer C1.1, C18.1, C61.1, REG_3V3.EN/UVLO, REG_3V3.PVIN_1, REG_3V3.PVIN_2, REG_3V3.PVIN_3, REG_3V3.VIN, REG_5V.EN/UVLO, REG_5V.PVIN_1, REG_5V.PVIN_2, REG_5V.PVIN_3, REG_5V.VIN, REG_CAM.PVIN_1, REG_CAM.PVIN_2, REG_CAM.PVIN_3, REG_CAM.VIN
- net VOLT_DP: now also U9.AIN3; no longer R74.1
- net VOLT_MOTOR: now also U15.AIN3; no longer R76.1
- net V_CAM: now also C49.+, R23.1, U14.OUT; no longer C111.1, C112.2, R24.2, REG_CAM.ISN, REG_CAM.ISP, REG_CAM.PVOUT_1, REG_CAM.PVOUT_2
- net V_FIN_1: now also C42.+, R25.1, R27.1, R37.1, R38.1, R39.1, R53.1, U8.OUT; no longer C71.1, C72.2, FIN_1-2.1, FIN_2-2.1, R40.2, REG_FIN_1.ISN, REG_FIN_1.ISP, REG_FIN_1.PVOUT_1, REG_FIN_1.PVOUT_2
- net V_FIN_2: now also C44.+, R30.1, R45.1, R46.1, R47.1, R48.1, R66.1, U11.OUT; no longer C78.1, C79.2, FIN_3-2.1, FIN_4-2.1, R47.2, R88.1, REG_FIN_2.ISN, REG_FIN_2.ISP, REG_FIN_2.PVOUT_1, REG_FIN_2.PVOUT_2
- net XT60+: now also C41.+, C43.+, C45.+, C47.+, Q1.S_1, Q1.S_2, Q1.S_3, R61.1, U11.IN, U12.IN, U13.IN, U8.IN; no longer Q6.S_1, Q6.S_2, Q6.S_3, R16.1
Other:
- note added: "Telemetry communicates with pico on SPI0 bus"
- note removed: "SX1272"
- moved on the sheet: AC1, C1, C100, C101, C29, C30, C31, C34, C35, C38, C39, C4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
