File: Eagle files/Ground-station/GND_SATION_PCB_1.01_.sch (EAGLE design)
At the start: 59 parts, among them IC1 BMP280, J1 USB4110GFA, J2 2.4" TFT, J6 503182-1852, U1 TPS62142RGTR, U2 SOIC127P790X216-8NW25Q128JVJSQ

Commit message: Finalized power regulation
Parts:
- removed L2: SRP4020-2R2MIND_BOURNS_SRP4020, SRP4020-2R2M:SRP4020-2R2MIND_BOURNS_SRP4020
- removed LED: (no value), standardparts:LED.0603
- removed R1: 60 ohm, standardparts:RESISTOR.0603
- removed R18: 100k, rcl:R-EU_R0603
- added C22, C23, C24: 10uF, rcl:C-EUC0603
- added U3: AMS1117-3.3, AMS1117-3.3:AMS1117-3.3
- added X1: (no value), con-wago-500:W237-102
- C17: value 6.8nF -> (none)
- C18: value 22uF -> (none)
- C19: value 10uF -> (none)
- U1: value TPS62142RGTR -> AMS1117-5.0; device TPS62142RGTR:TPS62142RGTR -> AMS1117-5.0:AMS1117-5.0
Connections:
- removed net LED: LED.1
- removed net N$17: L2.2, U1.SW_1, U1.SW_2, U1.SW_3
- removed net N$20: R18.1, U1.PG
- removed net VIN: C19.1, D1.K, D2.K, U1.AVIN, U1.EN, U1.PVIN_11, U1.PVIN_12
- removed net V_BAT: D2.A
- new net +5V: C22.1, D1.K, D2.K, U3.VIN
- new net N$16: C17.1, U1.VIN, X1-1.KL
- net 0: now also C22.2, C23.2, C24.2, U3.GND/ADJ, X1-2.KL; no longer C17.2, C18.2, C19.2, U1.AGND, U1.DEF, U1.EXP, U1.FB, U1.PGND_15, U1.PGND_16
- net 3V3: now also C23.1, C24.1, U3.VOUT; no longer C18.1, L2.1, R18.2, U1.FSW, U1.VOS
- net GND: no longer R1.2
- net N$10: now also C18.1, C19.1, D2.A, U1.VOUT; no longer C17.1, U1.SS/TR
- net N$2: now also C17.2, C18.2, C19.2, U1.GND/ADJ; no longer LED.2, R1.1
Other:
- moved on the sheet: C17, C18, C19, D2, J1

Commit message: Refined power supply design for 5V and added the XT60 M connector
Connections:
- removed net 3V3_OP: C115.2, J6.VDD, R13.2, R43.1, R72.2
- removed net VCC: C1.1, C2.1, C21.2, IC1.VDD, IC1.VDDIO, J2.VCC, R11.1, R12.1, R14.2, R19.1, R2.1, R3.1, R5.1, U$2.VDD
- net +3V3: now also C1.1, C2.1, IC1.VDD, IC1.VDDIO, R5.1, U$2.VDD
- net 0: now also C1.2, C2.2, IC1.GND, R4.1, RP2040.GND, RP2040.TESTEN, U$2.GND
- net 3V3: now also C115.2, C21.2, J2.VCC, J6.VDD, R11.1, R12.1, R13.2, R14.2, R19.1, R2.1, R3.1, R43.1, R72.2
- net GND: no longer C1.2, C2.2, IC1.GND, R4.1, RP2040.GND, RP2040.TESTEN, U$2.GND
