File: Eagle files/Ground-station/GND_SATION_PCB_1.02.sch (EAGLE design)
At the start: 64 parts, among them IC1 BMP280, J1 USB4110GFA, J2 XT60-M, J3 B4B-XH-AM_(LF)(SN), J6 503182-1852, U1 AMS1117-5.0, U3 AMS1117-3.3, U4 SOIC127P790X216-8NW25Q128JVJSQ

Commit message: Update GND_SATION_PCB_1.02.sch
NJIIUHHJ IH
Parts:
- removed R9: 10k ohm, standardparts:RESISTOR.0603
- added D2: SS14, SS14:SS14
- added R6: 27 ohm, rcl:R-EU_R0805
- R8: value 10k ohm -> 27 ohm; device standardparts:RESISTOR.0603 -> rcl:R-EU_R0805
Connections:
- net 5V_OUT: now also D1.K, D2.A, D2.K
- net D_N: now also R6.1; no longer R9.2
- net D_P: now also R8.1; no longer R8.2
- net N$6: now also R8.2; no longer R8.1
- net N$7: now also R6.2; no longer R9.1
Changed lines of the file:
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@@
 <?xml version="1.0" encoding="utf-8"?>
 <!DOCTYPE eagle SYSTEM "eagle.dtd">
-<eagle version="9.6.2">
+<eagle version="9.7.0">
 <drawing>
 <settings>
@@
 <layers>
 <layer number="1" name="Top" color="4" fill="1" visible="no" active="no"/>
-<layer number="2" name="Route2" color="16" fill="1" visible="no" active="no"/>
-<layer number="3" name="Route3" color="17" fill="1" visible="no" active="no"/>
-<layer number="4" name="Route4" color="18" fill="1" visible="no" active="no"/>
-<layer number="5" name="Route5" color="19" fill="1" visible="no" active="no"/>
-<layer number="6" name="Route6" color="25" fill="1" visible="no" active="no"/>
-<layer number="7" name="Route7" color="26" fill="1" visible="no" active="no"/>
-<layer number="8" name="Route8" color="27" fill="1" visible="no" active="no"/>
-<layer number="9" name="Route9" color="28" fill="1" visible="no" active="no"/>
-<layer number="10" name="Route10" color="29" fill="1" visible="no" active="no"/>
-<layer number="11" name="Route11" color="30" fill="1" visible="no" active="no"/>
-<layer number="12" name="Route12" color="20" fill="1" visible="no" active="no"/>
-<layer number="13" name="Route13" color="21" fill="1" visible="no" active="no"/>
-<layer number="14" name="Route14" color="22" fill="1" visible="no" active="no"/>
-<layer number="15" name="Route15" color="23" fill="1" visible="no" active="no"/>
+<layer number="2" name="Route2" color="16" fill="3" visible="no" active="no"/>
+<layer number="3" name="Route3" color="17" fill="3" visible="no" active="no"/>
+<layer number="4" name="Route4" color="18" fill="4" visible="no" active="no"/>
+<layer number="5" name="Route5" color="19" fill="4" visible="no" active="no"/>
+<layer number="6" name="Route6" color="25" fill="8" visible="no" active="no"/>
+<layer number="7" name="Route7" color="26" fill="8" visible="no" active="no"/>
+<layer number="8" name="Route8" color="27" fill="2" visible="no" active="no"/>
+<layer number="9" name="Route9" color="28" fill="2" visible="no" active="no"/>
+<layer number="10" name="Route10" color="29" fill="7" visible="no" active="no"/>
+<layer number="11" name="Route11" color="30" fill="7" visible="no" active="no"/>
+<layer number="12" name="Route12" color="20" fill="5" visible="no" active="no"/>
+<layer number="13" name="Route13" color="21" fill="5" visible="no" active="no"/>
+<layer number="14" name="Route14" color="22" fill="6" visible="no" active="no"/>
+<layer number="15" name="Route15" color="23" fill="6" visible="no" active="no"/>
 <layer number="16" name="Bottom" color="1" fill="1" visible="no" active="no"/>
 <layer number="17" name="Pads" color="2" fill="1" visible="no" active="no"/>
@@
 <part name="R5" library="standardparts" deviceset="RESISTOR" device=".0603" value="10k ohm"/>
 <part name="R18" library="standardparts" deviceset="RESISTOR" device=".0603" value="10k ohm"/>
-<part name="R8" library="standardparts" deviceset="RESISTOR" device=".0603" value="10k ohm"/>
-<part name="R9" library="standardparts" deviceset="RESISTOR" device=".0603" value="10k ohm"/>
 <part name="J2" library="XT60-M" deviceset="XT60-M" device=""/>
 <part name="R16" library="rcl" library_urn="urn:adsk.eagle:library:334" deviceset="R-EU_" device="R0603" package3d_urn="urn:adsk.eagle:package:23555/3" value="1k"/>
@@
 <part name="R19" library="rcl" library_urn="urn:adsk.eagle:library:334" deviceset="R-EU_" device="R0805" package3d_urn="urn:adsk.eagle:package:23553/2" value="10k"/>
 <part name="R22" library="rcl" library_urn="urn:adsk.eagle:library:334" deviceset="R-EU_" device="R0805" package3d_urn="urn:adsk.eagle:package:23553/2" value="1k"/>
+<part name="R8" library="rcl" library_urn="urn:adsk.eagle:library:334" deviceset="R-EU_" device="R0805" package3d_urn="urn:adsk.eagle:package:23553/2" value="27 ohm"/>
+<part name="R6" library="rcl" library_urn="urn:adsk.eagle:library:334" deviceset="R-EU_" device="R0805" package3d_urn="urn:adsk.eagle:package:23553/2" value="27 ohm"/>
+<part name="D2" library="SS14" deviceset="SS14" device=""/>
 </parts>
 <sheets>
@@
 <instance part="D1" gate="G$1" x="43.18" y="58.42" smashed="yes">
 <attribute name="NAME" x="38.1" y="60.96" size="1.778" layer="95"/>
-<attribute name="VALUE" x="38.1" y="54.61" size="1.778" layer="96"/>
+<attribute name="VALUE" x="40.64" y="52.07" size="1.778" layer="96"/>
 </instance>
 <instance part="U3" gate="G$1" x="99.06" y="55.88" smashed="yes">
@@
 <attribute name="NAME" x="-547.37" y="100.33" size="1.016" layer="95" rot="MR0"/>
 <attribute name="VALUE" x="-547.37" y="102.87" size="1.016" layer="96" rot="R180"/>
-</instance>
-<instance part="R8" gate="G$1" x="-414.02" y="-60.96" smashed="yes">
-<attribute name="NAME" x="-415.29" y="-59.69" size="1.016" layer="95" rot="MR90"/>
-<attribute name="VALUE" x="-412.75" y="-59.69" size="1.016" layer="96" rot="R90"/>
-</instance>
-<instance part="R9" gate="G$1" x="-414.02" y="-66.04" smashed="yes">
-<attribute name="NAME" x="-415.29" y="-64.77" size="1.016" layer="95" rot="MR90"/>
-<attribute name="VALUE" x="-412.75" y="-64.77" size="1.016" layer="96" rot="R90"/>
 </instance>
 <instance part="J2" gate="G$1" x="-40.64" y="99.06" smashed="yes" rot="R180">
@@
 <attribute name="NAME" x="-217.17" y="87.8586" size="1.778" layer="95"/>
 <attribute name="VALUE" x="-217.17" y="83.058" size="1.778" layer="96"/>
+</instance>
+<instance part="R8" gate="G$1" x="-411.48" y="-60.96" smashed="yes" rot="R180">
+<attribute name="NAME" x="-407.67" y="-64.9986" size="1.778" layer="95" rot="R270"/>
+<attribute name="VALUE" x="-407.67" y="-57.658" size="1.778" layer="96"/>
+</instance>
+<instance part="R6" gate="G$1" x="-411.48" y="-66.04" smashed="yes" rot="R180">
+<attribute name="NAME" x="-407.67" y="-70.0786" size="1.778" layer="95" rot="R270"/>
+<attribute name="VALUE" x="-407.67" y="-62.738" size="1.778" layer="96"/>
+</instance>
+<instance part="D2" gate="G$1" x="60.96" y="96.52" smashed="yes">
+<attribute name="NAME" x="55.88" y="99.06" size="1.778" layer="95"/>
+<attribute name="VALUE" x="58.42" y="90.17" size="1.778" layer="96"/>
 </instance>
 </instances>
@@
 <wire x1="-419.1" y1="-63.5" x2="-419.1" y2="-60.96" width="0.1524" layer="91"/>
 <wire x1="-419.1" y1="-60.96" x2="-416.56" y2="-60.96" width="0.1524" layer="91"/>
-<pinref part="R8" gate="G$1" pin="1"/>
+<pinref part="R8" gate="G$1" pin="2"/>
 </segment>
 </net>
@@
 <pinref part="RP2040" gate="IC$1" pin="USB_DM"/>
 <wire x1="-422.91" y1="-66.04" x2="-416.56" y2="-66.04" width="0.1524" layer="91"/>
-<pinref part="R9" gate="G$1" pin="1"/>
+<pinref part="R6" gate="G$1" pin="2"/>
 </segment>
 </net>
@@
 </segment>
 <segment>
-<wire x1="-411.48" y1="-60.96" x2="-403.86" y2="-60.96" width="0.1524" layer="91"/>
+<wire x1="-406.4" y1="-60.96" x2="-398.78" y2="-60.96" width="0.1524" layer="91"/>
 <label x="-403.86" y="-60.96" size="1.778" layer="95"/>
-<pinref part="R8" gate="G$1" pin="2"/>
+<pinref part="R8" gate="G$1" pin="1"/>
 </segment>
 </net>
@@
 </segment>
 <segment>
-<pinref part="R9" gate="G$1" pin="2"/>
-<wire x1="-411.48" y1="-66.04" x2="-403.86" y2="-66.04" width="0.1524" layer="91"/>
+<wire x1="-406.4" y1="-66.04" x2="-398.78" y2="-66.04" width="0.1524" layer="91"/>
 <label x="-403.86" y="-66.04" size="1.778" layer="95"/>
+<pinref part="R6" gate="G$1" pin="1"/>
 </segment>
 </net>
@@
 <wire x1="35.56" y1="96.52" x2="55.88" y2="96.52" width="0.1524" layer="91"/>
 <junction x="35.56" y="96.52"/>
-<label x="55.88" y="96.52" size="1.778" layer="95" xref="yes"/>
 <pinref part="C3" gate="G$1" pin="1"/>
 <pinref part="C17" gate="G$1" pin="1"/>
+<pinref part="D2" gate="G$1" pin="A"/>
 </segment>
 <segment>
@@
 <pinref part="C22" gate="G$1" pin="1"/>
 </segment>
-</net>
+<segment>
+<pinref part="D1" gate="G$1" pin="K"/>
+<wire x1="48.26" y1="58.42" x2="50.8" y2="58.42" width="0.1524" layer="91"/>
+<wire x1="50.8" y1="58.42" x2="50.8" y2="50.8" width="0.1524" layer="91"/>
+<label x="50.8" y="48.26" size="1.778" layer="95" xref="yes"/>
+</segment>
+<segment>
+<pinref part="D2" gate="G$1" pin="K"/>
+<wire x1="66.04" y1="96.52" x2="91.44" y2="96.52" width="0.1524" layer="91"/>
+<wire x1="91.44" y1="96.52" x2="91.44" y2="93.98" width="0.1524" layer="91"/>
+<label x="91.44" y="93.98" size="1.778" layer="95" xref="yes"/>
+</segment>
+</net>

Commit message: Refined the connections for peripherals
Parts:
- removed C115: 1 uF, standardparts:CAPACITOR.0603
- removed R1, R11, R12, R14, R2, R43: 10k ohm, standardparts:RESISTOR.0603
- added C13: 100nF, rcl:C-EUC0805
- added R23, R24, R9: (no value), rcl:R-EU_R0805
- C1, C2: value (none) -> 100nF
- R4, R5: value 10k ohm -> 10k; device standardparts:RESISTOR.0603 -> rcl:R-EU_R0805
Connections:
- net A renamed UART_RX
- removed net B: J3.3, RP2040.GPIO18
- removed net RESET: LCD.6
- removed net RESET_LCD: RP2040.GPIO6
- removed net SCL: IC1.SCK, R11.1, RP2040.GPIO12, U$2.SCL
- removed net SDA: IC1.SDI, R1.1, RP2040.GPIO13, U$2.SDA
- removed net VCC: R1.2, R11.2, R12.2, R14.1, R2.2
- new net RST: LCD.6, RP2040.GPIO8
- new net SCL_BMP: IC1.SCK, RP2040.GPIO12
- new net SCL_RH: R9.2, RP2040.GPIO15, U$2.SCL
- new net SDA_BMP: IC1.SDI, RP2040.GPIO11
- new net SDA_RH: R23.1, RP2040.GPIO14, U$2.SDA
- net 3V3: now also C13.1, C2.2, R23.2, R24.1, R9.1; no longer C115.2, C2.1, R43.1
- net CS_LCD: now also RP2040.GPIO9; no longer RP2040.GPIO5
- net CS_SD: now also R24.2, RP2040.GPIO5; no longer R43.2, RP2040.GPIO1
- net DC: now also RP2040.GPIO7; no longer RP2040.GPIO4
- net GND: now also C13.2, C2.1, J3.3; no longer C115.1, C2.2
- net MISO: now also RP2040.GPIO4; no longer R2.1, RP2040.GPIO0
- net MOSI: no longer R12.1, RP2040.GPIO2
- net SCK: now also RP2040.GPIO2; no longer R14.2
Other:
- note added: "BMP280"
- note added: "Humidity Sensor"
- note added: "I2C0 bus is used I2C register is 0x76 as SD0 is pulled low"
- note added: "SD Card Connector"
- note added: "SD card and display both drives on SPI0. SD card has GPIO5 as CS Display has GPIO9 as CS"
- note added: "TFT LCD Display Header Pins"
- note removed: "Mismatch in footprint and actual chip"
- note removed: "REDO"
- moved on the sheet: C2, J3, J6, LCD, R13, R18, R3, R72, U$2

Commit message: pcb
Parts:
- added U2: SI7615ADN-T1-GE3SON8_SI7615ADN-T1-GE3_VIS, 2025-03-10_11-27-14_Library:SI7615ADN-T1-GE3SON8_SI7615ADN-T1-GE3_VIS
- D1, D2: value SS14 -> SCHOTTKY_MBR0520LT1GDO-219; device SS14:SS14 -> Diode:SCHOTTKY_MBR0520LT1GDO-219
Connections:
- removed net N$9: D1.A, J1.VBUS
- new net 5V: C22.1, D1.C, D2.C, U3.VIN
- new net 5V5: D1.A, U2.5, U2.6, U2.7, U2.8
- new net USB-: D2.A, J1.VBUS, U2.4
- net 5V_OUT: now also U2.1, U2.2, U2.3; no longer C22.1, D1.K, D2.A, D2.K, U3.VIN
Other:
- moved on the sheet: C19, C21, C22, U3
