File: Eagle files/Ground-station/GND_SATION_PCB_1.02.sch (EAGLE design)
At the start: 63 parts, among them IC1 BMP280, J1 USB4110GFA, J2 XT60-M, J3 B4B-XH-AM_(LF)(SN), J6 503182-1852, U1 AMS1117-5.0, U2 SI7615ADN-T1-GE3SON8_SI7615AD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, U3 AMS1117-3.3, U4 SOIC127P790X216-8NW25Q128JVJSQ

Commit message: gs 1.0 update
Parts:
- removed C13, C2: 100nF, rcl:C-EUC0805
- removed C20: 100nF, rcl:C-EUC0603
- removed J3: B4B-XH-AM_(LF)(SN), B4B-XH-AM__LF__SN_:B4B-XH-AM_(LF)(SN)
- removed J6: 503182-1852, 503182-1852:503182-1852
- removed R13, R72: 10k ohm, standardparts:RESISTOR.0603
- removed R15: 1k, rcl:R-EU_R0805
- removed R17: 10k, rcl:R-EU_R0603
- removed R24: (no value), rcl:R-EU_R0805
- removed R5: 10k, rcl:R-EU_R0805
- removed S2: DTS-3, DTS-3:DTS-3
- added C40: 10 uF, standardparts:CAPACITOR.0603
- added R1: 1k, rcl:R-EU_R0805
- added R2: 10k ohm, standardparts:RESISTOR.0603
- added XBEE: XBP9B-XCST-021, XBP9B-XCST-021:XBP9B-XCST-021
- C1: value 100nF -> 10 uF; device rcl:C-EUC0805 -> standardparts:CAPACITOR.0603
- R23, R9: value (none) -> 10k
- R4: value 10k -> 10k ohm; device rcl:R-EU_R0805 -> standardparts:RESISTOR.0603
Connections:
- removed net +3V3: C10.1, C11.1, C12.1, C15.1, C16.1, C7.1, C8.1, C9.1, R17.1, RP2040.ADC_AVDD, RP2040.IOVDD0, RP2040.IOVDD1, RP2040.IOVDD2, RP2040.IOVDD3, RP2040.IOVDD4, RP2040.IOVDD5, RP2040.USB_VDD, RP2040.VREG_IN
- removed net CS_SD: J6.CD/DAT3, R24.2, RP2040.GPIO5
- removed net N$1: IC1.SDO, R4.2
- removed net N$11: C23.1, R15.1, U$3.OUT
- removed net N$12: J6.DAT1, R72.1
- removed net N$14: C20.1, R17.2, RP2040.RUN, S2.2
- removed net N$3: IC1.CSB, R5.2
- removed net N$8: J6.DATA2, R13.1
- removed net QSPI_SCLK: RP2040.QSPI_SCLK
- removed net QSPI_SD0: RP2040.QSPI_SD0
- removed net QSPI_SD1: RP2040.QSPI_SD1
- removed net QSPI_SD2: RP2040.QSPI_SD2
- removed net QSPI_SD3: RP2040.QSPI_SD3
- removed net QSPI_SS: RP2040.QSPI_SS
- removed net SCL_BMP: IC1.SCK, RP2040.GPIO12
- removed net SCL_RH: R9.2, RP2040.GPIO15, U$2.SCL
- removed net SDA_BMP: IC1.SDI, RP2040.GPIO11
- removed net SDA_RH: R23.1, RP2040.GPIO14, U$2.SDA
- new net CSB: IC1.CSB, R4.1
- new net CTS: XBEE.NCTS/DIO7
- new net DTR: XBEE.NDTR/SLEEP_RQ/DIO8
- new net FLASH_HOLD: RP2040.QSPI_SD3, U4./HOLD(IO3)
- new net FLASH_WP: RP2040.QSPI_SD2, U4./WP(IO2)
- new net MOSI_SD: LCD.4, R3.2
- new net RSSI: XBEE.DIO10/PWM0
- new net RTS: XBEE.NRTS/DIO6
- new net SCL: IC1.SCK, R9.2, RP2040.GPIO12, U$2.SCL
- new net SDA: IC1.SDI, R23.1, RP2040.GPIO11, U$2.SDA
- new net SDO1: IC1.SDO, R2.2
- new net TEL_RST: XBEE.!RESET
- new net TEL_RX: XBEE.DIN/NCONFIG/DIO14
- new net TEL_TX: XBEE.DOUT/DIO13
- net 3V3: now also C40.2, XBEE.VCC; no longer C1.2, C13.1, C2.2, IC1.VDD, IC1.VDDIO, J6.VDD, R13.2, R24.1, R5.1, U4./HOLD(IO3), U4./WP(IO2)
- net 3V3_OP: now also C1.2, C10.1, C11.1, C12.1, C15.1, C16.1, C7.1, C8.1, C9.1, IC1.VDD, IC1.VDDIO, R4.2, RP2040.ADC_AVDD, RP2040.IOVDD0, RP2040.IOVDD1, RP2040.IOVDD2, RP2040.IOVDD3, RP2040.IOVDD4, RP2040.IOVDD5, RP2040.RUN, RP2040.USB_VDD, RP2040.VREG_IN; no longer R72.2
- net 3V3_OUT: no longer RP2040.GPIO24
- net 5V_OUT: no longer J3.2
- net FLASH_CLK: now also RP2040.QSPI_SCLK
- net FLASH_CS: now also RP2040.QSPI_SS
- net FLASH_DI: now also RP2040.QSPI_SD0
- net FLASH_DO: now also RP2040.QSPI_SD1
- net GND: now also C40.1, R2.1, XBEE.GND; no longer C13.2, C2.1, C20.2, J3.1, J3.3, J6.VSS, R4.1, S2.1
- net MISO: no longer J6.DAT0
- net MOSI: no longer J6.CMD, LCD.4, R3.2
- net SCK: no longer J6.CLK
- net UART_RX: no longer J3.4
- net XIN: now also C23.1, U$3.OUT; no longer R15.2
- net XOUT: now also R1.1, R1.2
Other:
- note added: "XBEE??"
- note removed: "SD Card Connector"
- moved on the sheet: C17, C18, C19, C21, C22, C23, C24, C3, D1, D2, IC1, J1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

Commit message: gs updates
Parts:
- removed C17, C19, C21, C22: 10uF, rcl:C-EUC0805
- removed CN1, CN2, CN3: (no value), microbuilder:HEADER_1X02
- removed D1, D2: SCHOTTKY_MBR0520LT1GDO-219, Diode:SCHOTTKY_MBR0520LT1GDO-219
- removed J1: USB4110GFA, USB4110GFA:USB4110GFA
- removed LCD: (no value), microbuilder:HEADER-1X9
- removed R10: 5.1k, rcl:R-EU_R0805
- removed R16, R20, R21: 1k, rcl:R-EU_R0603
- removed R18, R3: 10k ohm, standardparts:RESISTOR.0603
- removed R6, R8: 27 ohm, rcl:R-EU_R0805
- removed U3: AMS1117-3.3, AMS1117-3.3:AMS1117-3.3
- added C13: 22uF, rcl:C-EUC0805
- added C2: 10uF, rcl:C-EUC0805
- added D3, D4: SCHOTTKY_MBR0520LT1GDO-219, Diode:SCHOTTKY_MBR0520LT1GDO-219
- added Q3: SI7625DN-T1-GE3, SI7625DN-T1-GE3:SI7625DN-T1-GE3
- added R5: 5.1k ohm, standardparts:RESISTOR.0603
- added SV1: (no value), con-lsta:FE10-1
- added X1: USB Type C, microbuilder:USB_C
- C3: value 10uF -> 22uF
- R7: value 5.1k -> 5.1k ohm; device rcl:R-EU_R0805 -> standardparts:RESISTOR.0603
- U2: value SI7615ADN-T1-GE3SON8_SI7615ADN-T1-GE3_VIS -> AMS1117-3.3; device 2025-03-10_11-27-14_Library:SI7615ADN-T1-GE3SON8_SI7615ADN-T1-GE3_VIS -> AMS1117-3.3:AMS1117-3.3
Connections:
- removed net 0: R16.1, R20.1, R21.1
- removed net 3V3_OUT: CN1.1
- removed net 5V5: D1.A, U2.5, U2.6, U2.7, U2.8
- removed net 5V_OUT: C17.1, C3.1, U1.VOUT, U2.1, U2.2, U2.3
- removed net DC: LCD.5, RP2040.GPIO7
- removed net D_N: J1.DN1, J1.DN2, R6.1
- removed net D_P: J1.DP1, J1.DP2, R8.1
- removed net MOSI_SD: LCD.4, R3.2
- removed net N$10: CN1.2, CN2.1, CN3.1, R16.2
- removed net N$15: J1.CC2, R10.2
- removed net N$18: CN3.2, R20.2, RP2040.GPIO20
- removed net N$19: CN2.2, R21.2, RP2040.GPIO21
- removed net N$5: J1.CC1, R7.2
- removed net N$7: R6.2, RP2040.USB_DM
- removed net RST: LCD.6, RP2040.GPIO8
- removed net SDO: LCD.1, R3.1
- removed net UART_RX: RP2040.GPIO17
- removed net USB-: D2.A, J1.VBUS, U2.4
- new net 5V_BATT: C3.1, D4.C, Q3.S_1, Q3.S_2, Q3.S_3, U1.VOUT
- new net 5V_USB: D3.A, X1.VBUS
- new net CC3: R5.1, X1.CC2
- new net CC4: R7.1, X1.CC1
- new net CLK: SV1.3
- new net D+: X1.D+
- new net D-: X1.D-
- new net N$1: D4.A
- new net N$12: SV1.10
- new net N$3: C2.1
- new net N$4: SV1.5
- new net Q1-G: Q3.G
- new net RST_LSD: SV1.6
- net 3V3: now also C1.2, IC1.VDD, IC1.VDDIO, R4.2, SV1.2, SV1.9; no longer C19.1, C21.1, LCD.2, LCD.9, R18.2, U3.VOUT, U4.VCC
- net 3V3_OP: now also U4.VCC; no longer C1.2, IC1.VDD, IC1.VDDIO, R4.2
- net 5V: now also D3.C, Q3.D_1, Q3.D_2, Q3.D_3, Q3.D_4, Q3.D_5, Q3.D_6, Q3.D_7, U2.VIN; no longer C22.1, D1.C, D2.C, U3.VIN
- net CS_LCD: now also SV1.7; no longer LCD.7, R18.1, RP2040.GPIO9
- net GND: now also C13.2, C2.2, R5.2, R7.2, SV1.8, U2.GND/ADJ, X1.GND; no longer C17.2, C19.2, C21.2, C22.2, J1.GND, LCD.8, R10.1, R7.1, U3.GND/ADJ
- net MISO: now also SV1.1
- net MOSI: now also SV1.4
- net N$6: now also C13.1, U2.VOUT; no longer R8.2, RP2040.USB_DP
- net SCK: no longer LCD.3
- net SCL: now also RP2040.GPIO11; no longer RP2040.GPIO12
- net SDA: now also RP2040.GPIO12; no longer RP2040.GPIO11
Other:
- note removed: "SD card and display both drives on SPI0. SD card has GPIO5 as CS Display has GPIO9 as CS"
- moved on the sheet: C1, C10, C11, C12, C15, C16, C18, C23, C24, C4, C40, C5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
