File: Eagle files/FLYTE 3/FLYTE 3.02/FLYTE_3.02.sch (EAGLE design)
At the start: 198 parts, among them IC1 BMP280, IC2 MPXV5100DP, IC9 MCP73844-840I_MS, J1 JST-XH-2B, J2 CON-SMA-EDGE-S, J3 JST-XH-2B, J7 XT60-M, Q1 SI7625DN-T1-GE3, Q3 SI7625DN-T1-GE3, Q4 SI7625DN-T1-GE3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

Commit message: gs updates
Other:
- moved on the sheet: C101, C18, C25, C27, C42, C52, D10, D11, D13, D2, D3, D4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
