File: Eagle files/Ground-station/past_iters/GND_STN.sch (EAGLE design)
At the start: 43 parts, among them IC1 BMP280, J2 XT60-M, Q3 SI7625DN-T1-GE3, U1 AMS1117-5.0, U2 AMS1117-3.3, U4 SOIC127P790X216-8NW25Q128JVJSQ, X1 USB Type C

Commit message: .
Parts:
- removed C15, C16: 100nF, rcl:C-EUC0603
- removed C18: 10uF, rcl:C-EUC0805
- removed C23, C24: 18pF, rcl:C-EUC0805
- removed C40: 10 uF, standardparts:CAPACITOR.0603
- removed D3, D4: SCHOTTKY_MBR0520LT1GDO-219, Diode:SCHOTTKY_MBR0520LT1GDO-219
- removed IC1: BMP280, BMP280-standalone:BMP280
- removed J2: XT60-M, XT60-M:XT60-M
- removed Q3: SI7625DN-T1-GE3, SI7625DN-T1-GE3:SI7625DN-T1-GE3
- removed R19, R23, R9: 10k, rcl:R-EU_R0805
- removed R22: 1k, rcl:R-EU_R0805
- removed R7: 5.1k ohm, standardparts:RESISTOR.0603
- removed S3: DTS-3, DTS-3:DTS-3
- removed SV1: (no value), con-lsta:FE10-1
- removed U$2: HDC1080, Texas-HDC1080:HDC1080
- removed U$3: ASE, crystal:ASE
- removed U1: AMS1117-5.0, AMS1117-5.0:AMS1117-5.0
- removed U4: SOIC127P790X216-8NW25Q128JVJSQ, SOIC127P790X216-8N:SOIC127P790X216-8NW25Q128JVJSQ
- removed X1: USB Type C, microbuilder:USB_C
- removed XBEE: XBP9B-XCST-021, XBP9B-XCST-021:XBP9B-XCST-021
- added C14: 15pF, rcl:C-EUC0603
- added R3: 27.4, rcl:R-EU_R0603
- added S1: DTS-3, DTS-3:DTS-3
- added U$1: ABM8-272-T3, ABM8-272-T3:ABM8-272-T3
- C1: value 10 uF -> 100nF; device standardparts:CAPACITOR.0603 -> rcl:C-EUC0603
- C13: value 22uF -> 15pF; device rcl:C-EUC0805 -> rcl:C-EUC0603
- C2: value 10uF -> 100nF; device rcl:C-EUC0805 -> rcl:C-EUC0603
- C3: value 22uF -> 100nF; device rcl:C-EUC0805 -> rcl:C-EUC0603
- C4, C5: value 100nF -> 1uF
- C6, C7: value 1uF -> 100nF
- R1: value 1k -> 10k; device rcl:R-EU_R0805 -> rcl:R-EU_R0603
- R2: value 10k ohm -> 1k; device standardparts:RESISTOR.0603 -> rcl:R-EU_R0603
- R4: value 10k ohm -> 27.4; device standardparts:RESISTOR.0603 -> rcl:R-EU_R0603
- R5: value 5.1k ohm -> 1k; device standardparts:RESISTOR.0603 -> rcl:R-EU_R0603
- U2: value AMS1117-3.3 -> SOIC127P790X216-8NW25Q128JVJSQ; device AMS1117-3.3:AMS1117-3.3 -> SOIC127P790X216-8N:SOIC127P790X216-8NW25Q128JVJSQ
Connections:
- net SCK renamed CAM
- removed net 3V3: C1.2, C40.2, IC1.VDD, IC1.VDDIO, R19.2, R23.2, R4.2, R9.1, SV1.2, SV1.9, U$2.VDD, XBEE.VCC
- removed net 3V3_OP: C10.1, C11.1, C12.1, C15.1, C16.1, C7.1, C8.1, C9.1, RP2040.ADC_AVDD, RP2040.IOVDD0, RP2040.IOVDD1, RP2040.IOVDD2, RP2040.IOVDD3, RP2040.IOVDD4, RP2040.IOVDD5, RP2040.RUN, RP2040.USB_VDD, RP2040.VREG_IN, U4.VCC
- removed net 5V: D3.C, Q3.D_1, Q3.D_2, Q3.D_3, Q3.D_4, Q3.D_5, Q3.D_6, Q3.D_7, U2.VIN
- removed net 5V_BATT: C3.1, D4.C, Q3.S_1, Q3.S_2, Q3.S_3, U1.VOUT
- removed net 5V_USB: D3.A, X1.VBUS
- removed net CC3: R5.1, X1.CC2
- removed net CC4: R7.1, X1.CC1
- removed net CLK: SV1.3
- removed net CSB: IC1.CSB, R4.1
- removed net CS_LCD: SV1.7
- removed net CTS: XBEE.NCTS/DIO7
- removed net D+: X1.D+
- removed net D-: X1.D-
- removed net DTR: XBEE.NDTR/SLEEP_RQ/DIO8
- removed net FLASH_CLK: RP2040.QSPI_SCLK, U4.CLK
- removed net FLASH_CS: R19.1, R22.2, RP2040.QSPI_SS, U4./CS
- removed net FLASH_DI: RP2040.QSPI_SD0, U4.DI(IO0)
- removed net FLASH_DO: RP2040.QSPI_SD1, U4.DO(I01)
- removed net FLASH_HOLD: RP2040.QSPI_SD3, U4./HOLD(IO3)
- removed net FLASH_WP: RP2040.QSPI_SD2, U4./WP(IO2)
- removed net GND: C1.1, C10.2, C11.2, C12.2, C13.2, C15.2, C16.2, C18.2, C2.2, C23.2, C24.1, C3.2, C4.2, C40.1, C5.2, C6.2, C7.2, C8.2, C9.2, IC1.GND, J2.NEG, R2.1, R5.2, R7.2, RP2040.GND, RP2040.TESTEN, S3.1, SV1.8, U$2.GND, U$3.GND, U$3.VDD, U1.GND/ADJ, U2.GND/ADJ, U4.GND, X1.GND, XBEE.GND
- removed net MISO: RP2040.GPIO4, SV1.1
- removed net MOSI: RP2040.GPIO3, SV1.4
- removed net N$12: SV1.10
- removed net N$16: C18.1, J2.POS, U1.VIN
- removed net N$6: C13.1, U2.VOUT
- removed net Q1-G: Q3.G
- removed net RST_LSD: SV1.6
- removed net RTS: XBEE.NRTS/DIO6
- removed net SDO1: IC1.SDO, R2.2
- new net +3V3: C1.1, C10.1, C11.1, C12.1, C5.1, C6.1, C7.1, C8.1, C9.1, R1.2, RP2040.ADC_AVDD, RP2040.IOVDD0, RP2040.IOVDD1, RP2040.IOVDD2, RP2040.IOVDD3, RP2040.IOVDD4, RP2040.IOVDD5, RP2040.RUN, RP2040.USB_VDD, RP2040.VREG_IN, U2.VCC
- new net 0: C1.2, C10.2, C11.2, C12.2, C13.1, C14.1, C2.2, C3.2, C4.2, C5.2, C6.2, C7.2, C8.2, C9.2, RP2040.GND, RP2040.TESTEN, S1.1, U$1.2, U$1.4, U2.GND
- new net BUZZER: RP2040.GPIO0
- new net CTRL: RP2040.GPIO3
- new net DROGUE: RP2040.GPIO18
- new net FIN_1: RP2040.GPIO7
- new net FIN_2: RP2040.GPIO6
- new net FIN_3: RP2040.GPIO5
- new net FIN_4: RP2040.GPIO4
- new net GPS_RX: RP2040.GPIO16
- new net GPS_TX: RP2040.GPIO17
- new net IGN1: RP2040.GPIO20
- new net IGN2: RP2040.GPIO21
- new net LED: RP2040.GPIO1
- new net MAIN: RP2040.GPIO19
- new net QSPI_SCLK: RP2040.QSPI_SCLK, U2.CLK
- new net QSPI_SD0: RP2040.QSPI_SD0, U2.DI(IO0)
- new net QSPI_SD1: RP2040.QSPI_SD1, U2.DO(I01)
- new net QSPI_SD2: RP2040.QSPI_SD2, U2./WP(IO2)
- new net QSPI_SD3: RP2040.QSPI_SD3, U2./HOLD(IO3)
- new net QSPI_SS: R1.1, R2.2, RP2040.QSPI_SS, U2./CS
- net 1V1: now also C2.1, C3.1; no longer C5.1, C6.1
- net N$1: now also C14.2, R5.1, U$1.3; no longer D4.A
- net N$2: now also R2.1, S1.2; no longer R22.1, S3.2
- net N$3: now also R3.1, RP2040.USB_DP; no longer C2.1
- net N$4: now also R4.1, RP2040.USB_DM; no longer SV1.5
- net RSSI: now also RP2040.GPIO23; no longer XBEE.DIO10/PWM0
- net SCL: now also RP2040.GPIO13; no longer IC1.SCK, R9.2, RP2040.GPIO11, U$2.SCL
- net SDA: no longer IC1.SDI, R23.1, U$2.SDA
- net TEL_RST: now also RP2040.GPIO22; no longer XBEE.!RESET
- net TEL_RX: now also RP2040.GPIO24; no longer XBEE.DIN/NCONFIG/DIO14
- net TEL_TX: now also RP2040.GPIO25; no longer XBEE.DOUT/DIO13
- net XIN: now also C13.2, U$1.1; no longer C23.1, U$3.OUT
- net XOUT: now also R5.2; no longer C24.2, R1.1, R1.2, U$3.TRI
Other:
- note added: "GROUND STATION COMPUTER"
- note removed: "BMP280"
- note removed: "Crystal Oscillator"
- note removed: "Flash chip (W25Q125JV)"
- note removed: "Humidity Sensor"
- note removed: "I2C0 bus is used I2C register is 0x76 as SD0 is pulled low"
- note removed: "Power Supply"
- note removed: "TFT LCD Display Header Pins"
- note removed: "Use YSX321SL 12pF 10PPM oscillator. If of different load resistance change the C23 and C24."
- note removed: "XBEE??"
- moved on the sheet: C10, C11, C12, C13, C2, C4, C5, C6, C7, C8, C9, R1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
